File: kicad/ALU/ALU.kicad_sch (KiCad schematic)
At the start: 85 parts, among them J1 Control Connector, J10 Backplane Signal, J2 Data Connector, J20 Backplane Bus, U1 74LS377, U10 74LS253, U11 74LS253, U12 74LS253, U13 74LS253, U14 74LS253, U15 74LS253, U16 74LS253, U17 74F382, U18 74F382, U19 74F382, U2 74LS377, U20 74F382, U21 74F382, U22 74LS283, U23 74LS283, U24 74LS283, U25 74LS283, U26 74LS283, U27 74LS244, U28 74LS244, U29 74LS244, U3 74LS377, U30 74LS386, U31 74LS08, U32 74LS32, U33 74LS04, U34 74LS253, U35 74LS27, U36 74LS27, U37 74LS11, U38 74LS257, U39 74LS32, U4 74LS377, U5 74LS377, U6 74LS377, U7 74LS253, U8 74LS253, U9 74LS253

Commit message: Fix electrical rule issues
Parts:
- removed J10: Backplane Signal, symbol Connector_Generic:Conn_02x30_Odd_Even
- removed J20: Backplane Bus, symbol Connector_Generic:Conn_02x20_Odd_Even
Connections:
- net *ARITH_OUT: now reaches U27.1 (OEa), U27.19 (OEb), U28.1 (OEa), U28.19 (OEb), U29.1 (OEa), U29.19 (OEb), U39.3
- net *SHIFT_OUT: now reaches U10.1 (OEa), U10.15 (OEb), U11.1 (OEa), U11.15 (OEb), U12.1 (OEa), U12.15 (OEb), U13.1 (OEa), U13.15 (OEb), U14.1 (OEa), U14.15 (OEb), U15.1 (OEa), U15.15 (OEb), U39.6, U7.1 (OEa), U7.15 (OEb), U8.1 (OEa), U8.15 (OEb), U9.1 (OEa), U9.15 (OEb)
- net FLAG_SIGN renamed OB17
- no-connect marks 187 -> 113
Other:
- moved on the sheet: J1, J2

Commit message: Finish control logic
Connections:
- net EXTRA10 renamed MA_AUTO_INX
- net EXTRA11 renamed FP0
- net EXTRA12 renamed FP1
- net EXTRA13 renamed FP2
- net EXTRA14 renamed FP3
- net EXTRA9 renamed REST_PEND
Changed lines of the file:
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@@
-    (effects (font (size 1.27 1.27)) (justify right bottom))
-  )
-  (label "EXTRA13" (at 501.015 210.82 180) (fields_autoplaced)
     (effects (font (size 1.27 1.27)) (justify right bottom))
   )
@@
     (effects (font (size 1.27 1.27)) (justify left bottom))
   )
-  (label "EXTRA11" (at 501.015 208.28 180) (fields_autoplaced)
-    (effects (font (size 1.27 1.27)) (justify right bottom))
-  )
   (label "FLAG_AC_SIGN" (at 513.715 41.91 0) (fields_autoplaced)
     (effects (font (size 1.27 1.27)) (justify left bottom))
@@
     (effects (font (size 1.27 1.27)) (justify left bottom))
   )
+  (label "FP2" (at 501.015 210.82 180) (fields_autoplaced)
+    (effects (font (size 1.27 1.27)) (justify right bottom))
+  )
   (label "MB5" (at 77.47 213.36 180) (fields_autoplaced)
     (effects (font (size 1.27 1.27)) (justify right bottom))
@@
     (effects (font (size 1.27 1.27)) (justify right bottom))
   )
+  (label "FP0" (at 501.015 208.28 180) (fields_autoplaced)
+    (effects (font (size 1.27 1.27)) (justify right bottom))
+  )
   (label "D6" (at 179.07 123.19 0) (fields_autoplaced)
     (effects (font (size 1.27 1.27)) (justify left bottom))
@@
     (effects (font (size 1.27 1.27)) (justify left bottom))
   )
-  (label "EXTRA10" (at 513.715 205.74 0) (fields_autoplaced)
-    (effects (font (size 1.27 1.27)) (justify left bottom))
-  )
   (label "OB8" (at 116.84 199.39 180) (fields_autoplaced)
     (effects (font (size 1.27 1.27)) (justify right bottom))
@@
     (effects (font (size 1.27 1.27)) (justify right bottom))
   )
-  (label "EXTRA9" (at 501.015 205.74 180) (fields_autoplaced)
-    (effects (font (size 1.27 1.27)) (justify right bottom))
-  )
   (label "D13" (at 71.12 59.69 0) (fields_autoplaced)
     (effects (font (size 1.27 1.27)) (justify left bottom))
@@
     (effects (font (size 1.27 1.27)) (justify right bottom))
   )
+  (label "MA_AUTO_INX" (at 513.715 205.74 0) (fields_autoplaced)
+    (effects (font (size 1.27 1.27)) (justify left bottom))
+  )
   (label "AR16" (at 403.86 46.99 180) (fields_autoplaced)
     (effects (font (size 1.27 1.27)) (justify right bottom))
@@
     (effects (font (size 1.27 1.27)) (justify right bottom))
   )
+  (label "REST_PEND" (at 501.015 205.74 180) (fields_autoplaced)
+    (effects (font (size 1.27 1.27)) (justify right bottom))
+  )
   (label "OB11" (at 102.87 54.61 180) (fields_autoplaced)
     (effects (font (size 1.27 1.27)) (justify right bottom))
@@
     (effects (font (size 1.27 1.27)) (justify right bottom))
   )
-  (label "EXTRA12" (at 513.715 208.28 0) (fields_autoplaced)
-    (effects (font (size 1.27 1.27)) (justify left bottom))
-  )
   (label "OB8" (at 35.56 353.06 180) (fields_autoplaced)
     (effects (font (size 1.27 1.27)) (justify right bottom))
@@
     (effects (font (size 1.27 1.27)) (justify right bottom))
   )
+  (label "FP1" (at 513.715 208.28 0) (fields_autoplaced)
+    (effects (font (size 1.27 1.27)) (justify left bottom))
+  )
   (label "OB13" (at 156.21 201.93 180) (fields_autoplaced)
     (effects (font (size 1.27 1.27)) (justify right bottom))
   )
+  (label "FP3" (at 513.715 210.82 0) (fields_autoplaced)
+    (effects (font (size 1.27 1.27)) (justify left bottom))
+  )
   (label "*DEV_REQ" (at 501.015 41.91 180) (fields_autoplaced)
     (effects (font (size 1.27 1.27)) (justify right bottom))
@@
     (effects (font (size 1.27 1.27)) (justify left bottom))
   )
-  (label "EXTRA14" (at 513.715 210.82 0) (fields_autoplaced)
-    (effects (font (size 1.27 1.27)) (justify left bottom))
-  )
