File: kicad/ALU/ALU.kicad_sch (KiCad schematic)
At the start: 83 parts, among them J1 Control Connector, J2 Data Connector, U1 74LS377, U10 74LS253, U11 74LS253, U12 74LS253, U13 74LS253, U14 74LS253, U15 74LS253, U16 74LS253, U17 74F382, U18 74F382, U19 74F382, U2 74LS377, U20 74F382, U21 74F382, U22 74LS283, U23 74LS283, U24 74LS283, U25 74LS283, U26 74LS283, U27 74LS244, U28 74LS244, U29 74LS244, U3 74LS377, U30 74LS386, U31 74LS08, U32 74LS32, U33 74LS04, U34 74LS253, U35 74LS27, U36 74LS27, U37 74LS11, U38 74LS257, U39 74LS32, U4 74LS377, U5 74LS377, U6 74LS377, U7 74LS253, U8 74LS253, U9 74LS253

Commit message: Start work on memory / addressing board
Connections:
- net WRITE_CORE renamed *WRITE_CORE
Changed lines of the file:
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@@
     (effects (font (size 1.27 1.27)) (justify left bottom))
   )
-  (label "WRITE_CORE" (at 501.015 77.47 180) (fields_autoplaced)
+  (label "*WRITE_CORE" (at 501.015 77.47 180) (fields_autoplaced)
     (effects (font (size 1.27 1.27)) (justify right bottom))
   )

Commit message: Continue work on memory board
Connections:
- net EXTRA7 renamed NEXT_BANK0
- net EXTRA8 renamed NEXT_BANK1
- net REST_PEND renamed *REST_PEND

Commit message: Work on ALU PCB layout
Parts:
- removed U30: 74LS386, symbol 74xx:74LS386
- added U30: 74LS86, Package_DIP:DIP-14_W7.62mm, symbol 74xx:74LS86
- C1, C10, C11, C12, C13, C14, C15, C16, C17, C18, C19, C2, C20, C21, C22, C23, C24, C25, C26, C27, C28, C29, C3, C30, C31, C32, C33, C34, C35, C36, C37, C38, C39, C4, C5, C6, C7, C8, C9: footprint (none) -> Capacitor_THT:C_Disc_D5.0mm_W2.5mm_P5.00mm
- J1, J2: footprint (none) -> Connector_DIN:DIN41612_B_2x32_Male_Horizontal_THT
- R1, R2: footprint (none) -> Resistor_THT:R_Axial_DIN0207_L6.3mm_D2.5mm_P7.62mm_Horizontal
- U1, U17, U18, U19, U2, U20, U21, U27, U28, U29, U3, U4, U5, U6: footprint (none) -> Package_DIP:DIP-20_W7.62mm
- U10, U11, U12, U13, U14, U15, U16, U22, U23, U24, U25, U26, U34, U38, U7, U8, U9: footprint (none) -> Package_DIP:DIP-16_W7.62mm
- U31, U32, U33, U35, U36, U37, U39: footprint (none) -> Package_DIP:DIP-14_W7.62mm
Connections:
- net +5V: now also U30.14 (VCC)
- net AR17: now also U30.1
- net ARITH_CARRY_OUT: now also U30.10
- net FLAG_LINK: now also U30.9
- net GND: now also U30.12, U30.13, U30.7 (GND)
- net MB17: now also U30.5
- net OB17: now also U30.2
- net at U31.10: now also U30.6
- net at U33.4: now also U30.4
- net at U31.9: now also U30.3
- net at U32.2: now also U30.8

Commit message: Finish pinout audit + fanout correction
Connections:
- net *SHIFT_OUT: now also U39.10, U39.9; no longer U10.1 (OEa), U10.15 (OEb), U11.1 (OEa), U11.15 (OEb), U7.1 (OEa), U7.15 (OEb), U8.1 (OEa), U8.15 (OEb), U9.1 (OEa), U9.15 (OEb)
- net FLAG_LINK: now also U39.11, U39.12, U39.13
- net GND: no longer U39.10, U39.12, U39.13, U39.9
- net at U39.8: now also U10.1 (OEa), U10.15 (OEb), U11.1 (OEa), U11.15 (OEb), U7.1 (OEa), U7.15 (OEb), U8.1 (OEa), U8.15 (OEb), U9.1 (OEa), U9.15 (OEb)
- no-connect marks 113 -> 112
Other:
- moved on the sheet: U39C, U39D
Changed lines of the file:
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@@
   (junction (at 342.265 175.895) (diameter 0) (color 0 0 0 0)
   )
+  (junction (at 224.155 170.815) (diameter 0) (color 0 0 0 0)
+  )
   (junction (at 342.9 91.44) (diameter 0) (color 0 0 0 0)
   )
@@
   (junction (at 274.32 196.215) (diameter 0) (color 0 0 0 0)
   )
-  (junction (at 184.785 175.895) (diameter 0) (color 0 0 0 0)
-  )
   (junction (at 27.94 306.705) (diameter 0) (color 0 0 0 0)
   )
@@
   (junction (at 342.265 153.67) (diameter 0) (color 0 0 0 0)
   )
+  (junction (at 451.485 41.275) (diameter 0) (color 0 0 0 0)
+  )
   (junction (at 416.56 80.01) (diameter 0) (color 0 0 0 0)
   )
@@
   (junction (at 140.97 101.6) (diameter 0) (color 0 0 0 0)
   )
+  (junction (at 224.155 175.895) (diameter 0) (color 0 0 0 0)
+  )
   (junction (at 111.76 57.15) (diameter 0) (color 0 0 0 0)
   )
@@
   (junction (at 146.05 183.515) (diameter 0) (color 0 0 0 0)
   )
+  (junction (at 184.785 175.895) (diameter 0) (color 0 0 0 0)
+  )
   (junction (at 68.58 241.935) (diameter 0) (color 0 0 0 0)
   )
@@
   (junction (at 387.985 148.59) (diameter 0) (color 0 0 0 0)
   )
-  (junction (at 327.025 360.68) (diameter 0) (color 0 0 0 0)
-  )
   (junction (at 403.86 64.77) (diameter 0) (color 0 0 0 0)
   )
@@
   (junction (at 403.86 72.39) (diameter 0) (color 0 0 0 0)
   )
-  (junction (at 327.025 374.65) (diameter 0) (color 0 0 0 0)
-  )
   (junction (at 74.93 288.29) (diameter 0) (color 0 0 0 0)
   )
@@
   (junction (at 345.44 224.79) (diameter 0) (color 0 0 0 0)
   )
-  (junction (at 224.155 175.895) (diameter 0) (color 0 0 0 0)
-  )
   (junction (at 64.77 241.935) (diameter 0) (color 0 0 0 0)
   )
@@
   (no_connect (at 487.68 29.21))
   (no_connect (at 527.05 82.55))
-  (no_connect (at 342.265 372.11))
   (no_connect (at 487.68 77.47))
   (no_connect (at 527.05 172.72))
@@
     (stroke (width 0) (type default))
   )
+  (wire (pts (xy 441.96 41.275) (xy 451.485 41.275))
+    (stroke (width 0) (type default))
+  )
   (wire (pts (xy 353.06 54.61) (xy 355.6 54.61))
     (stroke (width 0) (type default))
@@
     (stroke (width 0) (type default))
   )
-  (wire (pts (xy 327.025 355.6) (xy 327.025 360.68))
-    (stroke (width 0) (type default))
-  )
   (wire (pts (xy 71.12 270.51) (xy 74.93 270.51))
     (stroke (width 0) (type default))
@@
     (stroke (width 0) (type default))
   )
+  (wire (pts (xy 224.155 170.815) (xy 224.155 175.895))
+    (stroke (width 0) (type default))
+  )
   (wire (pts (xy 139.7 262.89) (xy 143.51 262.89))
     (stroke (width 0) (type default))
@@
     (stroke (width 0) (type default))
   )
+  (wire (pts (xy 208.915 173.355) (xy 208.915 175.895))
+    (stroke (width 0) (type default))
+  )
   (bus (pts (xy 26.67 309.245) (xy 224.79 309.245))
     (stroke (width 0) (type default))
@@
     (stroke (width 0) (type default))
   )
-  (wire (pts (xy 441.96 101.6) (xy 441.96 18.415))
-    (stroke (width 0) (type default))
-  )
   (wire (pts (xy 30.48 375.92) (xy 35.56 375.92))
     (stroke (width 0) (type default))
@@
     (stroke (width 0) (type default))
   )
+  (wire (pts (xy 224.155 170.815) (xy 224.155 153.67))
+    (stroke (width 0) (type default))
+  )
   (wire (pts (xy 193.04 285.75) (xy 193.04 283.21))
     (stroke (width 0) (type default))
@@
     (stroke (width 0) (type default))
   )
+  (wire (pts (xy 441.96 101.6) (xy 441.96 41.275))
+    (stroke (width 0) (type default))
+  )
   (wire (pts (xy 447.675 272.415) (xy 448.945 272.415))
     (stroke (width 0) (type default))
@@
     (stroke (width 0) (type default))
   )
-  (wire (pts (xy 224.155 175.895) (xy 224.155 153.67))
-    (stroke (width 0) (type default))
-  )
   (bus (pts (xy 264.16 120.65) (xy 264.16 123.19))
     (stroke (width 0) (type default))
@@
     (stroke (width 0) (type default))
   )
-  (wire (pts (xy 327.025 369.57) (xy 327.025 374.65))
-    (stroke (width 0) (type default))
-  )
   (wire (pts (xy 111.76 99.06) (xy 111.76 72.39))
     (stroke (width 0) (type default))
@@
     (stroke (width 0) (type default))
   )
+  (wire (pts (xy 208.915 175.895) (xy 184.785 175.895))
+    (stroke (width 0) (type default))
+  )
   (wire (pts (xy 281.305 247.015) (xy 281.305 263.525))
     (stroke (width 0) (type default))
@@
     (stroke (width 0) (type default))
   )
-  (wire (pts (xy 184.785 175.895) (xy 224.155 175.895))
-    (stroke (width 0) (type default))
-  )
   (wire (pts (xy 513.715 182.88) (xy 527.05 182.88))
     (stroke (width 0) (type default))
@@
     (stroke (width 0) (type default))
   )
+  (wire (pts (xy 451.485 41.275) (xy 456.565 41.275))
+    (stroke (width 0) (type default))
+  )
   (bus (pts (xy 222.25 204.47) (xy 222.25 241.935))
     (stroke (width 0) (type default))
@@
     (stroke (width 0) (type default))
   )
+  (wire (pts (xy 454.025 18.415) (xy 454.025 26.035))
+    (stroke (width 0) (type default))
+  )
   (bus (pts (xy 67.31 54.61) (xy 67.31 57.15))
     (stroke (width 0) (type default))
@@
     (stroke (width 0) (type default))
   )
-  (wire (pts (xy 441.96 18.415) (xy 539.75 18.415))
-    (stroke (width 0) (type default))
-  )
   (wire (pts (xy 179.07 265.43) (xy 182.88 265.43))
     (stroke (width 0) (type default))
@@
     (stroke (width 0) (type default))
   )
+  (wire (pts (xy 454.025 18.415) (xy 539.75 18.415))
+    (stroke (width 0) (type default))
+  )
   (bus (pts (xy 104.14 207.01) (xy 104.14 209.55))
     (stroke (width 0) (type default))
@@
     )
   )
-  (symbol (lib_id "power:GND") (at 327.025 374.65 0) (unit 1)
-    (in_bom yes) (on_board yes) (dnp no) (fields_autoplaced)
-    (property "Reference" "#PWR096" (at 327.025 381 0)
-      (effects (font (size 1.27 1.27)) hide)
-    )
-    (property "Value" "GND" (at 327.025 378.7831 0)
-      (effects (font (size 1.27 1.27)))
-    )
-    (property "Footprint" "" (at 327.025 374.65 0)
-      (effects (font (size 1.27 1.27)) hide)
-    )
-    (property "Datasheet" "" (at 327.025 374.65 0)
-      (effects (font (size 1.27 1.27)) hide)
-    )
-    (pin "1")
-    (instances
-      (project "ALU"
-        (path "/b26dce39-0c19-4808-8ddd-74847f21ad13"
-          (reference "#PWR096") (unit 1)
-        )
-      )
-    )
-  )
   (symbol (lib_id "Device:C") (at 478.155 259.715 90) (unit 1)
     (in_bom yes) (on_board yes) (dnp no)
@@
     )
   )
-  (symbol (lib_id "74xx:74LS32") (at 334.645 358.14 0) (unit 3)
-    (in_bom yes) (on_board yes) (dnp no) (fields_autoplaced)
-    (property "Reference" "U39" (at 334.645 350.1857 0)
+  (symbol (lib_id "74xx:74LS32") (at 216.535 173.355 0) (mirror y) (unit 3)
+    (in_bom yes) (on_board yes) (dnp no)
+    (property "Reference" "U39" (at 216.535 165.4007 0)
       (effects (font (size 1.27 1.27)))
     )
-    (property "Value" "74LS32" (at 334.645 352.6099 0)
+    (property "Value" "74LS32" (at 216.535 167.8249 0)
       (effects (font (size 1.27 1.27)))
     )
-    (property "Footprint" "Package_DIP:DIP-14_W7.62mm" (at 334.645 358.14 0)
+    (property "Footprint" "Package_DIP:DIP-14_W7.62mm" (at 216.535 173.355 0)
       (effects (font (size 1.27 1.27)) hide)
     )
-    (property "Datasheet" "http://www.ti.com/lit/gpn/sn74LS32" (at 334.645 358.14 0)
+    (property "Datasheet" "http://www.ti.com/lit/gpn/sn74LS32" (at 216.535 173.355 0)
       (effects (font (size 1.27 1.27)) hide)
     )
@@
     )
   )
-  (symbol (lib_id "power:GND") (at 327.025 360.68 0) (unit 1)
-    (in_bom yes) (on_board yes) (dnp no) (fields_autoplaced)
-    (property "Reference" "#PWR094" (at 327.025 367.03 0)
-      (effects (font (size 1.27 1.27)) hide)
-    )
-    (property "Value" "GND" (at 327.025 364.8131 0)
-      (effects (font (size 1.27 1.27)))
-    )
-    (property "Footprint" "" (at 327.025 360.68 0)
-      (effects (font (size 1.27 1.27)) hide)
-    )
-    (property "Datasheet" "" (at 327.025 360.68 0)
-      (effects (font (size 1.27 1.27)) hide)
-    )
-    (pin "1")
-    (instances
-      (project "ALU"
-        (path "/b26dce39-0c19-4808-8ddd-74847f21ad13"
-          (reference "#PWR094") (unit 1)
-        )
-      )
-    )
-  )
   (symbol (lib_id "power:GND") (at 457.835 259.715 0) (unit 1)
     (in_bom yes) (on_board yes) (dnp no) (fields_autoplaced)
@@
     )
   )
-  (symbol (lib_id "74xx:74LS32") (at 334.645 372.11 0) (unit 4)
+  (symbol (lib_id "74xx:74LS32") (at 454.025 33.655 90) (unit 4)
     (in_bom yes) (on_board yes) (dnp no) (fields_autoplaced)
-    (property "Reference" "U39" (at 334.645 364.1557 0)
-      (effects (font (size 1.27 1.27)))
+    (property "Reference" "U39" (at 458.597 32.4429 90)
+      (effects (font (size 1.27 1.27)) (justify right))
     )
-    (property "Value" "74LS32" (at 334.645 366.5799 0)
-      (effects (font (size 1.27 1.27)))
+    (property "Value" "74LS32" (at 458.597 34.8671 90)
+      (effects (font (size 1.27 1.27)) (justify right))
     )
-    (property "Footprint" "Package_DIP:DIP-14_W7.62mm" (at 334.645 372.11 0)
+    (property "Footprint" "Package_DIP:DIP-14_W7.62mm" (at 454.025 33.655 0)
       (effects (font (size 1.27 1.27)) hide)
     )
-    (property "Datasheet" "http://www.ti.com/lit/gpn/sn74LS32" (at 334.645 372.11 0)
+    (property "Datasheet" "http://www.ti.com/lit/gpn/sn74LS32" (at 454.025 33.655 0)
       (effects (font (size 1.27 1.27)) hide)
     )
