File: kicad/ALU/ALU.kicad_pcb (KiCad board)
At the start: 2 copper layers, 206.4 x 137.5 mm, 84 parts, among them J1 Control Connector, J2 Data Connector, U1 74LS377, U10 74LS253, U11 74LS253, U12 74LS253, U13 74LS253, U14 74LS253, U15 74LS253, U16 74LS253, U17 74F382, U18 74F382, U19 74F382, U2 74LS377, U20 74F382, U21 74F382, U22 74LS283, U23 74LS283, U24 74LS283, U25 74LS283, U26 74LS283, U27 74LS244, U28 74LS244, U29 74LS244, U3 74LS377, U30 74LS86, U31 74LS08, U32 74LS32, U33 74LS04, U34 74LS253, U35 74LS27, U36 74LS27, U37 74LS11, U38 74LS257, U39 74LS32, U4 74LS377, U5 74LS377, U6 74LS377, U7 74LS253, U8 74LS253, U9 74LS253

Commit message: Start work on backplane and fix connectors
Parts:
- removed UX0: DIP-16_W7.62mm, Package_DIP:DIP-16_W7.62mm
- J1: value Control Connector -> Signal Connector
Connections:
- J1 pad b1: (no net) -> +5V
- J1 pad b10: (no net) -> /BUS_SELECT1
- J1 pad b11: (no net) -> /BUS_SELECT2
- J1 pad b12: (no net) -> /*SELECT_AC
- J1 pad b13: (no net) -> /*SELECT_STEP
- J1 pad b14: (no net) -> /*SELECT_MQ
- J1 pad b15: (no net) -> /*SELECT_CROSS
- J1 pad b16: (no net) -> /*SELECT_ALU
- J1 pad b17: (no net) -> /*SELECT_CORE
- J1 pad b18: (no net) -> /*SELECT_SWR
- J1 pad b19: (no net) -> /*SELECT_EXTRN
- J1 pad b2: (no net) -> unconnected-(J1-Pin_b2-Padb2)
- J1 pad b20: (no net) -> /IOT_PULSE
- J1 pad b21: (no net) -> /DRQ_GRANT
- J1 pad b22: (no net) -> /REQ_ADDR
- J1 pad b23: (no net) -> /JMP_I_DETECT
- J1 pad b24: (no net) -> /INT_DETECT
- J1 pad b25: (no net) -> /READ_IN_PULSE
- J1 pad b26: (no net) -> /HALT
- J1 pad b27: (no net) -> /ADDR_MODE0
- J1 pad b28: (no net) -> /ADDR_MODE1
- J1 pad b29: (no net) -> /CTL_CONST
- J1 pad b3: (no net) -> /STEP_ZERO
- J1 pad b30: (no net) -> /EXTRA0
- J1 pad b31: (no net) -> unconnected-(J1-Pin_b31-Padb31)
- J1 pad b32: (no net) -> GND
- J1 pad b4: (no net) -> /FLAG_ZERO
- J1 pad b5: (no net) -> /OB17
- J1 pad b6: (no net) -> /FLAG_LINK
- J1 pad b7: (no net) -> /FLAG_LINK_INIT
- J1 pad b8: (no net) -> /FLAG_AC_SIGN
- J1 pad b9: (no net) -> /BUS_SELECT0
- J2 pad b1: (no net) -> +5V
- J2 pad b10: (no net) -> /A7
- J2 pad b11: (no net) -> /A8
- J2 pad b12: (no net) -> /A9
- J2 pad b13: (no net) -> /A10
- J2 pad b14: (no net) -> /A11
- J2 pad b15: (no net) -> /A12
- J2 pad b16: (no net) -> /A13
- J2 pad b17: (no net) -> /A14
- J2 pad b18: (no net) -> /SC0
- J2 pad b19: (no net) -> /SC1
- J2 pad b2: (no net) -> unconnected-(J2-Pin_b2-Padb2)
- J2 pad b20: (no net) -> /SC2
- J2 pad b21: (no net) -> /SC3
- J2 pad b22: (no net) -> /SC4
- J2 pad b23: (no net) -> /SC5
- J2 pad b24: (no net) -> /EXTRA2
- J2 pad b25: (no net) -> /EXTRA4
- J2 pad b26: (no net) -> /EXTRA6
- J2 pad b27: (no net) -> /NEXT_BANK1
- J2 pad b28: (no net) -> /MA_AUTO_INX
- J2 pad b29: (no net) -> /FP1
- J2 pad b3: (no net) -> /A0
- J2 pad b30: (no net) -> /FP3
- J2 pad b31: (no net) -> unconnected-(J2-Pin_b31-Padb31)
- J2 pad b32: (no net) -> GND
- J2 pad b4: (no net) -> /A1
- J2 pad b5: (no net) -> /A2
- J2 pad b6: (no net) -> /A3
- J2 pad b7: (no net) -> /A4
- J2 pad b8: (no net) -> /A5
- J2 pad b9: (no net) -> /A6
- U10 pad 1: /*SHIFT_OUT -> Net-(U10-OEa)
- U10 pad 15: /*SHIFT_OUT -> Net-(U10-OEa)
- U11 pad 1: /*SHIFT_OUT -> Net-(U10-OEa)
- U11 pad 15: /*SHIFT_OUT -> Net-(U10-OEa)
- U39 pad 10: GND -> /*SHIFT_OUT
- U39 pad 11: unconnected-(U39-Pad11) -> /FLAG_LINK
- U39 pad 12: GND -> /FLAG_LINK
- U39 pad 13: GND -> /FLAG_LINK
- U39 pad 8: unconnected-(U39-Pad8) -> Net-(U10-OEa)
- U39 pad 9: GND -> /*SHIFT_OUT
- U7 pad 1: /*SHIFT_OUT -> Net-(U10-OEa)
- U7 pad 15: /*SHIFT_OUT -> Net-(U10-OEa)
- U8 pad 1: /*SHIFT_OUT -> Net-(U10-OEa)
- U8 pad 15: /*SHIFT_OUT -> Net-(U10-OEa)
- U9 pad 1: /*SHIFT_OUT -> Net-(U10-OEa)
- U9 pad 15: /*SHIFT_OUT -> Net-(U10-OEa)

Commit message: Continue work on routing
Other:
- board text added: "Gavin Tersteeg, 2026"
- board text added: "JLCJLCJLCJLC"
Changed lines of the file:
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@@
   (gr_rect (start 35.56 17.78) (end 241.935 155.321)
     (stroke (width 0.1) (type default)) (fill none) (layer "Edge.Cuts"))
+  (gr_text "Gavin Tersteeg, 2026\n" (at 52.705 19.685) (layer "B.SilkS")
+    (effects (font (size 1 1) (thickness 0.15)) (justify left bottom mirror))
+  )
+  (gr_text "JLCJLCJLCJLC" (at 46.99 21.59) (layer "B.SilkS")
+    (effects (font (size 1 1) (thickness 0.15)) (justify left bottom mirror))
+  )
   (gr_text "RDP-9A-ALU-0" (at 36.195 20.955) (layer "F.SilkS")
     (effects (font (size 2 2) (thickness 0.4) bold) (justify left bottom))

Commit message: The great PCB layout-athon
Parts:
- J1: value Signal Connector -> Control Connector
Connections:
- net /DRQ_GRANT renamed /*DRQ_GRANT
- net /INT_DETECT renamed /*INT_DETECT
- net /IOT_PULSE renamed /*IOT_PULSE
- net /JMP_I_DETECT renamed /*JMP_I_DETECT
- net /READ_IN_PULSE renamed /*READ_IN_PULSE

Commit message: Gerber creation marathon
Routing:
- net GND: track 0.00 -> 1489.4 mm
- net +5V: track 0.00 -> 1132.8 mm
- net /OB17: track 0.00 -> 506.4 mm, vias 0 -> 1
- net /FLAG_LINK: track 0.00 -> 488.0 mm, vias 0 -> 4
- net /ALUO1: track 0.00 -> 418.1 mm
- net /ALUO0: track 0.00 -> 417.7 mm
- net /OB0: track 0.00 -> 411.2 mm
- net /OB1: track 0.00 -> 366.6 mm
- net /ALU_SHIFT: track 0.00 -> 332.5 mm
- net /OB14: track 0.00 -> 329.8 mm, vias 0 -> 4
- net /LINKS0: track 0.00 -> 326.2 mm
- net /OB3: track 0.00 -> 311.0 mm, vias 0 -> 3
- net /OB10: track 0.00 -> 308.2 mm, vias 0 -> 2
- net Net-(U33-Pad12): track 0.00 -> 300.7 mm
- net /OB2: track 0.00 -> 299.4 mm
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- added copper zone on B.Cu, net GND
- added copper zone on F.Cu, net GND
Other:
- board text removed: "JLCJLCJLCJLC"
