File: kicad/Control/Control.kicad_sch (KiCad schematic)
At the start: 65 parts, among them J3 Control Connector, J4 Data Connector, U1 27C64, U10 74LS377, U11 74LS253, U12 74LS253, U13 74LS253, U14 74LS253, U15 74LS253, U16 74LS253, U17 74LS253, U18 74LS257, U19 74LS377, U2 27C64, U20 74LS377, U21 74LS377, U22 74LS138, U23 74LS32, U24 74LS08, U25 74LS86, U26 74LS74, U3 27C64, U4 27C64, U5 27C64, U6 74LS273, U7 74LS377, U8 74LS377, U9 74LS377

Commit message: Continue work on register file
Parts:
- added R11: 4.7K, symbol Device:R
Connections:
- net *INT_REQ: now also U23.9; no longer U17.12 (I2b)
- net *PI_ENABLE: now also U23.10
- net +5V: now also R11.2
- net GND: no longer U23.10, U23.9, U25.4, U25.5
- net at U23.8: now also U25.4
- net INT_PEND: now reaches U25.6
- net INT_PEND: now also U17.12 (I2b)
- new net: R11.1, U25.5
- no-connect marks 57 -> 54
Other:
- moved on the sheet: U23C, U25B
Changed lines of the file:
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@@
   (junction (at 379.095 299.085) (diameter 0) (color 0 0 0 0)
   )
-  (junction (at 57.15 321.945) (diameter 0) (color 0 0 0 0)
-  )
   (junction (at 191.135 27.305) (diameter 0) (color 0 0 0 0)
   )
@@
   (junction (at 57.15 340.995) (diameter 0) (color 0 0 0 0)
   )
-  (junction (at 31.75 321.945) (diameter 0) (color 0 0 0 0)
-  )
   (junction (at 259.715 88.9) (diameter 0) (color 0 0 0 0)
   )
@@
   (no_connect (at 458.47 294.005))
   (no_connect (at 497.84 243.205))
-  (no_connect (at 72.39 319.405))
   (no_connect (at 497.84 281.305))
   (no_connect (at 419.735 358.14))
@@
   (no_connect (at 497.84 255.905))
   (no_connect (at 458.47 288.925))
-  (no_connect (at 458.47 56.515))
   (no_connect (at 497.84 288.925))
   (no_connect (at 471.805 127.635))
@@
   (no_connect (at 497.84 296.545))
   (no_connect (at 484.505 311.785))
-  (no_connect (at 46.99 319.405))
   (no_connect (at 497.84 258.445))
   (no_connect (at 458.47 301.625))
@@
     (stroke (width 0) (type default))
   )
-  (wire (pts (xy 389.255 71.755) (xy 389.255 280.035))
-    (stroke (width 0) (type default))
-  )
   (wire (pts (xy 318.135 308.61) (xy 310.515 308.61))
     (stroke (width 0) (type default))
@@
     (stroke (width 0) (type default))
   )
-  (wire (pts (xy 273.685 326.39) (xy 266.065 326.39))
+  (wire (pts (xy 389.255 118.745) (xy 389.255 280.035))
     (stroke (width 0) (type default))
   )
-  (wire (pts (xy 57.15 316.865) (xy 57.15 321.945))
+  (wire (pts (xy 273.685 326.39) (xy 266.065 326.39))
     (stroke (width 0) (type default))
   )
@@
     (stroke (width 0) (type default))
   )
+  (wire (pts (xy 387.985 56.515) (xy 387.985 86.995))
+    (stroke (width 0) (type default))
+  )
   (wire (pts (xy 445.135 350.52) (xy 450.215 350.52))
     (stroke (width 0) (type default))
@@
     (stroke (width 0) (type default))
   )
-  (wire (pts (xy 458.47 56.515) (xy 471.805 56.515))
+  (wire (pts (xy 387.985 56.515) (xy 471.805 56.515))
     (stroke (width 0) (type default))
   )
@@
     (stroke (width 0) (type default))
   )
+  (wire (pts (xy 375.285 86.995) (xy 375.285 88.265))
+    (stroke (width 0) (type default))
+  )
   (wire (pts (xy 445.135 306.705) (xy 450.215 306.705))
     (stroke (width 0) (type default))
@@
     (stroke (width 0) (type default))
   )
-  (wire (pts (xy 31.75 316.865) (xy 31.75 321.945))
-    (stroke (width 0) (type default))
-  )
   (wire (pts (xy 75.565 114.3) (xy 79.375 114.3))
     (stroke (width 0) (type default))
@@
     (stroke (width 0) (type default))
   )
+  (wire (pts (xy 387.985 86.995) (xy 375.285 86.995))
+    (stroke (width 0) (type default))
+  )
   (wire (pts (xy 77.47 223.52) (xy 69.215 223.52))
     (stroke (width 0) (type default))
@@
     (stroke (width 0) (type default))
   )
+  (wire (pts (xy 375.285 118.745) (xy 389.255 118.745))
+    (stroke (width 0) (type default))
+  )
   (bus (pts (xy 225.425 60.96) (xy 225.425 106.68))
     (stroke (width 0) (type default))
@@
     (stroke (width 0) (type default))
   )
+  (wire (pts (xy 380.365 88.265) (xy 389.255 88.265))
+    (stroke (width 0) (type default))
+  )
   (wire (pts (xy 484.505 258.445) (xy 497.84 258.445))
     (stroke (width 0) (type default))
@@
     (stroke (width 0) (type default))
   )
+  (wire (pts (xy 389.255 71.755) (xy 389.255 88.265))
+    (stroke (width 0) (type default))
+  )
   (wire (pts (xy 484.505 122.555) (xy 500.38 122.555))
     (stroke (width 0) (type default))
@@
     (effects (font (size 1.27 1.27)) (justify left bottom))
   )
-  (label "*INT_REQ" (at 310.515 323.85 0) (fields_autoplaced)
+  (label "INT_PEND" (at 310.515 323.85 0) (fields_autoplaced)
     (effects (font (size 1.27 1.27)) (justify left bottom))
   )
@@
     (effects (font (size 1.27 1.27)) (justify left bottom))
   )
+  (label "INT_PEND" (at 389.255 118.745 180) (fields_autoplaced)
+    (effects (font (size 1.27 1.27)) (justify right bottom))
+  )
   (label "UD[0..7]" (at 225.425 90.17 90) (fields_autoplaced)
     (effects (font (size 1.27 1.27)) (justify left bottom))
@@
     )
   )
+  (symbol (lib_id "power:+5V") (at 365.125 103.505 0) (mirror y) (unit 1)
+    (in_bom yes) (on_board yes) (dnp no) (fields_autoplaced)
+    (property "Reference" "#PWR085" (at 365.125 107.315 0)
+      (effects (font (size 1.27 1.27)) hide)
+    )
+    (property "Value" "+5V" (at 365.125 99.3719 0)
+      (effects (font (size 1.27 1.27)))
+    )
+    (property "Footprint" "" (at 365.125 103.505 0)
+      (effects (font (size 1.27 1.27)) hide)
+    )
+    (property "Datasheet" "" (at 365.125 103.505 0)
+      (effects (font (size 1.27 1.27)) hide)
+    )
+    (pin "1")
+    (instances
+      (project "Control"
+        (path "/9aceca4c-796d-4c9d-8044-fc5cfdda262d"
+          (reference "#PWR085") (unit 1)
+        )
+      )
+    )
+  )
   (symbol (lib_id "power:GND") (at 448.31 353.06 0) (unit 1)
     (in_bom yes) (on_board yes) (dnp no) (fields_autoplaced)
@@
     )
   )
-  (symbol (lib_id "74xx:74LS32") (at 39.37 319.405 0) (unit 3)
+  (symbol (lib_id "74xx:74LS32") (at 377.825 95.885 270) (unit 3)
     (in_bom yes) (on_board yes) (dnp no) (fields_autoplaced)
-    (property "Reference" "U23" (at 39.37 311.4507 0)
+    (property "Reference" "U23" (at 385.7793 95.885 0)
       (effects (font (size 1.27 1.27)))
     )
-    (property "Value" "74LS32" (at 39.37 313.8749 0)
+    (property "Value" "74LS32" (at 383.3551 95.885 0)
       (effects (font (size 1.27 1.27)))
     )
-    (property "Footprint" "" (at 39.37 319.405 0)
+    (property "Footprint" "" (at 377.825 95.885 0)
       (effects (font (size 1.27 1.27)) hide)
     )
-    (property "Datasheet" "http://www.ti.com/lit/gpn/sn74LS32" (at 39.37 319.405 0)
+    (property "Datasheet" "http://www.ti.com/lit/gpn/sn74LS32" (at 377.825 95.885 0)
       (effects (font (size 1.27 1.27)) hide)
     )
@@
     )
   )
-  (symbol (lib_id "power:GND") (at 31.75 321.945 0) (unit 1)
-    (in_bom yes) (on_board yes) (dnp no) (fields_autoplaced)
-    (property "Reference" "#PWR080" (at 31.75 328.295 0)
-      (effects (font (size 1.27 1.27)) hide)
-    )
-    (property "Value" "GND" (at 31.75 326.0781 0)
-      (effects (font (size 1.27 1.27)))
-    )
-    (property "Footprint" "" (at 31.75 321.945 0)
-      (effects (font (size 1.27 1.27)) hide)
-    )
-    (property "Datasheet" "" (at 31.75 321.945 0)
-      (effects (font (size 1.27 1.27)) hide)
-    )
-    (pin "1")
-    (instances
-      (project "Control"
-        (path "/9aceca4c-796d-4c9d-8044-fc5cfdda262d"
-          (reference "#PWR080") (unit 1)
-        )
-      )
-    )
-  )
   (symbol (lib_id "power:GND") (at 484.505 130.175 0) (unit 1)
     (in_bom yes) (on_board yes) (dnp no) (fields_autoplaced)
@@
     )
   )
+  (symbol (lib_id "Device:R") (at 368.935 103.505 270) (mirror x) (unit 1)
+    (in_bom yes) (on_board yes) (dnp no)
+    (property "Reference" "R11" (at 368.935 100.965 90)
+      (effects (font (size 1.27 1.27)))
+    )
+    (property "Value" "4.7K" (at 368.935 103.505 90)
+      (effects (font (size 1.27 1.27)))
+    )
+    (property "Footprint" "" (at 368.935 105.283 90)
+      (effects (font (size 1.27 1.27)) hide)
+    )
+    (property "Datasheet" "~" (at 368.935 103.505 0)
+      (effects (font (size 1.27 1.27)) hide)
+    )
+    (pin "1")
+    (pin "2")
+    (instances
+      (project "Control"
+        (path "/9aceca4c-796d-4c9d-8044-fc5cfdda262d"
+          (reference "R11") (unit 1)
+        )
+      )
+      (project "ALU"
+        (path "/b26dce39-0c19-4808-8ddd-74847f21ad13"
+          (reference "R1") (unit 1)
+        )
+      )
+    )
+  )
   (symbol (lib_id "power:+5V") (at 468.63 318.135 0) (unit 1)
     (in_bom yes) (on_board yes) (dnp no) (fields_autoplaced)
@@
     )
   )
-  (symbol (lib_id "74xx:74LS86") (at 64.77 319.405 0) (unit 2)
+  (symbol (lib_id "74xx:74LS86") (at 375.285 111.125 270) (unit 2)
     (in_bom yes) (on_board yes) (dnp no) (fields_autoplaced)
-    (property "Reference" "U25" (at 64.4652 311.4507 0)
+    (property "Reference" "U25" (at 383.2393 110.8202 0)
       (effects (font (size 1.27 1.27)))
     )
-    (property "Value" "74LS86" (at 64.4652 313.8749 0)
+    (property "Value" "74LS86" (at 380.8151 110.8202 0)
       (effects (font (size 1.27 1.27)))
     )
-    (property "Footprint" "" (at 64.77 319.405 0)
+    (property "Footprint" "" (at 375.285 111.125 0)
       (effects (font (size 1.27 1.27)) hide)
     )
-    (property "Datasheet" "74xx/74ls86.pdf" (at 64.77 319.405 0)
+    (property "Datasheet" "74xx/74ls86.pdf" (at 375.285 111.125 0)
       (effects (font (size 1.27 1.27)) hide)
     )
@@
         )
       )
-    )
-  )
-  (symbol (lib_id "power:GND") (at 57.15 321.945 0) (unit 1)
-    (in_bom yes) (on_board yes) (dnp no) (fields_autoplaced)
-    (property "Reference" "#PWR085" (at 57.15 328.295 0)
-      (effects (font (size 1.27 1.27)) hide)
-    )
-    (property "Value" "GND" (at 57.15 326.0781 0)
-      (effects (font (size 1.27 1.27)))
-    )
-    (property "Footprint" "" (at 57.15 321.945 0)
-      (effects (font (size 1.27 1.27)) hide)
-    )
-    (property "Datasheet" "" (at 57.15 321.945 0)
-      (effects (font (size 1.27 1.27)) hide)
-    )
-    (pin "1")
-    (instances
-      (project "Control"
-        (path "/9aceca4c-796d-4c9d-8044-fc5cfdda262d"
-          (reference "#PWR085") (unit 1)
-        )
-      )
