File: kicad/Control/Control.kicad_pcb (KiCad board)
At the start: 2 copper layers, 206.4 x 137.5 mm, 67 parts, among them J1 Control Connector, J2 Data Connector, J3 State Debug, U1 27C64, U10 74LS377, U11 74LS253, U12 74LS253, U13 74LS253, U14 74LS253, U15 74LS253, U16 74LS253, U17 74LS253, U18 74LS257, U19 74LS377, U2 27C64, U20 74LS377, U21 74LS377, U22 74LS138, U23 74LS32, U24 74LS08, U25 74LS86, U26 74LS74, U3 27C64, U4 27C64, U5 27C64, U6 74LS273, U7 74LS377, U8 74LS377, U9 74LS377

Commit message: Gerber creation marathon
Routing:
- net GND: track 0.00 -> 1289.8 mm
- net +5V: track 0.00 -> 883.6 mm
- net /ST12: track 0.00 -> 446.3 mm
- net /ST11: track 0.00 -> 401.0 mm
- net /CLK: track 0.00 -> 387.0 mm, vias 0 -> 1
- net /*RESET: track 0.00 -> 371.5 mm
- net /STEP4: track 0.00 -> 287.0 mm, vias 0 -> 1
- net /STEP5: track 0.00 -> 280.6 mm, vias 0 -> 1
- net /*LATCH_IR: track 0.00 -> 275.2 mm, vias 0 -> 1
- net /STEP2: track 0.00 -> 243.5 mm, vias 0 -> 1
- net /STEP1: track 0.00 -> 240.7 mm
- net /ST0: track 0.00 -> 238.5 mm
- net /STEP3: track 0.00 -> 229.1 mm, vias 0 -> 1
- net /ALU_ONES: track 0.00 -> 222.8 mm
- net /ST7: track 0.00 -> 220.4 mm
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- added copper zone on B.Cu, net GND
- added copper zone on F.Cu, net GND
Other:
- board text removed: "JLCJLCJLCJLC"
