File: kicad/Registers/Registers.kicad_sch (KiCad schematic)
At the start: 26 parts, among them J1 Control Connector, J2 Data Connector, U1 74LS253, U10 74LS244, U11 74LS244, U12 74LS244, U13 74LS377, U14 74LS377, U15 74LS377, U16 74LS377, U17 74LS377, U18 74LS377, U19 74LS169, U2 74LS253, U20 74LS169, U21 74LS283, U22 74LS283, U23 74LS283, U24 74LS283, U3 74LS253, U4 74LS253, U5 74LS253, U6 74LS253, U7 74LS253, U8 74LS253, U9 74LS253

Commit message: Continue work on register file
Parts:
- added U25: 74LS32, symbol 74xx:74LS32
- added U26: 74LS02, symbol 74xx:74LS02
Connections:
- net *MEMM_ENABLE: now also U26.5, U26.6
- net *PROT_ENABLE: now also U26.8, U26.9
- net A13: now also U7.13 (I3b)
- net A14: now also U8.3 (I3a)
- net AC10: now also U6.6 (I0a)
- net AC11: now also U6.10 (I0b)
- net AC12: now also U7.6 (I0a)
- net AC13: now also U7.10 (I0b)
- net AC14: now also U8.6 (I0a)
- net AC15: now also U8.10 (I0b)
- net AC16: now also U9.6 (I0a)
- net AC2: now also U2.6 (I0a)
- net AC3: now also U2.10 (I0b)
- net AC4: now also U3.6 (I0a)
- net AC5: now also U3.10 (I0b)
- net AC6: now also U4.6 (I0a)
- net AC7: now also U4.10 (I0b)
- net AC8: now also U5.6 (I0a)
- net AC9: now also U5.10 (I0b)
- net CB10: now also U6.3 (I3a)
- net CB11: now also U6.13 (I3b)
- net CB12: now also U7.3 (I3a)
- net CB2: now also U2.3 (I3a)
- net CB3: now also U2.13 (I3b)
- net CB4: now also U3.3 (I3a)
- net CB5: now also U3.13 (I3b)
- net CB6: now also U4.3 (I3a)
- net CB7: now also U4.13 (I3b)
- net CB8: now also U5.3 (I3a)
- net CB9: now also U5.13 (I3b)
- net FLAG_LINK: now also U9.13 (I3b)
- net GND: now also U1.1 (OEa), U1.15 (OEb), U2.1 (OEa), U2.15 (OEb), U3.1 (OEa), U3.15 (OEb), U4.1 (OEa), U4.11 (I1b), U4.15 (OEb), U4.5 (I1a), U5.1 (OEa), U5.11 (I1b), U5.15 (OEb), U5.5 (I1a), U6.1 (OEa), U6.11 (I1b), U6.15 (OEb), U6.5 (I1a), U7.1 (OEa), U7.11 (I1b), U7.15 (OEb), U7.5 (I1a), U8.1 (OEa), U8.11 (I1b), U8.15 (OEb), U8.5 (I1a), U9.1 (OEa), U9.11 (I1b), U9.15 (OEb), U9.5 (I1a)
- net MQ10: now also U6.4 (I2a)
- net MQ11: now also U6.12 (I2b)
- net MQ12: now also U7.4 (I2a)
- net MQ13: now also U7.12 (I2b)
- net MQ14: now also U8.4 (I2a)
- net MQ15: now also U8.12 (I2b)
- net MQ16: now also U9.4 (I2a)
- net MQ17: now also U9.12 (I2b)
- net MQ2: now also U2.4 (I2a)
- net MQ3: now also U2.12 (I2b)
- net MQ4: now also U3.4 (I2a)
- net MQ5: now also U3.12 (I2b)
- net MQ6: now also U4.4 (I2a)
- net MQ7: now also U4.12 (I2b)
- net MQ8: now also U5.4 (I2a)
- net MQ9: now also U5.12 (I2b)
- net SC0: now also U25.1
- net SC1: now also U25.2
- net SC2: now also U2.5 (I1a), U25.4
- net SC3: now also U2.11 (I1b), U25.5
- net SC4: now also U3.5 (I1a), U25.9
- net SC5: now also U3.11 (I1b), U25.10
- net STEP_ZERO: now also U26.1
- net at U9.3 (I3a): now also U26.4
- net at U8.13 (I3b): now also U26.10
- new net: U25.11, U26.2
- new net: U25.8, U26.3
- new net: U25.12, U25.3
- new net: U25.13, U25.6
- no-connect marks 108 -> 100
Other:
- moved on the sheet: U2, U3, U4, U5, U6, U7, U8, U9
