File: kicad/Registers/Registers.kicad_sch (KiCad schematic)
At the start: 28 parts, among them J1 Control Connector, J2 Data Connector, U1 74LS253, U10 74LS244, U11 74LS244, U12 74LS244, U13 74LS377, U14 74LS377, U15 74LS377, U16 74LS377, U17 74LS377, U18 74LS377, U19 74LS169, U2 74LS253, U20 74LS169, U21 74LS283, U22 74LS283, U23 74LS283, U24 74LS283, U25 74LS32, U26 74LS02, U3 74LS253, U4 74LS253, U5 74LS253, U6 74LS253, U7 74LS253, U8 74LS253, U9 74LS253

Commit message: Continue work on register file
Parts:
- added R1, R2: 4.7K, symbol Device:R
- added U27: 74LS32, symbol 74xx:74LS32
Connections:
- net *LATCH_AC: now also U13.1 (~{E}), U14.1 (~{E}), U15.1 (~{E})
- net *LATCH_MQ: now also U16.1 (~{E}), U17.1 (~{E}), U18.1 (~{E})
- net *LATCH_STEP: now also U19.7 (~{CEP}), U20.7 (~{CEP}), U27.1
- net +5V: now also U25.14 (VCC), U26.14 (VCC), R1.2, R2.2, U27.14 (VCC)
- net BUS_SELECT0: now also U1.14 (A0), U2.14 (A0), U3.14 (A0), U4.14 (A0), U5.14 (A0), U6.14 (A0), U7.14 (A0), U8.14 (A0), U9.14 (A0)
- net BUS_SELECT1: now also U1.2 (A1), U2.2 (A1), U3.2 (A1), U4.2 (A1), U5.2 (A1), U6.2 (A1), U7.2 (A1), U8.2 (A1), U9.2 (A1)
- net BUS_SELECT2: now also U1.1 (OEa), U1.15 (OEb), U2.1 (OEa), U2.15 (OEb), U3.1 (OEa), U3.15 (OEb), U4.1 (OEa), U4.15 (OEb), U5.1 (OEa), U5.15 (OEb), U6.1 (OEa), U6.15 (OEb), U7.1 (OEa), U7.15 (OEb), U8.1 (OEa), U8.15 (OEb), U9.1 (OEa), U9.15 (OEb)
- net CTL_CONST: now also U21.7 (C0), U27.2
- net GND: now also U25.7 (GND), U26.11, U26.12, U26.7 (GND), U27.10, U27.12, U27.13, U27.4, U27.5, U27.7 (GND), U27.9; no longer U1.1 (OEa), U1.15 (OEb), U2.1 (OEa), U2.15 (OEb), U3.1 (OEa), U3.15 (OEb), U4.1 (OEa), U4.15 (OEb), U5.1 (OEa), U5.15 (OEb), U6.1 (OEa), U6.15 (OEb), U7.1 (OEa), U7.15 (OEb), U8.1 (OEa), U8.15 (OEb), U9.1 (OEa), U9.15 (OEb)
- net at U20.1 (U/~{D}): now also R2.1
- net at U20.9 (~{PE}): now also U19.9 (~{PE}), U27.3
- net at U19.1 (U/~{D}): now also R1.1
- no-connect marks 100 -> 98
Other:
- moved on the sheet: U25E, U26D, U26E

Commit message: Finish register file
Parts:
- added C1, C10, C11, C12, C13, C14, C15, C16, C17, C18, C19, C2, C20, C21, C22, C23, C24, C25, C26, C27, C3, C4, C5, C6, C7, C8, C9: 0.1uF, symbol Device:C
- added C20: 100 uF, Capacitor_THT:CP_Radial_D6.3mm_P2.50mm, symbol Device:C_Polarized
Connections:
- net +5V: now also C1.1, C10.1, C11.1, C12.1, C13.1, C14.1, C15.1, C16.1, C17.1, C18.1, C19.1, C2.1, C20.1, C20.1, C21.1, C22.1, C23.1, C24.1, C25.1, C26.1, C27.1, C3.1, C4.1, C5.1, C6.1, C7.1, C8.1, C9.1
- net GND: now also C1.2, C10.2, C11.2, C12.2, C13.2, C14.2, C15.2, C16.2, C17.2, C18.2, C19.2, C2.2, C20.2, C20.2, C21.2, C22.2, C23.2, C24.2, C25.2, C26.2, C27.2, C3.2, C4.2, C5.2, C6.2, C7.2, C8.2, C9.2
Other:
- note added: "AC"
- note added: "MQ"
- note added: "Register"
- note added: "SC"

Commit message: Start work on memory / addressing board
Connections:
- net WRITE_CORE renamed *WRITE_CORE
Changed lines of the file:
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@@
     (stroke (width 0) (type default))
   )
+  (bus_entry (at 549.91 211.455) (size -2.54 -2.54)
+    (stroke (width 0) (type default))
+  )
   (bus_entry (at 347.345 350.52) (size 2.54 2.54)
     (stroke (width 0) (type default))
@@
     (stroke (width 0) (type default))
   )
+  (bus_entry (at 549.91 219.075) (size -2.54 -2.54)
+    (stroke (width 0) (type default))
+  )
   (bus_entry (at 76.835 358.14) (size 2.54 2.54)
     (stroke (width 0) (type default))
@@
     (stroke (width 0) (type default))
   )
+  (bus_entry (at 549.91 213.995) (size -2.54 -2.54)
+    (stroke (width 0) (type default))
+  )
   (bus_entry (at 36.195 142.24) (size 2.54 2.54)
     (stroke (width 0) (type default))
@@
     (stroke (width 0) (type default))
   )
+  (bus_entry (at 549.91 208.915) (size -2.54 -2.54)
+    (stroke (width 0) (type default))
+  )
   (bus_entry (at 165.735 58.42) (size -2.54 -2.54)
     (stroke (width 0) (type default))
@@
     (stroke (width 0) (type default))
   )
+  (bus_entry (at 549.91 216.535) (size -2.54 -2.54)
+    (stroke (width 0) (type default))
+  )
   (bus_entry (at 299.085 340.36) (size 2.54 2.54)
     (stroke (width 0) (type default))
@@
     (stroke (width 0) (type default))
   )
+  (bus_entry (at 549.91 221.615) (size -2.54 -2.54)
+    (stroke (width 0) (type default))
+  )
   (bus_entry (at 76.835 210.82) (size -2.54 -2.54)
     (stroke (width 0) (type default))
@@
     (stroke (width 0) (type default))
   )
+  (bus (pts (xy 549.91 213.995) (xy 549.91 216.535))
+    (stroke (width 0) (type default))
+  )
   (wire (pts (xy 177.165 186.69) (xy 177.165 208.28))
     (stroke (width 0) (type default))
@@
     (stroke (width 0) (type default))
   )
+  (bus (pts (xy 549.91 257.81) (xy 121.285 257.81))
+    (stroke (width 0) (type default))
+  )
   (wire (pts (xy 394.335 353.06) (xy 399.415 353.06))
     (stroke (width 0) (type default))
@@
     (stroke (width 0) (type default))
   )
+  (wire (pts (xy 530.86 211.455) (xy 547.37 211.455))
+    (stroke (width 0) (type default))
+  )
   (wire (pts (xy 530.86 231.775) (xy 544.195 231.775))
     (stroke (width 0) (type default))
@@
     (stroke (width 0) (type default))
   )
+  (wire (pts (xy 530.86 216.535) (xy 547.37 216.535))
+    (stroke (width 0) (type default))
+  )
   (wire (pts (xy 38.735 149.86) (xy 43.815 149.86))
     (stroke (width 0) (type default))
@@
     (stroke (width 0) (type default))
   )
+  (wire (pts (xy 530.86 219.075) (xy 547.37 219.075))
+    (stroke (width 0) (type default))
+  )
   (wire (pts (xy 262.255 213.36) (xy 266.065 213.36))
     (stroke (width 0) (type default))
@@
     (stroke (width 0) (type default))
   )
+  (bus (pts (xy 549.91 211.455) (xy 549.91 213.995))
+    (stroke (width 0) (type default))
+  )
   (wire (pts (xy 127.635 335.28) (xy 132.715 335.28))
     (stroke (width 0) (type default))
@@
     (stroke (width 0) (type default))
   )
+  (wire (pts (xy 530.86 206.375) (xy 547.37 206.375))
+    (stroke (width 0) (type default))
+  )
   (wire (pts (xy 386.715 276.86) (xy 386.715 342.9))
     (stroke (width 0) (type default))
@@
     (stroke (width 0) (type default))
   )
+  (bus (pts (xy 549.91 208.915) (xy 549.91 211.455))
+    (stroke (width 0) (type default))
+  )
   (bus (pts (xy 304.165 181.61) (xy 259.715 181.61))
     (stroke (width 0) (type default))
@@
     (stroke (width 0) (type default))
   )
+  (wire (pts (xy 530.86 208.915) (xy 547.37 208.915))
+    (stroke (width 0) (type default))
+  )
   (wire (pts (xy 530.86 188.595) (xy 535.94 188.595))
     (stroke (width 0) (type default))
@@
     (stroke (width 0) (type default))
   )
+  (wire (pts (xy 530.86 213.995) (xy 547.37 213.995))
+    (stroke (width 0) (type default))
+  )
   (wire (pts (xy 125.095 358.14) (xy 132.715 358.14))
     (stroke (width 0) (type default))
@@
     (stroke (width 0) (type default))
   )
+  (bus (pts (xy 549.91 216.535) (xy 549.91 219.075))
+    (stroke (width 0) (type default))
+  )
   (wire (pts (xy 257.175 360.68) (xy 266.065 360.68))
     (stroke (width 0) (type default))
@@
     (stroke (width 0) (type default))
   )
+  (bus (pts (xy 549.91 219.075) (xy 549.91 221.615))
+    (stroke (width 0) (type default))
+  )
   (wire (pts (xy 31.115 365.76) (xy 31.115 401.32))
     (stroke (width 0) (type default))
@@
     (stroke (width 0) (type default))
   )
+  (bus (pts (xy 549.91 221.615) (xy 549.91 257.81))
+    (stroke (width 0) (type default))
+  )
   (rectangle (start 212.09 107.315) (end 345.44 172.72)
     (stroke (width 0) (type dash) (color 72 72 72 1))
@@
     (effects (font (size 1.27 1.27)) (justify right bottom))
   )
+  (label "SC0" (at 530.86 206.375 0)
+    (effects (font (size 1.27 1.27)) (justify left bottom))
+  )
   (label "D16" (at 424.815 335.28 0) (fields_autoplaced)
     (effects (font (size 1.27 1.27)) (justify left bottom))
@@
     (effects (font (size 1.27 1.27)) (justify right bottom))
   )
-  (label "SC0" (at 530.86 206.375 0) (fields_autoplaced)
-    (effects (font (size 1.27 1.27)) (justify left bottom))
-  )
   (label "SC0" (at 43.815 337.82 180) (fields_autoplaced)
     (effects (font (size 1.27 1.27)) (justify right bottom))
@@
     (effects (font (size 1.27 1.27)) (justify left bottom))
   )
-  (label "WRITE_CORE" (at 518.16 102.235 180) (fields_autoplaced)
+  (label "*WRITE_CORE" (at 518.16 102.235 180) (fields_autoplaced)
     (effects (font (size 1.27 1.27)) (justify right bottom))
   )

Commit message: Continue work on memory board
Connections:
- net EXTRA7 renamed NEXT_BANK0
- net EXTRA8 renamed NEXT_BANK1
- net REST_PEND renamed *REST_PEND

Commit message: Finish pinout audit + fanout correction
Connections:
- net BUS_SELECT2: now also U27.10, U27.9; no longer U1.1 (OEa), U1.15 (OEb), U2.1 (OEa), U2.15 (OEb), U3.1 (OEa), U3.15 (OEb), U4.1 (OEa), U4.15 (OEb), U5.1 (OEa), U5.15 (OEb), U6.1 (OEa), U6.15 (OEb), U7.1 (OEa), U7.15 (OEb), U8.1 (OEa), U8.15 (OEb), U9.1 (OEa), U9.15 (OEb)
- net GND: no longer U27.10, U27.4, U27.5, U27.9
- net at U27.6: now also U1.1 (OEa), U1.15 (OEb), U2.1 (OEa), U2.15 (OEb), U3.1 (OEa), U3.15 (OEb), U4.1 (OEa), U4.15 (OEb), U5.1 (OEa), U5.15 (OEb)
- net at U27.8: now also U27.4, U27.5, U6.1 (OEa), U6.15 (OEb), U7.1 (OEa), U7.15 (OEb), U8.1 (OEa), U8.15 (OEb), U9.1 (OEa), U9.15 (OEb)
- no-connect marks 98 -> 96
Other:
- moved on the sheet: U27B, U27C, U27D

Commit message: Start work on backplane and fix connectors
Parts:
- removed J1: Control Connector, symbol Connector:DIN41612_02x32_AC
- removed J2: Data Connector, symbol Connector:DIN41612_02x32_AC
- added J1: Control Connector, Connector_DIN:DIN41612_B_2x32_Male_Horizontal_THT, symbol Connector:DIN41612_02x32_AB
- added J2: Data Connector, Connector_DIN:DIN41612_B_2x32_Male_Horizontal_THT, symbol Connector:DIN41612_02x32_AB
Connections:
- net *CAF: now also J2.a22 (Pin_a22)
- net *CHAN_REQ: now also J1.a7 (Pin_a7)
- net *DEV_REQ: now also J1.a8 (Pin_a8)
- net *DMA_REQ: now also J1.a6 (Pin_a6)
- net *INT_REQ: now also J1.a9 (Pin_a9)
- net *IOT_SKIP: now also J1.a10 (Pin_a10)
- net *IOT_SKIP_L: now also J1.a12 (Pin_a12)
- net *IOT_WAIT: now also J1.a11 (Pin_a11)
- net *LATCH_AC: now also J1.a16 (Pin_a16)
- net *LATCH_IR: now also J1.a13 (Pin_a13)
- net *LATCH_MA: now also J1.a14 (Pin_a14)
- net *LATCH_MB: now also J1.a19 (Pin_a19)
- net *LATCH_MQ: now also J1.a18 (Pin_a18)
- net *LATCH_OB: now also J1.a21 (Pin_a21)
- net *LATCH_PC: now also J1.a15 (Pin_a15)
- net *LATCH_STEP: now also J1.a17 (Pin_a17)
- net *LATCH_WRTBK: now also J1.a20 (Pin_a20)
- net *MEMM_ENABLE: now also J1.a4 (Pin_a4)
- net *PI_ENABLE: now also J1.a3 (Pin_a3)
- net *PROT_ENABLE: now also J1.a5 (Pin_a5)
- net *RESET: now also J2.a21 (Pin_a21)
- net *REST_PEND: now also J2.a28 (Pin_a28)
- net *SELECT_AC: now also J1.b12 (Pin_b12)
- net *SELECT_ALU: now also J1.b16 (Pin_b16)
- net *SELECT_CORE: now also J1.b17 (Pin_b17)
- net *SELECT_CROSS: now also J1.b15 (Pin_b15)
- net *SELECT_EXTRN: now also J1.b19 (Pin_b19)
- net *SELECT_MQ: now also J1.b14 (Pin_b14)
- net *SELECT_STEP: now also J1.b13 (Pin_b13)
- net *SELECT_SWR: now also J1.b18 (Pin_b18)
- net *WRITE_CORE: now also J1.a22 (Pin_a22)
- net +5V: now also J1.a32 (Pin_a32), J1.b1 (Pin_b1), J2.a32 (Pin_a32), J2.b1 (Pin_b1)
- net A0: now also J2.b3 (Pin_b3)
- net A1: now also J2.b4 (Pin_b4)
- net A10: now also J2.b13 (Pin_b13)
- net A11: now also J2.b14 (Pin_b14)
- net A12: now also J2.b15 (Pin_b15)
- net A13: now also J2.b16 (Pin_b16)
- net A14: now also J2.b17 (Pin_b17)
- net A2: now also J2.b5 (Pin_b5)
- net A3: now also J2.b6 (Pin_b6)
- net A4: now also J2.b7 (Pin_b7)
- net A5: now also J2.b8 (Pin_b8)
- net A6: now also J2.b9 (Pin_b9)
- net A7: now also J2.b10 (Pin_b10)
- net A8: now also J2.b11 (Pin_b11)
- net A9: now also J2.b12 (Pin_b12)
- net ADDR_MODE0: now also J1.b27 (Pin_b27)
- net ADDR_MODE1: now also J1.b28 (Pin_b28)
- net ALUO0: now also J1.a24 (Pin_a24)
- net ALUO1: now also J1.a25 (Pin_a25)
- net ALUO2: now also J1.a26 (Pin_a26)
- net ALU_ONES: now also J1.a30 (Pin_a30)
- net ALU_SHIFT: now also J1.a29 (Pin_a29)
- net BUS_SELECT0: now also J1.b9 (Pin_b9)
- net BUS_SELECT1: now also J1.b10 (Pin_b10)
- net BUS_SELECT2: now also J1.b11 (Pin_b11)
- net CLK: now also J2.a23 (Pin_a23)
- net CTL_CONST: now also J1.b29 (Pin_b29)
- net D0: now also J2.a3 (Pin_a3)
- net D1: now also J2.a4 (Pin_a4)
- net D10: now also J2.a13 (Pin_a13)
- net D11: now also J2.a14 (Pin_a14)
- net D12: now also J2.a15 (Pin_a15)
- net D13: now also J2.a16 (Pin_a16)
- net D14: now also J2.a17 (Pin_a17)
- net D15: now also J2.a18 (Pin_a18)
- net D16: now also J2.a19 (Pin_a19)
- net D17: now also J2.a20 (Pin_a20)
- net D2: now also J2.a5 (Pin_a5)
- net D3: now also J2.a6 (Pin_a6)
- net D4: now also J2.a7 (Pin_a7)
- net D5: now also J2.a8 (Pin_a8)
- net D6: now also J2.a9 (Pin_a9)
- net D7: now also J2.a10 (Pin_a10)
- net D8: now also J2.a11 (Pin_a11)
- net D9: now also J2.a12 (Pin_a12)
- net DRQ_GRANT: now also J1.b21 (Pin_b21)
- net EXTRA0: now also J1.b30 (Pin_b30)
- net EXTRA1: now also J2.a24 (Pin_a24)
- net EXTRA2: now also J2.b24 (Pin_b24)
- net EXTRA3: now also J2.a25 (Pin_a25)
- net EXTRA4: now also J2.b25 (Pin_b25)
- net EXTRA5: now also J2.a26 (Pin_a26)
- net EXTRA6: now also J2.b26 (Pin_b26)
- net FLAG_AC_SIGN: now also J1.b8 (Pin_b8)
- net FLAG_LINK: now also J1.b6 (Pin_b6)
- net FLAG_LINK_INIT: now also J1.b7 (Pin_b7)
- net FLAG_SIGN: now also J1.b5 (Pin_b5)
- net FLAG_ZERO: now also J1.b4 (Pin_b4)
- net FP0: now also J2.a29 (Pin_a29)
- net FP1: now also J2.b29 (Pin_b29)
- net FP2: now also J2.a30 (Pin_a30)
- net FP3: now also J2.b30 (Pin_b30)
- net GND: now also J1.a1 (Pin_a1), J1.b32 (Pin_b32), J2.a1 (Pin_a1), J2.b32 (Pin_b32)
- net HALT: now also J1.b26 (Pin_b26)
- net INT_DETECT: now also J1.b24 (Pin_b24)
- net IOT_PULSE: now also J1.b20 (Pin_b20)
- net JMP_I_DETECT: now also J1.b23 (Pin_b23)
- net LINKS0: now also J1.a27 (Pin_a27)
- net LINKS1: now also J1.a28 (Pin_a28)
- net MA_AUTO_INX: now also J2.b28 (Pin_b28)
- net NEXT_BANK0: now also J2.a27 (Pin_a27)
- net NEXT_BANK1: now also J2.b27 (Pin_b27)
- net READ_IN_PULSE: now also J1.b25 (Pin_b25)
- net REQ_ADDR: now also J1.b22 (Pin_b22)
- net SC0: now also J2.b18 (Pin_b18)
- net SC1: now also J2.b19 (Pin_b19)
- net SC2: now also J2.b20 (Pin_b20)
- net SC3: now also J2.b21 (Pin_b21)
- net SC4: now also J2.b22 (Pin_b22)
- net SC5: now also J2.b23 (Pin_b23)
- net SELECT_PCMA: now also J1.a23 (Pin_a23)
- net STEP_ZERO: now also J1.b3 (Pin_b3)

Commit message: Update backplane pin logic levels
Connections:
- net DRQ_GRANT renamed *DRQ_GRANT
- net INT_DETECT renamed *INT_DETECT
- net IOT_PULSE renamed *IOT_PULSE
- net JMP_I_DETECT renamed *JMP_I_DETECT
- net READ_IN_PULSE renamed *READ_IN_PULSE
Changed lines of the file:
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@@
     (effects (font (size 1.27 1.27)) (justify left bottom))
   )
-  (label "READ_IN_PULSE" (at 530.86 109.855 0) (fields_autoplaced)
+  (label "*READ_IN_PULSE" (at 530.86 109.855 0) (fields_autoplaced)
     (effects (font (size 1.27 1.27)) (justify left bottom))
   )
@@
     (effects (font (size 1.27 1.27)) (justify left bottom))
   )
-  (label "INT_DETECT" (at 530.86 107.315 0) (fields_autoplaced)
+  (label "*INT_DETECT" (at 530.86 107.315 0) (fields_autoplaced)
     (effects (font (size 1.27 1.27)) (justify left bottom))
   )
@@
     (effects (font (size 1.27 1.27)) (justify right bottom))
   )
-  (label "JMP_I_DETECT" (at 530.86 104.775 0) (fields_autoplaced)
+  (label "*JMP_I_DETECT" (at 530.86 104.775 0) (fields_autoplaced)
     (effects (font (size 1.27 1.27)) (justify left bottom))
   )
@@
     (effects (font (size 1.27 1.27)) (justify left bottom))
   )
-  (label "DRQ_GRANT" (at 530.86 99.695 0) (fields_autoplaced)
+  (label "*DRQ_GRANT" (at 530.86 99.695 0) (fields_autoplaced)
     (effects (font (size 1.27 1.27)) (justify left bottom))
   )
@@
     (effects (font (size 1.27 1.27)) (justify left bottom))
   )
-  (label "IOT_PULSE" (at 530.86 97.155 0) (fields_autoplaced)
-    (effects (font (size 1.27 1.27)) (justify left bottom))
-  )
+  (label "*IOT_PULSE" (at 530.86 97.155 0) (fields_autoplaced)
+    (effects (font (size 1.27 1.27)) (justify left bottom))
+  )
