File: kicad/Registers/Registers.kicad_sch (KiCad schematic)
At the start: 59 parts, among them J1 Control Connector, J2 Data Connector, U1 74LS253, U10 74LS244, U11 74LS244, U12 74LS244, U13 74LS377, U14 74LS377, U15 74LS377, U16 74LS377, U17 74LS377, U18 74LS377, U19 74LS169, U2 74LS253, U20 74LS169, U21 74LS283, U22 74LS283, U23 74LS283, U24 74LS283, U25 74LS32, U26 74LS02, U27 74LS32, U3 74LS253, U4 74LS253, U5 74LS253, U6 74LS253, U7 74LS253, U8 74LS253, U9 74LS253

Commit message: The great PCB layout-athon
Parts:
- C1, C10, C11, C12, C13, C14, C15, C16, C17, C18, C19, C2, C20, C21, C22, C23, C24, C25, C26, C27, C3, C4, C5, C6, C7, C8, C9: footprint (none) -> Capacitor_THT:C_Disc_D5.0mm_W2.5mm_P5.00mm
- R1, R2: footprint (none) -> Resistor_THT:R_Axial_DIN0207_L6.3mm_D2.5mm_P7.62mm_Horizontal
- U1, U19, U2, U20, U21, U22, U23, U24, U3, U4, U5, U6, U7, U8, U9: footprint (none) -> Package_DIP:DIP-16_W7.62mm
- U10, U11, U12, U13, U14, U15, U16, U17, U18: footprint (none) -> Package_DIP:DIP-20_W7.62mm
- U25, U26, U27: footprint (none) -> Package_DIP:DIP-14_W7.62mm
