File: kicad/Backplane/Backplane.kicad_sch (KiCad schematic)
At the start: 0 parts

Commit message: Continue work on blackplane
Parts:
- added J1, J3, J5, J7: Control Connector, Connector_DIN:DIN41612_B_2x32_Male_Horizontal_THT, symbol Connector:DIN41612_02x32_AB
- added J2, J4, J6, J8: Data Connector, Connector_DIN:DIN41612_B_2x32_Male_Horizontal_THT, symbol Connector:DIN41612_02x32_AB
- added U1, U2: 74LS244, symbol 74xx:74LS244
- added X1: 4 Mhz Oscillator, Oscillator:Oscillator_DIP-14, symbol Oscillator:GTXO-14T
Connections:
- new net: U1.11 (I0b), U1.13 (I1b), U1.15 (I2b), U1.16 (O1a), U1.17 (I3b)
- new net: U1.14 (O2a), U2.11 (I0b), U2.13 (I1b), U2.15 (I2b), U2.17 (I3b), U2.2 (I0a), U2.4 (I1a), U2.6 (I2a), U2.8 (I3a)
- new net: U1.18 (O0a), U1.4 (I1a), U1.6 (I2a), U1.8 (I3a)
- new net *CAF: J2.a22 (Pin_a22), J4.a22 (Pin_a22), J6.a22 (Pin_a22), J8.a22 (Pin_a22)
- new net *CHAN_REQ: J1.a7 (Pin_a7), J3.a7 (Pin_a7), J5.a7 (Pin_a7), J7.a7 (Pin_a7)
- new net *DEV_REQ: J1.a8 (Pin_a8), J3.a8 (Pin_a8), J5.a8 (Pin_a8), J7.a8 (Pin_a8)
- new net *DMA_REQ: J1.a6 (Pin_a6), J3.a6 (Pin_a6), J5.a6 (Pin_a6), J7.a6 (Pin_a6)
- new net *INT_REQ: J1.a9 (Pin_a9), J3.a9 (Pin_a9), J5.a9 (Pin_a9), J7.a9 (Pin_a9)
- new net *IOT_SKIP: J1.a10 (Pin_a10), J3.a10 (Pin_a10), J5.a10 (Pin_a10), J7.a10 (Pin_a10)
- new net *IOT_SKIP_L: J1.a12 (Pin_a12), J3.a12 (Pin_a12), J5.a12 (Pin_a12), J7.a12 (Pin_a12)
- new net *IOT_WAIT: J1.a11 (Pin_a11), J3.a11 (Pin_a11), J5.a11 (Pin_a11), J7.a11 (Pin_a11)
- new net *LATCH_AC: J1.a16 (Pin_a16), J3.a16 (Pin_a16), J5.a16 (Pin_a16), J7.a16 (Pin_a16)
- new net *LATCH_IR: J1.a13 (Pin_a13), J3.a13 (Pin_a13), J5.a13 (Pin_a13), J7.a13 (Pin_a13)
- new net *LATCH_MA: J1.a14 (Pin_a14), J3.a14 (Pin_a14), J5.a14 (Pin_a14), J7.a14 (Pin_a14)
- new net *LATCH_MB: J1.a19 (Pin_a19), J3.a19 (Pin_a19), J5.a19 (Pin_a19), J7.a19 (Pin_a19)
- new net *LATCH_MQ: J1.a18 (Pin_a18), J3.a18 (Pin_a18), J5.a18 (Pin_a18), J7.a18 (Pin_a18)
- new net *LATCH_OB: J1.a21 (Pin_a21), J3.a21 (Pin_a21), J5.a21 (Pin_a21), J7.a21 (Pin_a21)
- new net *LATCH_PC: J1.a15 (Pin_a15), J3.a15 (Pin_a15), J5.a15 (Pin_a15), J7.a15 (Pin_a15)
- new net *LATCH_STEP: J1.a17 (Pin_a17), J3.a17 (Pin_a17), J5.a17 (Pin_a17), J7.a17 (Pin_a17)
- new net *LATCH_WRTBK: J1.a20 (Pin_a20), J3.a20 (Pin_a20), J5.a20 (Pin_a20), J7.a20 (Pin_a20)
- new net *MEMM_ENABLE: J1.a4 (Pin_a4), J3.a4 (Pin_a4), J5.a4 (Pin_a4), J7.a4 (Pin_a4)
- new net *PI_ENABLE: J1.a3 (Pin_a3), J3.a3 (Pin_a3), J5.a3 (Pin_a3), J7.a3 (Pin_a3)
- new net *PROT_ENABLE: J1.a5 (Pin_a5), J3.a5 (Pin_a5), J5.a5 (Pin_a5), J7.a5 (Pin_a5)
- new net *RESET: J2.a21 (Pin_a21), J4.a21 (Pin_a21), J6.a21 (Pin_a21), J8.a21 (Pin_a21)
- new net *REST_PEND: J2.a28 (Pin_a28), J4.a28 (Pin_a28), J6.a28 (Pin_a28), J8.a28 (Pin_a28)
- new net *SELECT_AC: J1.b12 (Pin_b12), J3.b12 (Pin_b12), J5.b12 (Pin_b12), J7.b12 (Pin_b12)
- new net *SELECT_ALU: J1.b16 (Pin_b16), J3.b16 (Pin_b16), J5.b16 (Pin_b16), J7.b16 (Pin_b16)
- new net *SELECT_CORE: J1.b17 (Pin_b17), J3.b17 (Pin_b17), J5.b17 (Pin_b17), J7.b17 (Pin_b17)
- new net *SELECT_CROSS: J1.b15 (Pin_b15), J3.b15 (Pin_b15), J5.b15 (Pin_b15), J7.b15 (Pin_b15)
- new net *SELECT_EXTRN: J1.b19 (Pin_b19), J3.b19 (Pin_b19), J5.b19 (Pin_b19), J7.b19 (Pin_b19)
- new net *SELECT_MQ: J1.b14 (Pin_b14), J3.b14 (Pin_b14), J5.b14 (Pin_b14), J7.b14 (Pin_b14)
- new net *SELECT_STEP: J1.b13 (Pin_b13), J3.b13 (Pin_b13), J5.b13 (Pin_b13), J7.b13 (Pin_b13)
- new net *SELECT_SWR: J1.b18 (Pin_b18), J3.b18 (Pin_b18), J5.b18 (Pin_b18), J7.b18 (Pin_b18)
- new net *WRITE_CORE: J1.a22 (Pin_a22), J3.a22 (Pin_a22), J5.a22 (Pin_a22), J7.a22 (Pin_a22)
- new net +5V: J1.a32 (Pin_a32), J1.b1 (Pin_b1), J2.a32 (Pin_a32), J2.b1 (Pin_b1), J3.a32 (Pin_a32), J3.b1 (Pin_b1), J4.a32 (Pin_a32), J4.b1 (Pin_b1), J5.a32 (Pin_a32), J5.b1 (Pin_b1), J6.a32 (Pin_a32), J6.b1 (Pin_b1), J7.a32 (Pin_a32), J7.b1 (Pin_b1), J8.a32 (Pin_a32), J8.b1 (Pin_b1), U1.20 (VCC), U2.20 (VCC), X1.14 (Vcc)
- new net A0: J2.b3 (Pin_b3), J4.b3 (Pin_b3), J6.b3 (Pin_b3), J8.b3 (Pin_b3)
- new net A1: J2.b4 (Pin_b4), J4.b4 (Pin_b4), J6.b4 (Pin_b4), J8.b4 (Pin_b4)
- new net A10: J2.b13 (Pin_b13), J4.b13 (Pin_b13), J6.b13 (Pin_b13), J8.b13 (Pin_b13)
- new net A11: J2.b14 (Pin_b14), J4.b14 (Pin_b14), J6.b14 (Pin_b14), J8.b14 (Pin_b14)
- new net A12: J2.b15 (Pin_b15), J4.b15 (Pin_b15), J6.b15 (Pin_b15), J8.b15 (Pin_b15)
- new net A13: J2.b16 (Pin_b16), J4.b16 (Pin_b16), J6.b16 (Pin_b16), J8.b16 (Pin_b16)
- new net A14: J2.b17 (Pin_b17), J4.b17 (Pin_b17), J6.b17 (Pin_b17), J8.b17 (Pin_b17)
- new net A2: J2.b5 (Pin_b5), J4.b5 (Pin_b5), J6.b5 (Pin_b5), J8.b5 (Pin_b5)
- new net A3: J2.b6 (Pin_b6), J4.b6 (Pin_b6), J6.b6 (Pin_b6), J8.b6 (Pin_b6)
- new net A4: J2.b7 (Pin_b7), J4.b7 (Pin_b7), J6.b7 (Pin_b7), J8.b7 (Pin_b7)
- new net A5: J2.b8 (Pin_b8), J4.b8 (Pin_b8), J6.b8 (Pin_b8), J8.b8 (Pin_b8)
- new net A6: J2.b9 (Pin_b9), J4.b9 (Pin_b9), J6.b9 (Pin_b9), J8.b9 (Pin_b9)
- new net A7: J2.b10 (Pin_b10), J4.b10 (Pin_b10), J6.b10 (Pin_b10), J8.b10 (Pin_b10)
- new net A8: J2.b11 (Pin_b11), J4.b11 (Pin_b11), J6.b11 (Pin_b11), J8.b11 (Pin_b11)
- new net A9: J2.b12 (Pin_b12), J4.b12 (Pin_b12), J6.b12 (Pin_b12), J8.b12 (Pin_b12)
- new net ADDR_MODE0: J1.b27 (Pin_b27), J3.b27 (Pin_b27), J5.b27 (Pin_b27), J7.b27 (Pin_b27)
- new net ADDR_MODE1: J1.b28 (Pin_b28), J3.b28 (Pin_b28), J5.b28 (Pin_b28), J7.b28 (Pin_b28)
- new net ALUO0: J1.a24 (Pin_a24), J3.a24 (Pin_a24), J5.a24 (Pin_a24), J7.a24 (Pin_a24)
- new net ALUO1: J1.a25 (Pin_a25), J3.a25 (Pin_a25), J5.a25 (Pin_a25), J7.a25 (Pin_a25)
- new net ALUO2: J1.a26 (Pin_a26), J3.a26 (Pin_a26), J5.a26 (Pin_a26), J7.a26 (Pin_a26)
- new net ALU_ONES: J1.a30 (Pin_a30), J3.a30 (Pin_a30), J5.a30 (Pin_a30), J7.a30 (Pin_a30)
- new net ALU_SHIFT: J1.a29 (Pin_a29), J3.a29 (Pin_a29), J5.a29 (Pin_a29), J7.a29 (Pin_a29)
- new net BUS_SELECT0: J1.b9 (Pin_b9), J3.b9 (Pin_b9), J5.b9 (Pin_b9), J7.b9 (Pin_b9)
- new net BUS_SELECT1: J1.b10 (Pin_b10), J3.b10 (Pin_b10), J5.b10 (Pin_b10), J7.b10 (Pin_b10)
- new net BUS_SELECT2: J1.b11 (Pin_b11), J3.b11 (Pin_b11), J5.b11 (Pin_b11), J7.b11 (Pin_b11)
- new net CLK0: J2.a23 (Pin_a23), U1.9 (O0b)
- new net CLK1: J4.a23 (Pin_a23), U1.7 (O1b)
- new net CLK10: U2.5 (O2b)
- new net CLK11: U2.3 (O3b)
- new net CLK2: J6.a23 (Pin_a23), U1.5 (O2b)
- new net CLK3: J8.a23 (Pin_a23), U1.3 (O3b)
- new net CLK4: U2.18 (O0a)
- new net CLK5: U2.16 (O1a)
- new net CLK6: U2.14 (O2a)
- new net CLK7: U2.12 (O3a)
- new net CLK8: U2.9 (O0b)
- new net CLK9: U2.7 (O1b)
- new net CLKSRC: U1.12 (O3a)
- new net CTL_CONST: J1.b29 (Pin_b29), J3.b29 (Pin_b29), J5.b29 (Pin_b29), J7.b29 (Pin_b29)
- new net D0: J2.a3 (Pin_a3), J4.a3 (Pin_a3), J6.a3 (Pin_a3), J8.a3 (Pin_a3)
- new net D1: J2.a4 (Pin_a4), J4.a4 (Pin_a4), J6.a4 (Pin_a4), J8.a4 (Pin_a4)
- new net D10: J2.a13 (Pin_a13), J4.a13 (Pin_a13), J6.a13 (Pin_a13), J8.a13 (Pin_a13)
- new net D11: J2.a14 (Pin_a14), J4.a14 (Pin_a14), J6.a14 (Pin_a14), J8.a14 (Pin_a14)
- new net D12: J2.a15 (Pin_a15), J4.a15 (Pin_a15), J6.a15 (Pin_a15), J8.a15 (Pin_a15)
- new net D13: J2.a16 (Pin_a16), J4.a16 (Pin_a16), J6.a16 (Pin_a16), J8.a16 (Pin_a16)
- new net D14: J2.a17 (Pin_a17), J4.a17 (Pin_a17), J6.a17 (Pin_a17), J8.a17 (Pin_a17)
- new net D15: J2.a18 (Pin_a18), J4.a18 (Pin_a18), J6.a18 (Pin_a18), J8.a18 (Pin_a18)
- new net D16: J2.a19 (Pin_a19), J4.a19 (Pin_a19), J6.a19 (Pin_a19), J8.a19 (Pin_a19)
- new net D17: J2.a20 (Pin_a20), J4.a20 (Pin_a20), J6.a20 (Pin_a20), J8.a20 (Pin_a20)
- new net D2: J2.a5 (Pin_a5), J4.a5 (Pin_a5), J6.a5 (Pin_a5), J8.a5 (Pin_a5)
- new net D3: J2.a6 (Pin_a6), J4.a6 (Pin_a6), J6.a6 (Pin_a6), J8.a6 (Pin_a6)
- new net D4: J2.a7 (Pin_a7), J4.a7 (Pin_a7), J6.a7 (Pin_a7), J8.a7 (Pin_a7)
- new net D5: J2.a8 (Pin_a8), J4.a8 (Pin_a8), J6.a8 (Pin_a8), J8.a8 (Pin_a8)
- new net D6: J2.a9 (Pin_a9), J4.a9 (Pin_a9), J6.a9 (Pin_a9), J8.a9 (Pin_a9)
- new net D7: J2.a10 (Pin_a10), J4.a10 (Pin_a10), J6.a10 (Pin_a10), J8.a10 (Pin_a10)
- new net D8: J2.a11 (Pin_a11), J4.a11 (Pin_a11), J6.a11 (Pin_a11), J8.a11 (Pin_a11)
- new net D9: J2.a12 (Pin_a12), J4.a12 (Pin_a12), J6.a12 (Pin_a12), J8.a12 (Pin_a12)
- new net DRQ_GRANT: J1.b21 (Pin_b21), J3.b21 (Pin_b21), J5.b21 (Pin_b21), J7.b21 (Pin_b21)
- new net EXTRA0: J1.b30 (Pin_b30), J3.b30 (Pin_b30), J5.b30 (Pin_b30), J7.b30 (Pin_b30)
- new net EXTRA1: J2.a24 (Pin_a24), J4.a24 (Pin_a24), J6.a24 (Pin_a24), J8.a24 (Pin_a24)
- new net EXTRA2: J2.b24 (Pin_b24), J4.b24 (Pin_b24), J6.b24 (Pin_b24), J8.b24 (Pin_b24)
- new net EXTRA3: J2.a25 (Pin_a25), J4.a25 (Pin_a25), J6.a25 (Pin_a25), J8.a25 (Pin_a25)
- new net EXTRA4: J2.b25 (Pin_b25), J4.b25 (Pin_b25), J6.b25 (Pin_b25), J8.b25 (Pin_b25)
- new net EXTRA5: J2.a26 (Pin_a26), J4.a26 (Pin_a26), J6.a26 (Pin_a26), J8.a26 (Pin_a26)
- new net EXTRA6: J2.b26 (Pin_b26), J4.b26 (Pin_b26), J6.b26 (Pin_b26), J8.b26 (Pin_b26)
- new net FLAG_AC_SIGN: J1.b8 (Pin_b8), J3.b8 (Pin_b8), J5.b8 (Pin_b8), J7.b8 (Pin_b8)
- new net FLAG_LINK: J1.b6 (Pin_b6), J3.b6 (Pin_b6), J5.b6 (Pin_b6), J7.b6 (Pin_b6)
- new net FLAG_LINK_INIT: J1.b7 (Pin_b7), J3.b7 (Pin_b7), J5.b7 (Pin_b7), J7.b7 (Pin_b7)
- new net FLAG_SIGN: J1.b5 (Pin_b5), J3.b5 (Pin_b5), J5.b5 (Pin_b5), J7.b5 (Pin_b5)
- new net FLAG_ZERO: J1.b4 (Pin_b4), J3.b4 (Pin_b4), J5.b4 (Pin_b4), J7.b4 (Pin_b4)
- new net FP0: J2.a29 (Pin_a29), J4.a29 (Pin_a29), J6.a29 (Pin_a29), J8.a29 (Pin_a29)
- new net FP1: J2.b29 (Pin_b29), J4.b29 (Pin_b29), J6.b29 (Pin_b29), J8.b29 (Pin_b29)
- new net FP2: J2.a30 (Pin_a30), J4.a30 (Pin_a30), J6.a30 (Pin_a30), J8.a30 (Pin_a30)
- new net FP3: J2.b30 (Pin_b30), J4.b30 (Pin_b30), J6.b30 (Pin_b30), J8.b30 (Pin_b30)
- new net GND: J1.a1 (Pin_a1), J1.b32 (Pin_b32), J2.a1 (Pin_a1), J2.b32 (Pin_b32), J3.a1 (Pin_a1), J3.b32 (Pin_b32), J4.a1 (Pin_a1), J4.b32 (Pin_b32), J5.a1 (Pin_a1), J5.b32 (Pin_b32), J6.a1 (Pin_a1), J6.b32 (Pin_b32), J7.a1 (Pin_a1), J7.b32 (Pin_b32), J8.a1 (Pin_a1), J8.b32 (Pin_b32), U1.1 (OEa), U1.10 (GND), U1.19 (OEb), U2.1 (OEa), U2.10 (GND), U2.19 (OEb), X1.7 (GND)
- new net HALT: J1.b26 (Pin_b26), J3.b26 (Pin_b26), J5.b26 (Pin_b26), J7.b26 (Pin_b26)
- new net INT_DETECT: J1.b24 (Pin_b24), J3.b24 (Pin_b24), J5.b24 (Pin_b24), J7.b24 (Pin_b24)
- new net IOT_PULSE: J1.b20 (Pin_b20), J3.b20 (Pin_b20), J5.b20 (Pin_b20), J7.b20 (Pin_b20)
- new net JMP_I_DETECT: J1.b23 (Pin_b23), J3.b23 (Pin_b23), J5.b23 (Pin_b23), J7.b23 (Pin_b23)
- new net LINKS0: J1.a27 (Pin_a27), J3.a27 (Pin_a27), J5.a27 (Pin_a27), J7.a27 (Pin_a27)
- new net LINKS1: J1.a28 (Pin_a28), J3.a28 (Pin_a28), J5.a28 (Pin_a28), J7.a28 (Pin_a28)
- new net MA_AUTO_INX: J2.b28 (Pin_b28), J4.b28 (Pin_b28), J6.b28 (Pin_b28), J8.b28 (Pin_b28)
- new net NEXT_BANK0: J2.a27 (Pin_a27), J4.a27 (Pin_a27), J6.a27 (Pin_a27), J8.a27 (Pin_a27)
- new net NEXT_BANK1: J2.b27 (Pin_b27), J4.b27 (Pin_b27), J6.b27 (Pin_b27), J8.b27 (Pin_b27)
- new net READ_IN_PULSE: J1.b25 (Pin_b25), J3.b25 (Pin_b25), J5.b25 (Pin_b25), J7.b25 (Pin_b25)
- new net REQ_ADDR: J1.b22 (Pin_b22), J3.b22 (Pin_b22), J5.b22 (Pin_b22), J7.b22 (Pin_b22)
- new net SC0: J2.b18 (Pin_b18), J4.b18 (Pin_b18), J6.b18 (Pin_b18), J8.b18 (Pin_b18)
- new net SC1: J2.b19 (Pin_b19), J4.b19 (Pin_b19), J6.b19 (Pin_b19), J8.b19 (Pin_b19)
- new net SC2: J2.b20 (Pin_b20), J4.b20 (Pin_b20), J6.b20 (Pin_b20), J8.b20 (Pin_b20)
- new net SC3: J2.b21 (Pin_b21), J4.b21 (Pin_b21), J6.b21 (Pin_b21), J8.b21 (Pin_b21)
- new net SC4: J2.b22 (Pin_b22), J4.b22 (Pin_b22), J6.b22 (Pin_b22), J8.b22 (Pin_b22)
- new net SC5: J2.b23 (Pin_b23), J4.b23 (Pin_b23), J6.b23 (Pin_b23), J8.b23 (Pin_b23)
- new net SELECT_PCMA: J1.a23 (Pin_a23), J3.a23 (Pin_a23), J5.a23 (Pin_a23), J7.a23 (Pin_a23)
- new net STEP_ZERO: J1.b3 (Pin_b3), J3.b3 (Pin_b3), J5.b3 (Pin_b3), J7.b3 (Pin_b3)
- no-connect marks 0 -> 33
