File: kicad/Backplane/Backplane.kicad_sch (KiCad schematic)
At the start: 11 parts, among them J1 Control Connector, J2 Data Connector, J3 Control Connector, J4 Data Connector, J5 Control Connector, J6 Data Connector, J7 Control Connector, J8 Data Connector, U1 74LS244, U2 74LS244, X1 4 Mhz Oscillator

Commit message: Update backplane pin logic levels
Connections:
- net DRQ_GRANT renamed *DRQ_GRANT
- net INT_DETECT renamed *INT_DETECT
- net IOT_PULSE renamed *IOT_PULSE
- net JMP_I_DETECT renamed *JMP_I_DETECT
- net READ_IN_PULSE renamed *READ_IN_PULSE
Changed lines of the file:
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@@
     (effects (font (size 1.27 1.27)) (justify left bottom))
   )
-  (label "JMP_I_DETECT" (at 47.625 82.55 0) (fields_autoplaced)
+  (label "*JMP_I_DETECT" (at 47.625 82.55 0) (fields_autoplaced)
     (effects (font (size 1.27 1.27)) (justify left bottom))
   )
@@
     (effects (font (size 1.27 1.27)) (justify left bottom))
   )
-  (label "DRQ_GRANT" (at 47.625 77.47 0) (fields_autoplaced)
+  (label "*DRQ_GRANT" (at 47.625 77.47 0) (fields_autoplaced)
     (effects (font (size 1.27 1.27)) (justify left bottom))
   )
@@
     (effects (font (size 1.27 1.27)) (justify left bottom))
   )
-  (label "IOT_PULSE" (at 181.61 74.93 0) (fields_autoplaced)
+  (label "*IOT_PULSE" (at 181.61 74.93 0) (fields_autoplaced)
     (effects (font (size 1.27 1.27)) (justify left bottom))
   )
@@
     (effects (font (size 1.27 1.27)) (justify left bottom))
   )
-  (label "JMP_I_DETECT" (at 92.71 82.55 0) (fields_autoplaced)
+  (label "*JMP_I_DETECT" (at 92.71 82.55 0) (fields_autoplaced)
     (effects (font (size 1.27 1.27)) (justify left bottom))
   )
@@
     (effects (font (size 1.27 1.27)) (justify right bottom))
   )
-  (label "JMP_I_DETECT" (at 137.16 82.55 0) (fields_autoplaced)
+  (label "*JMP_I_DETECT" (at 137.16 82.55 0) (fields_autoplaced)
     (effects (font (size 1.27 1.27)) (justify left bottom))
   )
@@
     (effects (font (size 1.27 1.27)) (justify right bottom))
   )
-  (label "INT_DETECT" (at 137.16 85.09 0) (fields_autoplaced)
+  (label "*INT_DETECT" (at 137.16 85.09 0) (fields_autoplaced)
     (effects (font (size 1.27 1.27)) (justify left bottom))
   )
@@
     (effects (font (size 1.27 1.27)) (justify left bottom))
   )
-  (label "IOT_PULSE" (at 92.71 74.93 0) (fields_autoplaced)
+  (label "*IOT_PULSE" (at 92.71 74.93 0) (fields_autoplaced)
     (effects (font (size 1.27 1.27)) (justify left bottom))
   )
@@
     (effects (font (size 1.27 1.27)) (justify left bottom))
   )
-  (label "READ_IN_PULSE" (at 181.61 87.63 0) (fields_autoplaced)
+  (label "*READ_IN_PULSE" (at 181.61 87.63 0) (fields_autoplaced)
     (effects (font (size 1.27 1.27)) (justify left bottom))
   )
@@
     (effects (font (size 1.27 1.27)) (justify left bottom))
   )
-  (label "READ_IN_PULSE" (at 47.625 87.63 0) (fields_autoplaced)
+  (label "*READ_IN_PULSE" (at 47.625 87.63 0) (fields_autoplaced)
     (effects (font (size 1.27 1.27)) (justify left bottom))
   )
@@
     (effects (font (size 1.27 1.27)) (justify right bottom))
   )
-  (label "INT_DETECT" (at 181.61 85.09 0) (fields_autoplaced)
+  (label "*INT_DETECT" (at 181.61 85.09 0) (fields_autoplaced)
     (effects (font (size 1.27 1.27)) (justify left bottom))
   )
@@
     (effects (font (size 1.27 1.27)) (justify left bottom))
   )
-  (label "DRQ_GRANT" (at 92.71 77.47 0) (fields_autoplaced)
+  (label "*DRQ_GRANT" (at 92.71 77.47 0) (fields_autoplaced)
     (effects (font (size 1.27 1.27)) (justify left bottom))
   )
@@
     (effects (font (size 1.27 1.27)) (justify right bottom))
   )
-  (label "DRQ_GRANT" (at 137.16 77.47 0) (fields_autoplaced)
+  (label "*DRQ_GRANT" (at 137.16 77.47 0) (fields_autoplaced)
     (effects (font (size 1.27 1.27)) (justify left bottom))
   )
@@
     (effects (font (size 1.27 1.27)) (justify right bottom))
   )
-  (label "DRQ_GRANT" (at 181.61 77.47 0) (fields_autoplaced)
+  (label "*DRQ_GRANT" (at 181.61 77.47 0) (fields_autoplaced)
     (effects (font (size 1.27 1.27)) (justify left bottom))
   )
@@
     (effects (font (size 1.27 1.27)) (justify right bottom))
   )
-  (label "IOT_PULSE" (at 47.625 74.93 0) (fields_autoplaced)
+  (label "*IOT_PULSE" (at 47.625 74.93 0) (fields_autoplaced)
     (effects (font (size 1.27 1.27)) (justify left bottom))
   )
@@
     (effects (font (size 1.27 1.27)) (justify left bottom))
   )
-  (label "READ_IN_PULSE" (at 92.71 87.63 0) (fields_autoplaced)
+  (label "*READ_IN_PULSE" (at 92.71 87.63 0) (fields_autoplaced)
     (effects (font (size 1.27 1.27)) (justify left bottom))
   )
@@
     (effects (font (size 1.27 1.27)) (justify right bottom))
   )
-  (label "IOT_PULSE" (at 137.16 74.93 0) (fields_autoplaced)
+  (label "*IOT_PULSE" (at 137.16 74.93 0) (fields_autoplaced)
     (effects (font (size 1.27 1.27)) (justify left bottom))
   )
@@
     (effects (font (size 1.27 1.27)) (justify right bottom))
   )
-  (label "JMP_I_DETECT" (at 181.61 82.55 0) (fields_autoplaced)
+  (label "*JMP_I_DETECT" (at 181.61 82.55 0) (fields_autoplaced)
     (effects (font (size 1.27 1.27)) (justify left bottom))
   )
@@
     (effects (font (size 1.27 1.27)) (justify right bottom))
   )
-  (label "INT_DETECT" (at 47.625 85.09 0) (fields_autoplaced)
+  (label "*INT_DETECT" (at 47.625 85.09 0) (fields_autoplaced)
     (effects (font (size 1.27 1.27)) (justify left bottom))
   )
@@
     (effects (font (size 1.27 1.27)) (justify left bottom))
   )
-  (label "INT_DETECT" (at 92.71 85.09 0) (fields_autoplaced)
+  (label "*INT_DETECT" (at 92.71 85.09 0) (fields_autoplaced)
     (effects (font (size 1.27 1.27)) (justify left bottom))
   )
@@
     (effects (font (size 1.27 1.27)) (justify left bottom))
   )
-  (label "READ_IN_PULSE" (at 137.16 87.63 0) (fields_autoplaced)
-    (effects (font (size 1.27 1.27)) (justify left bottom))
-  )
+  (label "*READ_IN_PULSE" (at 137.16 87.63 0) (fields_autoplaced)
+    (effects (font (size 1.27 1.27)) (justify left bottom))
+  )

Commit message: Continue work on backplane
Parts:
- added J9: I/O Connector, Connector_DIN:DIN41612_B_2x32_Male_Horizontal_THT, symbol Connector:DIN41612_02x32_AB
Connections:
- net *CAF: now also J9.a22 (Pin_a22)
- net *INT_DETECT: now also J9.a26 (Pin_a26)
- net *INT_REQ: now also J9.b25 (Pin_b25)
- net *IOT_PULSE: now also J9.a28 (Pin_a28)
- net *IOT_SKIP: now also J9.b2 (Pin_b2)
- net *IOT_WAIT: now also J9.a31 (Pin_a31)
- net *JMP_I_DETECT: now also J9.a27 (Pin_a27)
- net *MEMM_ENABLE: now also J9.b23 (Pin_b23)
- net *PI_ENABLE: now also J9.b22 (Pin_b22)
- net *PROT_ENABLE: now also J9.b24 (Pin_b24)
- net *READ_IN_PULSE: now also J9.a29 (Pin_a29)
- net *RESET: now also J9.a21 (Pin_a21)
- net +5V: now also J9.a32 (Pin_a32), J9.b1 (Pin_b1)
- net CLK4: now also J9.a23 (Pin_a23)
- net GND: now also J9.a1 (Pin_a1), J9.b32 (Pin_b32)
- net REQ_ADDR: now also J9.a24 (Pin_a24)
- new net *CAF_REQ: J9.b29 (Pin_b29)
- new net *CHAN_REQ0: J9.b27 (Pin_b27)
- new net *DMA_REQ0: J9.b26 (Pin_b26)
- new net *EXTERNAL: J9.b28 (Pin_b28)
- new net *INCREMENT_ZERO: J9.b30 (Pin_b30)
- new net *IORS_FLAG0: J9.b14 (Pin_b14)
- new net *IORS_FLAG1: J9.b15 (Pin_b15)
- new net *IORS_FLAG2: J9.b16 (Pin_b16)
- new net *IORS_FLAG3: J9.b17 (Pin_b17)
- new net *PTP_FLAG: J9.b19 (Pin_b19)
- new net *PTP_TAPE: J9.b21 (Pin_b21)
- new net *PTR_FLAG: J9.b18 (Pin_b18)
- new net *PTR_TAPE: J9.b20 (Pin_b20)
- new net *READ_IN_CLEAR: J9.a30 (Pin_a30)
- new net A_DEVICE0: J9.b3 (Pin_b3)
- new net A_DEVICE1: J9.b4 (Pin_b4)
- new net A_DEVICE2: J9.b5 (Pin_b5)
- new net A_DEVICE3: J9.b6 (Pin_b6)
- new net A_DEVICE4: J9.b7 (Pin_b7)
- new net A_DEVICE5: J9.b8 (Pin_b8)
- new net A_PULSE0: J9.b11 (Pin_b11)
- new net A_PULSE1: J9.b12 (Pin_b12)
- new net A_PULSE2: J9.b13 (Pin_b13)
- new net A_SUBDEV0: J9.b9 (Pin_b9)
- new net A_SUBDEV1: J9.b10 (Pin_b10)
- new net ID0: J9.a3 (Pin_a3)
- new net ID1: J9.a4 (Pin_a4)
- new net ID10: J9.a13 (Pin_a13)
- new net ID11: J9.a14 (Pin_a14)
- new net ID12: J9.a15 (Pin_a15)
- new net ID13: J9.a16 (Pin_a16)
- new net ID14: J9.a17 (Pin_a17)
- new net ID15: J9.a18 (Pin_a18)
- new net ID16: J9.a19 (Pin_a19)
- new net ID17: J9.a20 (Pin_a20)
- new net ID2: J9.a5 (Pin_a5)
- new net ID3: J9.a6 (Pin_a6)
- new net ID4: J9.a7 (Pin_a7)
- new net ID5: J9.a8 (Pin_a8)
- new net ID6: J9.a9 (Pin_a9)
- new net ID7: J9.a10 (Pin_a10)
- new net ID8: J9.a11 (Pin_a11)
- new net ID9: J9.a12 (Pin_a12)
- no-connect marks 33 -> 35

Commit message: Continue work on backplane
Parts:
- added J10, J11, J12, J13, J14: I/O Connector, Connector_DIN:DIN41612_B_2x32_Male_Horizontal_THT, symbol Connector:DIN41612_02x32_AB
- added J15, J16: Front Panel Connector, Connector_IDC:IDC-Header_2x25_P2.54mm_Vertical, symbol Connector_Generic:Conn_02x25_Counter_Clockwise
- added J17: Run, symbol Connector:Conn_01x02_Pin
- added J18: Clock, symbol Connector:Conn_01x02_Pin
- added J19: Rept, symbol Connector:Conn_01x02_Pin
- added J20: Reset, symbol Connector:Conn_01x02_Pin
- added J21: I/O Reset, symbol Connector:Conn_01x02_Pin
- added R1, R2, R3, R4, R5: 4.7K, Resistor_THT:R_Axial_DIN0207_L6.3mm_D2.5mm_P7.62mm_Horizontal, symbol Device:R
Connections:
- net *CAF: now also J10.a22 (Pin_a22), J11.a22 (Pin_a22), J12.a22 (Pin_a22), J13.a22 (Pin_a22), J14.a22 (Pin_a22)
- net *CAF_REQ: now also J10.b29 (Pin_b29), J11.b29 (Pin_b29), J12.b29 (Pin_b29), J13.b29 (Pin_b29), J14.b29 (Pin_b29)
- net *EXTERNAL: now also J10.b28 (Pin_b28), J11.b28 (Pin_b28), J12.b28 (Pin_b28), J13.b28 (Pin_b28), J14.b28 (Pin_b28)
- net *INCREMENT_ZERO: now also J10.b30 (Pin_b30), J11.b30 (Pin_b30), J12.b30 (Pin_b30), J13.b30 (Pin_b30), J14.b30 (Pin_b30)
- net *INT_DETECT: now also J10.a26 (Pin_a26), J11.a26 (Pin_a26), J12.a26 (Pin_a26), J13.a26 (Pin_a26), J14.a26 (Pin_a26)
- net *INT_REQ: now also J10.b25 (Pin_b25), J11.b25 (Pin_b25), J12.b25 (Pin_b25), J13.b25 (Pin_b25), J14.b25 (Pin_b25)
- net *IORS_FLAG0: now also J10.b14 (Pin_b14), J11.b14 (Pin_b14), J12.b14 (Pin_b14), J13.b14 (Pin_b14), J14.b14 (Pin_b14)
- net *IORS_FLAG1: now also J10.b15 (Pin_b15), J11.b15 (Pin_b15), J12.b15 (Pin_b15), J13.b15 (Pin_b15), J14.b15 (Pin_b15)
- net *IORS_FLAG2: now also J10.b16 (Pin_b16), J11.b16 (Pin_b16), J12.b16 (Pin_b16), J13.b16 (Pin_b16), J14.b16 (Pin_b16)
- net *IORS_FLAG3: now also J10.b17 (Pin_b17), J11.b17 (Pin_b17), J12.b17 (Pin_b17), J13.b17 (Pin_b17), J14.b17 (Pin_b17)
- net *IOT_PULSE: now also J10.a28 (Pin_a28), J11.a28 (Pin_a28), J12.a28 (Pin_a28), J13.a28 (Pin_a28), J14.a28 (Pin_a28)
- net *IOT_SKIP: now also J10.b2 (Pin_b2), J11.b2 (Pin_b2), J12.b2 (Pin_b2), J13.b2 (Pin_b2), J14.b2 (Pin_b2)
- net *IOT_WAIT: now also J10.a31 (Pin_a31), J11.a31 (Pin_a31), J12.a31 (Pin_a31), J13.a31 (Pin_a31), J14.a31 (Pin_a31)
- net *JMP_I_DETECT: now also J10.a27 (Pin_a27), J11.a27 (Pin_a27), J12.a27 (Pin_a27), J13.a27 (Pin_a27), J14.a27 (Pin_a27)
- net *LATCH_AC: now also J15.33 (Pin_33), J16.33 (Pin_33)
- net *LATCH_IR: now also J15.35 (Pin_35), J16.35 (Pin_35)
- net *LATCH_MA: now also J15.37 (Pin_37), J16.37 (Pin_37)
- net *LATCH_MB: now also J15.34 (Pin_34), J16.34 (Pin_34)
- net *LATCH_MQ: now also J15.32 (Pin_32), J16.32 (Pin_32)
- net *LATCH_PC: now also J15.36 (Pin_36), J16.36 (Pin_36)
- net *MEMM_ENABLE: now also J10.b23 (Pin_b23), J11.b23 (Pin_b23), J12.b23 (Pin_b23), J13.b23 (Pin_b23), J14.b23 (Pin_b23), J15.44 (Pin_44), J16.44 (Pin_44)
- net *PI_ENABLE: now also J10.b22 (Pin_b22), J11.b22 (Pin_b22), J12.b22 (Pin_b22), J13.b22 (Pin_b22), J14.b22 (Pin_b22), J15.46 (Pin_46), J16.46 (Pin_46)
- net *PROT_ENABLE: now also J10.b24 (Pin_b24), J11.b24 (Pin_b24), J12.b24 (Pin_b24), J13.b24 (Pin_b24), J14.b24 (Pin_b24)
- net *PTP_FLAG: now also J10.b19 (Pin_b19), J11.b19 (Pin_b19), J12.b19 (Pin_b19), J13.b19 (Pin_b19), J14.b19 (Pin_b19)
- net *PTP_TAPE: now also J10.b21 (Pin_b21), J11.b21 (Pin_b21), J12.b21 (Pin_b21), J13.b21 (Pin_b21), J14.b21 (Pin_b21)
- net *PTR_FLAG: now also J10.b18 (Pin_b18), J11.b18 (Pin_b18), J12.b18 (Pin_b18), J13.b18 (Pin_b18), J14.b18 (Pin_b18)
- net *PTR_TAPE: now also J10.b20 (Pin_b20), J11.b20 (Pin_b20), J12.b20 (Pin_b20), J13.b20 (Pin_b20), J14.b20 (Pin_b20)
- net *READ_IN_CLEAR: now also J10.a30 (Pin_a30), J11.a30 (Pin_a30), J12.a30 (Pin_a30), J13.a30 (Pin_a30), J14.a30 (Pin_a30)
- net *READ_IN_PULSE: now also J10.a29 (Pin_a29), J11.a29 (Pin_a29), J12.a29 (Pin_a29), J13.a29 (Pin_a29), J14.a29 (Pin_a29)
- net *RESET: now also J10.a21 (Pin_a21), J11.a21 (Pin_a21), J12.a21 (Pin_a21), J13.a21 (Pin_a21), J14.a21 (Pin_a21)
- net *SELECT_SWR: now also J15.29 (Pin_29), J16.29 (Pin_29)
- net +5V: now also J10.a32 (Pin_a32), J10.b1 (Pin_b1), J11.a32 (Pin_a32), J11.b1 (Pin_b1), J12.a32 (Pin_a32), J12.b1 (Pin_b1), J13.a32 (Pin_a32), J13.b1 (Pin_b1), J14.a32 (Pin_a32), J14.b1 (Pin_b1), J15.1 (Pin_1), J15.50 (Pin_50), J16.1 (Pin_1), J16.50 (Pin_50), R1.2, R2.2, R3.2, R4.2, R5.2
- net A_DEVICE0: now also J10.b3 (Pin_b3), J11.b3 (Pin_b3), J12.b3 (Pin_b3), J13.b3 (Pin_b3), J14.b3 (Pin_b3)
- net A_DEVICE1: now also J10.b4 (Pin_b4), J11.b4 (Pin_b4), J12.b4 (Pin_b4), J13.b4 (Pin_b4), J14.b4 (Pin_b4)
- net A_DEVICE2: now also J10.b5 (Pin_b5), J11.b5 (Pin_b5), J12.b5 (Pin_b5), J13.b5 (Pin_b5), J14.b5 (Pin_b5)
- net A_DEVICE3: now also J10.b6 (Pin_b6), J11.b6 (Pin_b6), J12.b6 (Pin_b6), J13.b6 (Pin_b6), J14.b6 (Pin_b6)
- net A_DEVICE4: now also J10.b7 (Pin_b7), J11.b7 (Pin_b7), J12.b7 (Pin_b7), J13.b7 (Pin_b7), J14.b7 (Pin_b7)
- net A_DEVICE5: now also J10.b8 (Pin_b8), J11.b8 (Pin_b8), J12.b8 (Pin_b8), J13.b8 (Pin_b8), J14.b8 (Pin_b8)
- net A_PULSE0: now also J10.b11 (Pin_b11), J11.b11 (Pin_b11), J12.b11 (Pin_b11), J13.b11 (Pin_b11), J14.b11 (Pin_b11)
- net A_PULSE1: now also J10.b12 (Pin_b12), J11.b12 (Pin_b12), J12.b12 (Pin_b12), J13.b12 (Pin_b12), J14.b12 (Pin_b12)
- net A_PULSE2: now also J10.b13 (Pin_b13), J11.b13 (Pin_b13), J12.b13 (Pin_b13), J13.b13 (Pin_b13), J14.b13 (Pin_b13)
- net A_SUBDEV0: now also J10.b9 (Pin_b9), J11.b9 (Pin_b9), J12.b9 (Pin_b9), J13.b9 (Pin_b9), J14.b9 (Pin_b9)
- net A_SUBDEV1: now also J10.b10 (Pin_b10), J11.b10 (Pin_b10), J12.b10 (Pin_b10), J13.b10 (Pin_b10), J14.b10 (Pin_b10)
- net CLK10: now also J15.31 (Pin_31), J16.31 (Pin_31)
- net CLK11: now also J15.30 (Pin_30), J16.30 (Pin_30)
- net CLK5: now also J10.a23 (Pin_a23)
- net CLK6: now also J11.a23 (Pin_a23)
- net CLK7: now also J12.a23 (Pin_a23)
- net CLK8: now also J13.a23 (Pin_a23)
- net CLK9: now also J14.a23 (Pin_a23)
- net FLAG_LINK: now also J15.47 (Pin_47), J16.47 (Pin_47)
- net FP0: now also J15.20 (Pin_20), J16.20 (Pin_20)
- net FP1: now also J15.21 (Pin_21), J16.21 (Pin_21)
- net FP2: now also J15.22 (Pin_22), J16.22 (Pin_22)
- net FP3: now also J15.23 (Pin_23), J16.23 (Pin_23)
- net GND: now also J10.a1 (Pin_a1), J10.b32 (Pin_b32), J11.a1 (Pin_a1), J11.b32 (Pin_b32), J12.a1 (Pin_a1), J12.b32 (Pin_b32), J13.a1 (Pin_a1), J13.a25 (Pin_a25), J13.b32 (Pin_b32), J14.a1 (Pin_a1), J14.a25 (Pin_a25), J14.b32 (Pin_b32), J15.24 (Pin_24), J15.25 (Pin_25), J15.26 (Pin_26), J15.27 (Pin_27), J16.24 (Pin_24), J16.25 (Pin_25), J16.26 (Pin_26), J16.27 (Pin_27), J17.1 (Pin_1), J18.1 (Pin_1), J19.1 (Pin_1), J20.1 (Pin_1), J21.1 (Pin_1)
- net HALT: now also J15.45 (Pin_45), J16.45 (Pin_45)
- net ID0: now also J10.a3 (Pin_a3), J11.a3 (Pin_a3), J12.a3 (Pin_a3), J13.a3 (Pin_a3), J14.a3 (Pin_a3)
- net ID1: now also J10.a4 (Pin_a4), J11.a4 (Pin_a4), J12.a4 (Pin_a4), J13.a4 (Pin_a4), J14.a4 (Pin_a4)
- net ID10: now also J10.a13 (Pin_a13), J11.a13 (Pin_a13), J12.a13 (Pin_a13), J13.a13 (Pin_a13), J14.a13 (Pin_a13)
- net ID11: now also J10.a14 (Pin_a14), J11.a14 (Pin_a14), J12.a14 (Pin_a14), J13.a14 (Pin_a14), J14.a14 (Pin_a14)
- net ID12: now also J10.a15 (Pin_a15), J11.a15 (Pin_a15), J12.a15 (Pin_a15), J13.a15 (Pin_a15), J14.a15 (Pin_a15)
- net ID13: now also J10.a16 (Pin_a16), J11.a16 (Pin_a16), J12.a16 (Pin_a16), J13.a16 (Pin_a16), J14.a16 (Pin_a16)
- net ID14: now also J10.a17 (Pin_a17), J11.a17 (Pin_a17), J12.a17 (Pin_a17), J13.a17 (Pin_a17), J14.a17 (Pin_a17)
- net ID15: now also J10.a18 (Pin_a18), J11.a18 (Pin_a18), J12.a18 (Pin_a18), J13.a18 (Pin_a18), J14.a18 (Pin_a18)
- net ID16: now also J10.a19 (Pin_a19), J11.a19 (Pin_a19), J12.a19 (Pin_a19), J13.a19 (Pin_a19), J14.a19 (Pin_a19)
- net ID17: now also J10.a20 (Pin_a20), J11.a20 (Pin_a20), J12.a20 (Pin_a20), J13.a20 (Pin_a20), J14.a20 (Pin_a20)
- net ID2: now also J10.a5 (Pin_a5), J11.a5 (Pin_a5), J12.a5 (Pin_a5), J13.a5 (Pin_a5), J14.a5 (Pin_a5)
- net ID3: now also J10.a6 (Pin_a6), J11.a6 (Pin_a6), J12.a6 (Pin_a6), J13.a6 (Pin_a6), J14.a6 (Pin_a6)
- net ID4: now also J10.a7 (Pin_a7), J11.a7 (Pin_a7), J12.a7 (Pin_a7), J13.a7 (Pin_a7), J14.a7 (Pin_a7)
- net ID5: now also J10.a8 (Pin_a8), J11.a8 (Pin_a8), J12.a8 (Pin_a8), J13.a8 (Pin_a8), J14.a8 (Pin_a8)
- net ID6: now also J10.a9 (Pin_a9), J11.a9 (Pin_a9), J12.a9 (Pin_a9), J13.a9 (Pin_a9), J14.a9 (Pin_a9)
- net ID7: now also J10.a10 (Pin_a10), J11.a10 (Pin_a10), J12.a10 (Pin_a10), J13.a10 (Pin_a10), J14.a10 (Pin_a10)
- net ID8: now also J10.a11 (Pin_a11), J11.a11 (Pin_a11), J12.a11 (Pin_a11), J13.a11 (Pin_a11), J14.a11 (Pin_a11)
- net ID9: now also J10.a12 (Pin_a12), J11.a12 (Pin_a12), J12.a12 (Pin_a12), J13.a12 (Pin_a12), J14.a12 (Pin_a12)
- net NEXT_BANK0: now also J15.49 (Pin_49), J16.49 (Pin_49)
- net NEXT_BANK1: now also J15.48 (Pin_48), J16.48 (Pin_48)
- net REQ_ADDR: now also J10.a24 (Pin_a24), J11.a24 (Pin_a24), J12.a24 (Pin_a24), J13.a24 (Pin_a24), J14.a24 (Pin_a24)
- net SC0: now also J15.43 (Pin_43), J16.43 (Pin_43)
- net SC1: now also J15.42 (Pin_42), J16.42 (Pin_42)
- net SC2: now also J15.41 (Pin_41), J16.41 (Pin_41)
- net SC3: now also J15.40 (Pin_40), J16.40 (Pin_40)
- net SC4: now also J15.39 (Pin_39), J16.39 (Pin_39)
- net SC5: now also J15.38 (Pin_38), J16.38 (Pin_38)
- net *DRQ_GRANT0: now reaches J9.a25 (Pin_a25)
- new net: J18.2 (Pin_2), R2.1
- new net: J19.2 (Pin_2), R3.1
- new net: J17.2 (Pin_2), R1.1
- new net: J21.2 (Pin_2), R5.1
- new net: J20.2 (Pin_2), R4.1
- new net *CHAN_REQ1: J10.b27 (Pin_b27)
- new net *CHAN_REQ2: J11.b27 (Pin_b27)
- new net *CHAN_REQ3: J12.b27 (Pin_b27)
- new net *DMA_REQ1: J10.b26 (Pin_b26)
- new net *DMA_REQ2: J11.b26 (Pin_b26)
- new net *DMA_REQ3: J12.b26 (Pin_b26)
- new net *DRQ_GRANT1: J10.a25 (Pin_a25)
- new net *DRQ_GRANT2: J11.a25 (Pin_a25)
- new net *DRQ_GRANT3: J12.a25 (Pin_a25)
- new net BD0: J15.2 (Pin_2), J16.2 (Pin_2)
- new net BD1: J15.3 (Pin_3), J16.3 (Pin_3)
- new net BD10: J15.12 (Pin_12), J16.12 (Pin_12)
- new net BD11: J15.13 (Pin_13), J16.13 (Pin_13)
- new net BD12: J15.14 (Pin_14), J16.14 (Pin_14)
- new net BD13: J15.15 (Pin_15), J16.15 (Pin_15)
- new net BD14: J15.16 (Pin_16), J16.16 (Pin_16)
- new net BD15: J15.17 (Pin_17), J16.17 (Pin_17)
- new net BD16: J15.18 (Pin_18), J16.18 (Pin_18)
- new net BD17: J15.19 (Pin_19), J16.19 (Pin_19)
- new net BD2: J15.4 (Pin_4), J16.4 (Pin_4)
- new net BD3: J15.5 (Pin_5), J16.5 (Pin_5)
- new net BD4: J15.6 (Pin_6), J16.6 (Pin_6)
- new net BD5: J15.7 (Pin_7), J16.7 (Pin_7)
- new net BD6: J15.8 (Pin_8), J16.8 (Pin_8)
- new net BD7: J15.9 (Pin_9), J16.9 (Pin_9)
- new net BD8: J15.10 (Pin_10), J16.10 (Pin_10)
- new net BD9: J15.11 (Pin_11), J16.11 (Pin_11)
- new net SYNC_CLK: J15.28 (Pin_28), J16.28 (Pin_28)
- no-connect marks 35 -> 49
Other:
- moved on the sheet: J9

Commit message: Continue work on backplane
Parts:
- added R10, R11, R12, R13, R14, R15, R16, R17, R18, R19, R20, R21, R22, R23, R24, R25, R26, R27, R6, R7, R8, R9: 4.7K, Resistor_THT:R_Axial_DIN0207_L6.3mm_D2.5mm_P7.62mm_Horizontal, symbol Device:R
- added U10, U11, U12, U20: 74LS377, symbol 74xx:74LS377
- added U13, U14, U15, U17, U18, U19: 74LS244, symbol 74xx:74LS244
- added U16: 74LS04, symbol 74xx:74LS04
- added U21: 74LS148, symbol 74xx:74LS148
- added U22: 74LS153, symbol 74xx:74LS153
- added U3, U4: 74LS74, symbol 74xx:74LS74
- added U5: 74LS32, symbol 74xx:74LS32
- added U6: 74LS08, symbol 74xx:74LS08
- added U7, U8, U9: 74LS245, symbol 74xx:74LS245
Connections:
- net *CAF: now also U6.11
- net *CAF_REQ: now also R14.1, U6.13
- net *CHAN_REQ: now also U22.7 (Za)
- net *CHAN_REQ0: now also U20.18 (D7)
- net *CHAN_REQ1: now also U20.14 (D5)
- net *CHAN_REQ2: now also U20.8 (D3)
- net *CHAN_REQ3: now also U20.4 (D1)
- net *DMA_REQ: now also U22.9 (Zb)
- net *DMA_REQ0: now also U20.17 (D6)
- net *DMA_REQ1: now also U20.13 (D4)
- net *DMA_REQ2: now also U20.7 (D2)
- net *DMA_REQ3: now also U20.3 (D0)
- net *DRQ_GRANT: now also U16.3
- net *EXTERNAL: now also R27.1, U16.1
- net *LATCH_WRTBK: now also U10.1 (~{E}), U11.1 (~{E}), U12.1 (~{E})
- net *READ_IN_CLEAR: now also U5.8
- net *READ_IN_PULSE: now also U5.10
- net *RESET: now also U6.8
- net *SELECT_EXTRN: now also U17.1 (OEa), U17.19 (OEb), U18.1 (OEa), U18.19 (OEb), U19.1 (OEa), U19.19 (OEb)
- net *SELECT_SWR: now also U7.1 (A->B), U8.1 (A->B), U9.1 (A->B)
- net +5V: now also R10.2, R11.1, R12.2, R13.1, R14.2, R15.2, R16.2, R17.2, R18.2, R19.2, R20.2, R21.1, R22.1, R23.1, R24.1, R25.1, R26.1, R27.2, R6.2, R7.1, R8.2, R9.1, U10.20 (VCC), U11.20 (VCC), U12.20 (VCC), U13.20 (VCC), U14.20 (VCC), U15.20 (VCC), U17.20 (VCC), U18.20 (VCC), U19.20 (VCC), U20.20 (VCC), U21.16 (VCC), U22.16 (VCC), U7.20 (VCC), U8.20 (VCC), U9.20 (VCC)
- net BD0: now also U7.18 (B0)
- net BD1: now also U7.17 (B1)
- net BD10: now also U8.16 (B2)
- net BD11: now also U8.15 (B3)
- net BD12: now also U8.14 (B4)
- net BD13: now also U8.13 (B5)
- net BD14: now also U8.12 (B6)
- net BD15: now also U8.11 (B7)
- net BD16: now also U9.18 (B0)
- net BD17: now also U9.17 (B1)
- net BD2: now also U7.16 (B2)
- net BD3: now also U7.15 (B3)
- net BD4: now also U7.14 (B4)
- net BD5: now also U7.13 (B5)
- net BD6: now also U7.12 (B6)
- net BD7: now also U7.11 (B7)
- net BD8: now also U8.18 (B0)
- net BD9: now also U8.17 (B1)
- net CLK10: now also U10.11 (CP), U11.11 (CP), U12.11 (CP), U20.11 (CP)
- net CTL_CONST: now also U16.5
- net D0: now also U10.3 (D0), U17.2 (I0a), U7.2 (A0)
- net D1: now also U10.4 (D1), U17.4 (I1a), U7.3 (A1)
- net D10: now also U11.7 (D2), U18.6 (I2a), U8.4 (A2)
- net D11: now also U11.8 (D3), U18.8 (I3a), U8.5 (A3)
- net D12: now also U11.13 (D4), U18.11 (I0b), U8.6 (A4)
- net D13: now also U11.14 (D5), U18.13 (I1b), U8.7 (A5)
- net D14: now also U11.17 (D6), U18.15 (I2b), U8.8 (A6)
- net D15: now also U11.18 (D7), U18.17 (I3b), U8.9 (A7)
- net D16: now also U12.3 (D0), U19.2 (I0a), U9.2 (A0)
- net D17: now also U12.4 (D1), U19.4 (I1a), U9.3 (A1)
- net D2: now also U10.7 (D2), U17.6 (I2a), U7.4 (A2)
- net D3: now also U10.8 (D3), U17.8 (I3a), U7.5 (A3)
- net D4: now also U10.13 (D4), U17.11 (I0b), U7.6 (A4)
- net D5: now also U10.14 (D5), U17.13 (I1b), U7.7 (A5)
- net D6: now also U10.17 (D6), U17.15 (I2b), U7.8 (A6)
- net D7: now also U10.18 (D7), U17.17 (I3b), U7.9 (A7)
- net D8: now also U11.3 (D0), U18.2 (I0a), U8.2 (A0)
- net D9: now also U11.4 (D1), U18.4 (I1a), U8.3 (A1)
- net GND: now also U10.10 (GND), U11.10 (GND), U12.10 (GND), U12.13 (D4), U12.14 (D5), U12.17 (D6), U12.18 (D7), U12.7 (D2), U12.8 (D3), U13.10 (GND), U14.10 (GND), U15.10 (GND), U17.10 (GND), U18.10 (GND), U19.10 (GND), U19.12 (O3a), U19.14 (O2a), U19.3 (O3b), U19.5 (O2b), U19.7 (O1b), U19.9 (O0b), U20.10 (GND), U21.5 (EI), U21.8 (GND), U22.1 (Ea), U22.15 (Eb), U22.8 (GND), U7.10 (GND), U7.19 (CE), U8.10 (GND), U8.19 (CE), U9.10 (GND), U9.19 (CE); no longer J15.27 (Pin_27), J16.27 (Pin_27)
- net ID0: now also U13.18 (O0a), U17.18 (O0a)
- net ID1: now also U13.16 (O1a), U17.16 (O1a)
- net ID10: now also U14.14 (O2a), U18.14 (O2a)
- net ID11: now also U14.12 (O3a), U18.12 (O3a)
- net ID12: now also U14.9 (O0b), U18.9 (O0b)
- net ID13: now also U14.7 (O1b), U18.7 (O1b)
- net ID14: now also U14.5 (O2b), U18.5 (O2b)
- net ID15: now also U14.3 (O3b), U18.3 (O3b)
- net ID16: now also U15.18 (O0a), U19.18 (O0a)
- net ID17: now also U15.16 (O1a), U19.16 (O1a)
- net ID2: now also U13.14 (O2a), U17.14 (O2a)
- net ID3: now also U13.12 (O3a), U17.12 (O3a)
- net ID4: now also U13.9 (O0b), U17.9 (O0b)
- net ID5: now also U13.7 (O1b), U17.7 (O1b)
- net ID6: now also U13.5 (O2b), U17.5 (O2b)
- net ID7: now also U13.3 (O3b), U17.3 (O3b)
- net ID8: now also U14.18 (O0a), U18.18 (O0a)
- net ID9: now also U14.16 (O1a), U18.16 (O1a)
- net SYNC_CLK: now also J15.27 (Pin_27), J16.27 (Pin_27), U1.18 (O0a), U5.2; no longer J15.28 (Pin_28), J16.28 (Pin_28)
- net at J18.2 (Pin_2), R2.1: now also U3.12 (D)
- net at U1.11 (I0b), U1.13 (I1b), U1.15 (I2b)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: now also U2.2 (I0a), U2.4 (I1a)
- net at U1.14 (O2a), U2.11 (I0b), U2.13 (I1b)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: no longer U2.2 (I0a), U2.4 (I1a)
- net at U1.4 (I1a), U1.6 (I2a), U1.8 (I3a): now also U6.6; no longer U1.18 (O0a)
- net at U1.2 (I0a): now also X1.8 (OUT)
- net at J19.2 (Pin_2), R3.1: now also U4.2 (D)
- net at J17.2 (Pin_2), R1.1: now also U3.2 (D)
- net at J21.2 (Pin_2), R5.1: now also U4.12 (D)
- net at J20.2 (Pin_2), R4.1: now also U6.10, U6.9
- new net: R12.1, U4.13 (~{R})
- new net: U16.4, U20.1 (~{E})
- new net: U5.3, U6.4
- new net: U6.3, U6.5
- new net: U10.12 (Q4), U13.11 (I0b)
- new net: U10.15 (Q5), U13.13 (I1b)
- new net: U10.16 (Q6), U13.15 (I2b)
- new net: U10.19 (Q7), U13.17 (I3b)
- new net: U10.2 (Q0), U13.2 (I0a)
- new net: U10.5 (Q1), U13.4 (I1a)
- new net: U10.6 (Q2), U13.6 (I2a)
- new net: U10.9 (Q3), U13.8 (I3a)
- new net: U20.16 (Q6), U21.3 (I6), U22.10 (I0b)
- new net: U20.12 (Q4), U21.1 (I4), U22.11 (I1b)
- new net: U20.6 (Q2), U21.12 (I2), U22.12 (I2b)
- new net: U20.2 (Q0), U21.10 (IO), U22.13 (I3b)
- new net: U21.7 (S1), U22.14 (S0)
- new net: U21.6 (S2), U22.2 (S1)
- new net: U20.5 (Q1), U21.11 (I1), U22.3 (I3a)
- new net: U20.9 (Q3), U21.13 (I3), U22.4 (I2a)
- new net: U20.15 (Q5), U21.2 (I5), U22.5 (I1a)
- new net: U20.19 (Q7), U21.4 (I7), U22.6 (I0a)
- new net: U13.1 (OEa), U13.19 (OEb), U14.1 (OEa), U14.19 (OEb), U15.1 (OEa), U15.19 (OEb), U16.2
- new net: U12.12 (Q4), U15.11 (I0b)
- new net: U12.15 (Q5), U15.13 (I1b)
- new net: U12.16 (Q6), U15.15 (I2b)
- new net: U12.19 (Q7), U15.17 (I3b)
- new net: U12.2 (Q0), U15.2 (I0a)
- new net: U12.5 (Q1), U15.4 (I1a)
- new net: U12.6 (Q2), U15.6 (I2a)
- new net: U12.9 (Q3), U15.8 (I3a)
- new net: R13.2, U4.10 (~{S})
- new net: R18.1, U9.7 (A5)
- new net: R15.1, U9.4 (A2)
- new net: U16.6, U5.9
- new net: R21.2, U9.16 (B2)
- new net: R9.2, U3.10 (~{S})
- new net: U3.5 (Q), U5.1
- new net: R26.2, U9.11 (B7)
- new net: R10.1, U4.1 (~{R})
- new net: R11.2, U4.4 (~{S})
- new net: U3.9 (Q), U6.1
- new net: U5.6, U6.2
- new net: U4.5 (Q), U5.4
- new net: U11.12 (Q4), U14.11 (I0b)
- new net: U11.15 (Q5), U14.13 (I1b)
- new net: U11.16 (Q6), U14.15 (I2b)
- new net: U11.19 (Q7), U14.17 (I3b)
- new net: U11.2 (Q0), U14.2 (I0a)
- new net: U11.5 (Q1), U14.4 (I1a)
- new net: U11.6 (Q2), U14.6 (I2a)
- new net: U11.9 (Q3), U14.8 (I3a)
- new net: R25.2, U9.12 (B6)
- new net: R8.1, U3.13 (~{R})
- new net: R7.2, U3.4 (~{S})
- new net: R24.2, U9.13 (B5)
- new net: R23.2, U9.14 (B4)
- new net: R22.2, U9.15 (B3)
- new net: R16.1, U9.5 (A3)
- new net: R17.1, U9.6 (A4)
- new net: R19.1, U9.8 (A6)
- new net: R20.1, U9.9 (A7)
- new net: R6.1, U3.1 (~{R})
- new net: U4.9 (Q), U6.12
- new net DELAY_CLK: J15.28 (Pin_28), J16.28 (Pin_28), U3.11 (C), U3.3 (C), U4.11 (C), U4.3 (C), U5.5
- no-connect marks 49 -> 68
Other:
- moved on the sheet: J15, J16, J18, J19, J20, J21, R2, R3, R4, R5, U1, U2
