File: kicad/Backplane/Backplane.kicad_pcb (KiCad board)
At the start: 2 copper layers, 129 parts, among them J1 Control Connector, J10 I/O Connector, J11 I/O Connector, J12 I/O Connector, J13 I/O Connector, J14 I/O Connector, J15 Front Panel Connector, J16 Front Panel Connector, J17 Run, J18 Clock, J19 Rept, J2 Data Connector, J20 Reset, J21 I/O Reset, J22 Power, J23 Power LED, J3 Control Connector, J4 Data Connector, J5 Control Connector, J6 Data Connector, J7 Control Connector, J8 Data Connector, J9 I/O Connector, U1 74LS244, U10 74LS377, U11 74LS377, U12 74LS377, U13 74LS244, U14 74LS244, U15 74LS244, U16 74LS04, U17 74LS244, U18 74LS244, U19 74LS244, U2 74LS244, U20 74LS377, U21 74LS148, U22 74LS253, U23 74LS139, U24 74LS244, U25 74LS32, U3 74LS74, U4 74LS74, U5 74LS32, U6 74LS08, U7 74LS245, U8 74LS245, U9 74LS245, X1 4 Mhz Oscillator

Commit message: Continue work on backplane
Parts:
- moved J16 513.4 mm to (178.5, 305.7), turned to 90 degrees
- moved J15 509.2 mm to (178.5, 317.7), turned to 90 degrees
- moved J9 494.6 mm to (54.3, 22.3)
- moved J10 470.4 mm to (89.2, 22.2)
- moved J11 446.2 mm to (124.1, 22.3)
- moved J3 433.8 mm to (89.2, 234.9)
- moved J12 422.0 mm to (159.1, 22.3)
- moved J5 421.4 mm to (124.1, 234.9)
- moved J4 412.4 mm to (89.2, 131.4)
- moved J7 409.2 mm to (159.1, 234.9)
- moved J6 399.1 mm to (124.1, 131.4)
- moved J13 397.8 mm to (194.0, 22.3)
- moved J8 385.8 mm to (159.1, 131.4)
- moved J14 373.6 mm to (228.9, 22.3)
- moved C1 268.9 mm to (332.4, 185.9)
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
Commit message: Adjust backplane spacing
Parts:
- moved C1 18.6 mm to (332.3, 204.5)
- moved C10 18.6 mm to (340.4, 204.5)
- moved C15 18.6 mm to (340.4, 224.7)
- moved C19 18.6 mm to (348.6, 204.5)
- moved C24 18.6 mm to (348.6, 224.7)
- moved C26 18.6 mm to (342.2, 178.4)
- moved C6 18.6 mm to (332.3, 224.7)
- moved R15 18.6 mm to (289.2, 198.2)
- moved R20 18.6 mm to (289.2, 218.5)
- moved R26 18.6 mm to (300.0, 198.2)
- moved R31 18.6 mm to (300.0, 218.5)
- moved R37 18.6 mm to (310.8, 198.2)
- moved R4 18.6 mm to (278.4, 198.2)
- moved R42 18.6 mm to (310.8, 218.5)
- moved R48 18.6 mm to (321.5, 198.2)
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
Commit message: Continue backplane layout
Parts:
- moved R47 274.7 mm to (62.9, 101.6)
- moved R46 274.6 mm to (62.9, 97.8)
- moved R49 245.3 mm to (97.8, 101.6)
- moved R48 245.2 mm to (97.8, 97.8)
- moved J17 220.1 mm to (174.6, 339.1), turned to 90 degrees
- moved R51 217.9 mm to (132.7, 101.6)
- moved R50 217.8 mm to (132.7, 97.8)
- moved J18 214.3 mm to (187.3, 339.1), turned to 90 degrees
- moved J19 208.8 mm to (200.0, 339.1), turned to 90 degrees
- moved J20 203.4 mm to (212.7, 339.1), turned to 90 degrees
- moved J21 198.1 mm to (225.4, 339.1), turned to 90 degrees
- moved R53 193.2 mm to (167.6, 101.6)
- moved J23 193.1 mm to (238.1, 339.1), turned to 90 degrees
- moved R52 193.1 mm to (167.6, 97.8)
- moved C3 184.2 mm to (178.4, 313.7), turned to 180 degrees
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Other:
- board outline added: 200 x 321.3 mm

Commit message: Continue work on backplane
Parts:
- moved R38 21.6 mm to (210.8, 38.1)
- moved R39 20.3 mm to (210.8, 43.2)
- moved R40 19.1 mm to (210.8, 48.3)
- moved R41 17.8 mm to (210.8, 53.3)
- moved R42 16.5 mm to (210.8, 58.4)
- moved R43 15.2 mm to (210.8, 63.5)
- moved R44 14.0 mm to (210.8, 68.6)
- moved R45 12.7 mm to (210.8, 73.7)
- moved R37 11.4 mm to (210.8, 78.7)
- moved R36 10.2 mm to (210.8, 83.8)
- moved R35 7.62 mm to (210.8, 89.5)
- moved R34 6.35 mm to (210.8, 94.6)
- moved R33 5.08 mm to (210.8, 99.7)
- moved R32 3.81 mm to (210.8, 104.8)
- moved R31 2.54 mm to (210.8, 109.9)
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Changed lines of the file:
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@@
   )
   (footprint "Resistor_THT:R_Axial_DIN0207_L6.3mm_D2.5mm_P7.62mm_Horizontal" (layer "F.Cu")
-    (at 210.82 82.55)
+    (at 210.82 68.58)
     (descr "Resistor, Axial_DIN0207 series, Axial, Horizontal, pin pitch=7.62mm, 0.25W = 1/4W, length*diameter=6.3*2.5mm^2, http://cdn-reichelt.de/documents/datenblatt/B400/1_4W%23YAG.pdf")
     (tags "Resistor Axial_DIN0207 series Axial Horizontal pin pitch 7.62mm 0.25W = 1/4W length 6.3mm diameter 2.5mm")
@@
   )
   (footprint "Resistor_THT:R_Axial_DIN0207_L6.3mm_D2.5mm_P7.62mm_Horizontal" (layer "F.Cu")
-    (at 210.82 100.965)
+    (at 210.82 94.615)
     (descr "Resistor, Axial_DIN0207 series, Axial, Horizontal, pin pitch=7.62mm, 0.25W = 1/4W, length*diameter=6.3*2.5mm^2, http://cdn-reichelt.de/documents/datenblatt/B400/1_4W%23YAG.pdf")
     (tags "Resistor Axial_DIN0207 series Axial Horizontal pin pitch 7.62mm 0.25W = 1/4W length 6.3mm diameter 2.5mm")
@@
   )
   (footprint "Resistor_THT:R_Axial_DIN0207_L6.3mm_D2.5mm_P7.62mm_Horizontal" (layer "F.Cu")
-    (at 210.82 104.775)
+    (at 210.82 99.695)
     (descr "Resistor, Axial_DIN0207 series, Axial, Horizontal, pin pitch=7.62mm, 0.25W = 1/4W, length*diameter=6.3*2.5mm^2, http://cdn-reichelt.de/documents/datenblatt/B400/1_4W%23YAG.pdf")
     (tags "Resistor Axial_DIN0207 series Axial Horizontal pin pitch 7.62mm 0.25W = 1/4W length 6.3mm diameter 2.5mm")
@@
   )
   (footprint "Resistor_THT:R_Axial_DIN0207_L6.3mm_D2.5mm_P7.62mm_Horizontal" (layer "F.Cu")
-    (at 210.82 74.93)
+    (at 210.82 58.42)
     (descr "Resistor, Axial_DIN0207 series, Axial, Horizontal, pin pitch=7.62mm, 0.25W = 1/4W, length*diameter=6.3*2.5mm^2, http://cdn-reichelt.de/documents/datenblatt/B400/1_4W%23YAG.pdf")
     (tags "Resistor Axial_DIN0207 series Axial Horizontal pin pitch 7.62mm 0.25W = 1/4W length 6.3mm diameter 2.5mm")
@@
   )
   (footprint "Resistor_THT:R_Axial_DIN0207_L6.3mm_D2.5mm_P7.62mm_Horizontal" (layer "F.Cu")
-    (at 210.82 97.155)
+    (at 210.82 89.535)
     (descr "Resistor, Axial_DIN0207 series, Axial, Horizontal, pin pitch=7.62mm, 0.25W = 1/4W, length*diameter=6.3*2.5mm^2, http://cdn-reichelt.de/documents/datenblatt/B400/1_4W%23YAG.pdf")
     (tags "Resistor Axial_DIN0207 series Axial Horizontal pin pitch 7.62mm 0.25W = 1/4W length 6.3mm diameter 2.5mm")
@@
   )
   (footprint "Resistor_THT:R_Axial_DIN0207_L6.3mm_D2.5mm_P7.62mm_Horizontal" (layer "F.Cu")
-    (at 210.82 112.395)
+    (at 210.82 109.855)
     (descr "Resistor, Axial_DIN0207 series, Axial, Horizontal, pin pitch=7.62mm, 0.25W = 1/4W, length*diameter=6.3*2.5mm^2, http://cdn-reichelt.de/documents/datenblatt/B400/1_4W%23YAG.pdf")
     (tags "Resistor Axial_DIN0207 series Axial Horizontal pin pitch 7.62mm 0.25W = 1/4W length 6.3mm diameter 2.5mm")
@@
   )
   (footprint "Resistor_THT:R_Axial_DIN0207_L6.3mm_D2.5mm_P7.62mm_Horizontal" (layer "F.Cu")
-    (at 210.82 93.98)
+    (at 210.82 83.82)
     (descr "Resistor, Axial_DIN0207 series, Axial, Horizontal, pin pitch=7.62mm, 0.25W = 1/4W, length*diameter=6.3*2.5mm^2, http://cdn-reichelt.de/documents/datenblatt/B400/1_4W%23YAG.pdf")
     (tags "Resistor Axial_DIN0207 series Axial Horizontal pin pitch 7.62mm 0.25W = 1/4W length 6.3mm diameter 2.5mm")
@@
   )
   (footprint "Resistor_THT:R_Axial_DIN0207_L6.3mm_D2.5mm_P7.62mm_Horizontal" (layer "F.Cu")
-    (at 210.82 116.205)
+    (at 210.82 114.935)
     (descr "Resistor, Axial_DIN0207 series, Axial, Horizontal, pin pitch=7.62mm, 0.25W = 1/4W, length*diameter=6.3*2.5mm^2, http://cdn-reichelt.de/documents/datenblatt/B400/1_4W%23YAG.pdf")
     (tags "Resistor Axial_DIN0207 series Axial Horizontal pin pitch 7.62mm 0.25W = 1/4W length 6.3mm diameter 2.5mm")
@@
   )
   (footprint "Resistor_THT:R_Axial_DIN0207_L6.3mm_D2.5mm_P7.62mm_Horizontal" (layer "F.Cu")
-    (at 210.82 67.31)
+    (at 210.82 48.26)
     (descr "Resistor, Axial_DIN0207 series, Axial, Horizontal, pin pitch=7.62mm, 0.25W = 1/4W, length*diameter=6.3*2.5mm^2, http://cdn-reichelt.de/documents/datenblatt/B400/1_4W%23YAG.pdf")
     (tags "Resistor Axial_DIN0207 series Axial Horizontal pin pitch 7.62mm 0.25W = 1/4W length 6.3mm diameter 2.5mm")
@@
   )
   (footprint "Resistor_THT:R_Axial_DIN0207_L6.3mm_D2.5mm_P7.62mm_Horizontal" (layer "F.Cu")
-    (at 210.82 90.17)
+    (at 210.82 78.74)
     (descr "Resistor, Axial_DIN0207 series, Axial, Horizontal, pin pitch=7.62mm, 0.25W = 1/4W, length*diameter=6.3*2.5mm^2, http://cdn-reichelt.de/documents/datenblatt/B400/1_4W%23YAG.pdf")
     (tags "Resistor Axial_DIN0207 series Axial Horizontal pin pitch 7.62mm 0.25W = 1/4W length 6.3mm diameter 2.5mm")
@@
   )
   (footprint "Resistor_THT:R_Axial_DIN0207_L6.3mm_D2.5mm_P7.62mm_Horizontal" (layer "F.Cu")
-    (at 210.82 108.585)
+    (at 210.82 104.775)
     (descr "Resistor, Axial_DIN0207 series, Axial, Horizontal, pin pitch=7.62mm, 0.25W = 1/4W, length*diameter=6.3*2.5mm^2, http://cdn-reichelt.de/documents/datenblatt/B400/1_4W%23YAG.pdf")
     (tags "Resistor Axial_DIN0207 series Axial Horizontal pin pitch 7.62mm 0.25W = 1/4W length 6.3mm diameter 2.5mm")
@@
   )
   (footprint "Resistor_THT:R_Axial_DIN0207_L6.3mm_D2.5mm_P7.62mm_Horizontal" (layer "F.Cu")
-    (at 210.82 71.12)
+    (at 210.82 53.34)
     (descr "Resistor, Axial_DIN0207 series, Axial, Horizontal, pin pitch=7.62mm, 0.25W = 1/4W, length*diameter=6.3*2.5mm^2, http://cdn-reichelt.de/documents/datenblatt/B400/1_4W%23YAG.pdf")
     (tags "Resistor Axial_DIN0207 series Axial Horizontal pin pitch 7.62mm 0.25W = 1/4W length 6.3mm diameter 2.5mm")
@@
   )
   (footprint "Resistor_THT:R_Axial_DIN0207_L6.3mm_D2.5mm_P7.62mm_Horizontal" (layer "F.Cu")
-    (at 210.82 78.74)
+    (at 210.82 63.5)
     (descr "Resistor, Axial_DIN0207 series, Axial, Horizontal, pin pitch=7.62mm, 0.25W = 1/4W, length*diameter=6.3*2.5mm^2, http://cdn-reichelt.de/documents/datenblatt/B400/1_4W%23YAG.pdf")
     (tags "Resistor Axial_DIN0207 series Axial Horizontal pin pitch 7.62mm 0.25W = 1/4W length 6.3mm diameter 2.5mm")
@@
   )
   (footprint "Resistor_THT:R_Axial_DIN0207_L6.3mm_D2.5mm_P7.62mm_Horizontal" (layer "F.Cu")
-    (at 210.82 63.5)
+    (at 210.82 43.18)
     (descr "Resistor, Axial_DIN0207 series, Axial, Horizontal, pin pitch=7.62mm, 0.25W = 1/4W, length*diameter=6.3*2.5mm^2, http://cdn-reichelt.de/documents/datenblatt/B400/1_4W%23YAG.pdf")
     (tags "Resistor Axial_DIN0207 series Axial Horizontal pin pitch 7.62mm 0.25W = 1/4W length 6.3mm diameter 2.5mm")
@@
   )
   (footprint "Resistor_THT:R_Axial_DIN0207_L6.3mm_D2.5mm_P7.62mm_Horizontal" (layer "F.Cu")
-    (at 210.82 59.69)
+    (at 210.82 38.1)
     (descr "Resistor, Axial_DIN0207 series, Axial, Horizontal, pin pitch=7.62mm, 0.25W = 1/4W, length*diameter=6.3*2.5mm^2, http://cdn-reichelt.de/documents/datenblatt/B400/1_4W%23YAG.pdf")
     (tags "Resistor Axial_DIN0207 series Axial Horizontal pin pitch 7.62mm 0.25W = 1/4W length 6.3mm diameter 2.5mm")
@@
   )
   (footprint "Resistor_THT:R_Axial_DIN0207_L6.3mm_D2.5mm_P7.62mm_Horizontal" (layer "F.Cu")
-    (at 210.82 86.36)
+    (at 210.82 73.66)
     (descr "Resistor, Axial_DIN0207 series, Axial, Horizontal, pin pitch=7.62mm, 0.25W = 1/4W, length*diameter=6.3*2.5mm^2, http://cdn-reichelt.de/documents/datenblatt/B400/1_4W%23YAG.pdf")
     (tags "Resistor Axial_DIN0207 series Axial Horizontal pin pitch 7.62mm 0.25W = 1/4W length 6.3mm diameter 2.5mm")

Commit message: Add mounting holes
Parts:
- moved J22 8.41 mm to (242.0, 153.0)
Changed lines of the file:
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@@
   )
   (footprint "Connector_TE-Connectivity:TE_MATE-N-LOK_350211-1_1x04_P5.08mm_Vertical" (layer "F.Cu")
-    (at 233.68 154.305 90)
+    (at 241.995 153.035 90)
     (descr "https://www.te.com/commerce/DocumentDelivery/DDEController?Action=showdoc&DocId=Customer+Drawing%7F350211%7FU5%7Fpdf%7FEnglish%7FENG_CD_350211_U5.pdf%7F350211-1")
     (tags "connector TE MATE-N-LOK top entry ATA PATA IDE 5.25 inch floppy drive power")

Commit message: Route address front panel
Parts:
- added H1: MountingHole, MountingHole:MountingHole_2.2mm_M2_Pad, F.Cu at (64.1, 25.4)
- added H2: MountingHole, MountingHole:MountingHole_2.2mm_M2_Pad, F.Cu at (116.8, 25.4)
- added H3: MountingHole, MountingHole:MountingHole_2.2mm_M2_Pad, F.Cu at (168.9, 25.4)
- added H4: MountingHole, MountingHole:MountingHole_2.2mm_M2_Pad, F.Cu at (245.1, 25.4)
- added H5: MountingHole, MountingHole:MountingHole_2.2mm_M2_Pad, F.Cu at (245.1, 339.1)
- added H6: MountingHole, MountingHole:MountingHole_2.2mm_M2_Pad, F.Cu at (151.8, 339.1)
- added H7: MountingHole, MountingHole:MountingHole_2.2mm_M2_Pad, F.Cu at (116.8, 339.1)
- added H8: MountingHole, MountingHole:MountingHole_2.2mm_M2_Pad, F.Cu at (64.1, 339.1)
- moved J23 3.17 mm to (234.9, 339.1)
- moved J21 2.53 mm to (222.9, 339.1)
- moved J20 1.90 mm to (210.8, 339.1)
- moved J19 1.27 mm to (198.8, 339.1)
- moved J18 0.63 mm to (186.7, 339.1)
Other:
- board text added: "Gavin Tersteeg, 2026"
- board text added: "JLCJLCJLCJLC"
- board text added: "RDP-9A-BKP-0"

Commit message: Continue work on routing
Routing:
- net GND: track 0.00 -> 1958.8 mm
- net +5V: track 0.00 -> 1865.8 mm, vias 0 -> 2
- net /*PI_ENABLE: track 0.00 -> 615.4 mm
- net /*MEMM_ENABLE: track 0.00 -> 605.0 mm
- net /*CAF: track 0.00 -> 603.1 mm, vias 0 -> 2
- net /*IOT_SKIP: track 0.00 -> 576.6 mm
- net /*RESET: track 0.00 -> 574.3 mm, vias 0 -> 2
- net /*READ_IN_PULSE: track 0.00 -> 568.3 mm, vias 0 -> 1
- net /*IOT_PULSE: track 0.00 -> 506.3 mm
- net /*INT_DETECT: track 0.00 -> 503.4 mm
- net /REQ_ADDR: track 0.00 -> 500.7 mm
- net /*JMP_I_DETECT: track 0.00 -> 500.1 mm, vias 0 -> 1
- net /*IOT_WAIT: track 0.00 -> 491.0 mm, vias 0 -> 3
- net /*READ_IN_CLEAR: track 0.00 -> 487.5 mm, vias 0 -> 1
- net /*INT_REQ: track 0.00 -> 477.4 mm, vias 0 -> 1
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
Commit message: Gerber creation marathon
Routing:
- net +5V: track 1865.8 -> 1867.5 mm
- net /*DMA_REQ0: track 239.4 -> 240.3 mm
- net /*MEMM_ENABLE: track 605.0 -> 605.8 mm
- net /*INT_REQ: track 477.4 -> 478.1 mm
- added copper zone on B.Cu, net GND
- added copper zone on F.Cu, net GND
Other:
- board text removed: "JLCJLCJLCJLC"
