File: kicad/Front Panel Address/Front Panel Address.kicad_sch (KiCad schematic)
At the start: 1 part, among them J1 Front Panel Connector

Commit message: Continue work on front panel
Parts:
- removed J1: Front Panel Connector, symbol Connector_Generic:Conn_02x20_Counter_Clockwise
- added J1: Front Panel Connector, symbol Connector_Generic:Conn_02x25_Counter_Clockwise
- added U1: 74LS377, symbol 74xx:74LS377
- added U2: 74LS147, symbol 74xx:74LS147
Connections:
- new net *LATCH_AC: J1.33 (Pin_33)
- new net *LATCH_IR: J1.35 (Pin_35), U1.1 (~{E})
- new net *LATCH_MA: J1.37 (Pin_37)
- new net *LATCH_MB: J1.34 (Pin_34)
- new net *LATCH_MQ: J1.32 (Pin_32)
- new net *LATCH_PC: J1.36 (Pin_36)
- new net *MEMM_ENABLE: J1.44 (Pin_44)
- new net *PI_ENABLE: J1.46 (Pin_46)
- new net +5V: U1.20 (VCC), U2.16 (VCC)
- new net CLK_A: J1.31 (Pin_31), U1.11 (CP)
- new net CLK_B: J1.30 (Pin_30)
- new net D0: J1.2 (Pin_2)
- new net D1: J1.3 (Pin_3)
- new net D10: J1.12 (Pin_12)
- new net D11: J1.13 (Pin_13)
- new net D12: J1.14 (Pin_14)
- new net D13: J1.15 (Pin_15)
- new net D14: J1.16 (Pin_16)
- new net D15: J1.17 (Pin_17)
- new net D16: J1.18 (Pin_18)
- new net D17: J1.19 (Pin_19)
- new net D2: J1.4 (Pin_4)
- new net D3: J1.5 (Pin_5)
- new net D4: J1.6 (Pin_6)
- new net D5: J1.7 (Pin_7)
- new net D6: J1.8 (Pin_8)
- new net D7: J1.9 (Pin_9)
- new net D8: J1.10 (Pin_10)
- new net D9: J1.11 (Pin_11)
- new net FLAG_LINK: J1.47 (Pin_47)
- new net FP0: J1.20 (Pin_20), U2.9 (S0)
- new net FP1: J1.21 (Pin_21), U2.7 (S1)
- new net FP2: J1.22 (Pin_22), U2.6 (S2)
- new net FP3: J1.23 (Pin_23), U2.14 (S3)
- new net GND: J1.1 (Pin_1), J1.24 (Pin_24), J1.25 (Pin_25), J1.26 (Pin_26), J1.27 (Pin_27), J1.28 (Pin_28), J1.29 (Pin_29), J1.50 (Pin_50), U1.10 (GND), U2.8 (GND)
- new net HALT: J1.45 (Pin_45)
- new net NEXT_BANK0: J1.49 (Pin_49)
- new net NEXT_BANK1: J1.48 (Pin_48)
- new net SC0: J1.43 (Pin_43)
- new net SC1: J1.42 (Pin_42)
- new net SC2: J1.41 (Pin_41)
- new net SC3: J1.40 (Pin_40)
- new net SC4: J1.39 (Pin_39)
- new net SC5: J1.38 (Pin_38)

Commit message: Continue work on front panel
Parts:
- added U3: 74LS74, symbol 74xx:74LS74
- added U4: NE555P, Package_DIP:DIP-8_W7.62mm, symbol Timer:NE555P
Connections:
- net *LATCH_IR: no longer U1.1 (~{E})
- net +5V: now also U3.4 (~{S}), U4.4 (R), U4.8 (VCC)
- net CLK_A: no longer U1.11 (CP)
- net GND: now also U1.1 (~{E}), U3.1 (~{R}), U4.1 (GND), U4.5 (CV)
- net at U2.1 (E4): now also U1.9 (Q3)
- net at U2.10 (E9): now also U3.5 (Q)
- net at U2.11 (E1): now also U1.2 (Q0)
- net at U2.12 (E2): now also U1.5 (Q1)
- net at U2.13 (E3): now also U1.6 (Q2)
- net at U2.2 (E5): now also U1.12 (Q4)
- net at U2.3 (E6): now also U1.15 (Q5)
- net at U2.4 (E7): now also U1.16 (Q6)
- net at U2.5 (E8): now also U1.19 (Q7)
- new net: U4.2 (TR), U4.6 (THR)
- no-connect marks 0 -> 1
Other:
- moved on the sheet: U1

Commit message: Finish up address front panel schematic
Parts:
- added C1: 10 nF, symbol Device:C_Small
- added C10, C11, C12, C13, C3, C4, C5, C6, C7, C8, C9: 0.1uF, Capacitor_THT:C_Disc_D5.0mm_W2.5mm_P5.00mm, symbol Device:C
- added C2: 10 uF, symbol Device:C_Small
- added D1: PI, symbol Device:LED
- added D10: LINK, symbol Device:LED
- added D11: IR13, symbol Device:LED
- added D12: IR14, symbol Device:LED
- added D13: IR15, symbol Device:LED
- added D14: IR16, symbol Device:LED
- added D15: IR17, symbol Device:LED
- added D16: PC0, symbol Device:LED
- added D17: PC1, symbol Device:LED
- added D18: PC2, symbol Device:LED
- added D19: PC3, symbol Device:LED
- added D2: GO, symbol Device:LED
- added D20: PC4, symbol Device:LED
- added D21: PC5, symbol Device:LED
- added D22: PC6, symbol Device:LED
- added D23: PC7, symbol Device:LED
- added D24: PC8, symbol Device:LED
- added D25: PC9, symbol Device:LED
- added D26: PC10, symbol Device:LED
- added D27: PC11, symbol Device:LED
- added D28: PC12, symbol Device:LED
- added D29: PC13, symbol Device:LED
- added D3: MM, symbol Device:LED
- added D30: PC14, symbol Device:LED
- added D31: MA0, symbol Device:LED
- added D32: MA1, symbol Device:LED
- added D33: MA2, symbol Device:LED
- added D34: MA3, symbol Device:LED
- added D35: MA4, symbol Device:LED
- added D36: MA5, symbol Device:LED
- added D37: MA6, symbol Device:LED
- added D38: MA7, symbol Device:LED
- added D39: MA8, symbol Device:LED
- added D4: SC0, symbol Device:LED
- added D40: MA9, symbol Device:LED
- added D41: MA10, symbol Device:LED
- added D42: MA11, symbol Device:LED
- added D43: MA12, symbol Device:LED
- added D44: MA13, symbol Device:LED
- added D45: MA14, symbol Device:LED
- added D5: SC1, symbol Device:LED
- added D6: SC2, symbol Device:LED
- added D7: SC3, symbol Device:LED
- added D8: SC4, symbol Device:LED
- added D9: SC5, symbol Device:LED
- added R1, R10, R11, R12, R13, R14, R15, R2, R3, R4, R7, R8, R9: 4.7K, Resistor_THT:R_Axial_DIN0207_L6.3mm_D2.5mm_P7.62mm_Horizontal, symbol Device:R
- added R5, R6: 1K, symbol Device:R
- added RN1, RN2, RN3, RN4, RN5, RN6, RN7, RN8, RN9: 330R, Resistor_THT:R_Array_SIP6, symbol Device:R_Network05
- added SW1: HALT / STEP, symbol Switch:SW_SPDT
- added SW2: CONTINUE, symbol Switch:SW_SPDT
- added SW3: GOTO, symbol Switch:SW_SPDT
- added SW4: EXAMINE, symbol Switch:SW_SPDT
- added SW5: EXAM NEXT, symbol Switch:SW_SPDT
- added SW6: DEPOSIT, symbol Switch:SW_SPDT
- added SW7: DEP NEXT, symbol Switch:SW_SPDT
- added SW8: READ IN, symbol Switch:SW_SPDT
- added SW9: XCT, symbol Switch:SW_SPDT
- added U10, U11, U7, U8, U9: 74LS377, symbol 74xx:74LS377
- added U5: 74LS04, symbol 74xx:74LS04
- added U6: 74LS244, symbol 74xx:74LS244
Connections:
- net *LATCH_IR: now also U7.1 (~{E})
- net *LATCH_MA: now also U10.1 (~{E}), U11.1 (~{E})
- net *LATCH_PC: now also U8.1 (~{E}), U9.1 (~{E})
- net *MEMM_ENABLE: now also U5.5
- net *PI_ENABLE: now also U5.1
- net +5V: now also J1.1 (Pin_1), J1.50 (Pin_50), U3.14 (VCC), C10.1, C11.1, C12.1, C13.1, C3.1, C4.1, C5.1, C6.1, C7.1, C8.1, C9.1, R1.1, R10.2, R11.2, R12.2, R13.2, R14.2, R15.2, R2.1, R3.1, R4.1, R6.2, R7.2, R8.2, R9.2, U10.20 (VCC), U11.20 (VCC), U5.14 (VCC), U6.20 (VCC), U7.20 (VCC), U8.20 (VCC), U9.20 (VCC); no longer U3.4 (~{S})
- net CLK_A: now also U3.11 (C), U10.11 (CP), U11.11 (CP), U7.11 (CP), U8.11 (CP), U9.11 (CP)
- net D0: now also U10.3 (D0), U9.3 (D0)
- net D1: now also U10.4 (D1), U9.4 (D1)
- net D10: now also U11.7 (D2), U8.7 (D2)
- net D11: now also U11.8 (D3), U8.8 (D3)
- net D12: now also U11.13 (D4), U8.13 (D4)
- net D13: now also U7.3 (D0)
- net D14: now also U7.4 (D1)
- net D15: now also U7.7 (D2)
- net D16: now also U7.8 (D3)
- net D17: now also U7.13 (D4)
- net D2: now also U10.7 (D2), U9.7 (D2)
- net D3: now also U10.8 (D3), U9.8 (D3)
- net D4: now also U10.13 (D4), U9.13 (D4)
- net D5: now also U10.14 (D5), U9.14 (D5)
- net D6: now also U10.17 (D6), U9.17 (D6)
- net D7: now also U10.18 (D7), U9.18 (D7)
- net D8: now also U11.3 (D0), U8.3 (D0)
- net D9: now also U11.4 (D1), U8.4 (D1)
- net FLAG_LINK: now also U6.15 (I2b)
- net GND: now also U3.7 (GND), C1.2, C10.2, C11.2, C12.2, C13.2, C2.1, C3.2, C4.2, C5.2, C6.2, C7.2, C8.2, C9.2, RN1.1 (common), RN2.1 (common), RN3.1 (common), RN4.1 (common), RN5.1 (common), RN6.1 (common), RN7.1 (common), RN8.1 (common), RN9.1 (common), SW1.3 (C), SW2.3 (C), SW3.3 (C), SW4.3 (C), SW5.3 (C), SW6.3 (C), SW7.3 (C), SW8.3 (C), SW9.3 (C), U10.10 (GND), U11.10 (GND), U11.18 (D7), U5.11, U5.13, U5.7 (GND), U5.9, U6.1 (OEa), U6.10 (GND), U6.17 (I3b), U6.19 (OEb), U7.10 (GND), U7.14 (D5), U7.17 (D6), U7.18 (D7), U8.10 (GND), U8.18 (D7), U9.10 (GND); no longer J1.1 (Pin_1), J1.28 (Pin_28), J1.29 (Pin_29), J1.50 (Pin_50), U3.1 (~{R}), U4.5 (CV)
- net HALT: now also U5.3
- net NEXT_BANK0: now also U11.14 (D5), U8.14 (D5)
- net NEXT_BANK1: now also U11.17 (D6), U8.17 (D6)
- net SC0: now also U6.2 (I0a)
- net SC1: now also U6.4 (I1a)
- net SC2: now also U6.6 (I2a)
- net SC3: now also U6.8 (I3a)
- net SC4: now also U6.11 (I0b)
- net SC5: now also U6.13 (I1b)
- net at U3.2 (D): now also R15.1, SW9.2 (B)
- net at U3.3 (C): now also U1.11 (CP), U3.9 (Q)
- net at U1.13 (D4): now also R11.1, SW5.2 (B)
- net at U1.14 (D5): now also R12.1, SW6.2 (B)
- net at U1.17 (D6): now also R13.1, SW7.2 (B)
- net at U1.18 (D7): now also R14.1, SW8.2 (B)
- net at U1.3 (D0): now also R7.1, SW1.2 (B)
- net at U1.4 (D1): now also R8.1, SW2.2 (B)
- net at U1.7 (D2): now also R9.1, SW3.2 (B)
- net at U1.8 (D3): now also R10.1, SW4.2 (B)
- net at U4.2 (TR), U4.6 (THR): now also C2.2, R5.1
- net at U4.3 (Q): now also U3.12 (D)
- net at U4.7 (DIS): now also R5.2, R6.1
- net at U3.10 (~{S}): now also R3.2
- net at U3.13 (~{R}): now also R4.2
- new net: D9.1 (K), RN1.5 (R4)
- new net: D9.2 (A), U6.7 (O1b)
- new net: D28.1 (K), RN6.4 (R3)
- new net: D28.2 (A), U8.12 (Q4)
- new net: D45.1 (K), RN9.6 (R5)
- new net: D45.2 (A), U11.16 (Q6)
- new net: D1.2 (A), U5.2
- new net: D43.1 (K), RN9.4 (R3)
- new net: D43.2 (A), U11.12 (Q4)
- new net: D1.1 (K), RN2.2 (R1)
- new net: D36.1 (K), RN8.2 (R1)
- new net: D36.2 (A), U10.15 (Q5)
- new net: D13.1 (K), RN3.4 (R3)
- new net: D13.2 (A), U7.6 (Q2)
- new net: D32.1 (K), RN7.3 (R2)
- new net: D32.2 (A), U10.5 (Q1)
- new net: D27.1 (K), RN6.3 (R2)
- new net: D27.2 (A), U8.9 (Q3)
- new net: C1.1, U4.5 (CV)
- new net: D20.2 (A), U9.12 (Q4)
- new net: D21.2 (A), U9.15 (Q5)
- new net: D22.2 (A), U9.16 (Q6)
- new net: D23.2 (A), U9.19 (Q7)
- new net: D16.2 (A), U9.2 (Q0)
- new net: D17.2 (A), U9.5 (Q1)
- new net: D18.2 (A), U9.6 (Q2)
- new net: D19.2 (A), U9.9 (Q3)
- new net: D6.1 (K), RN1.2 (R1)
- new net: D7.1 (K), RN1.3 (R2)
- new net: D8.1 (K), RN1.4 (R3)
- new net: D10.1 (K), RN1.6 (R5)
- new net: D41.1 (K), RN9.2 (R1)
- new net: D42.1 (K), RN9.3 (R2)
- new net: D44.1 (K), RN9.5 (R4)
- new net: D7.2 (A), U6.12 (O3a)
- new net: D6.2 (A), U6.14 (O2a)
- new net: D5.2 (A), U6.16 (O1a)
- new net: D4.2 (A), U6.18 (O0a)
- new net: D10.2 (A), U6.5 (O2b)
- new net: D8.2 (A), U6.9 (O0b)
- new net: D42.2 (A), U11.9 (Q3)
- new net: R2.2, U3.1 (~{R})
- new net: R1.2, U3.4 (~{S})
- new net: D26.1 (K), RN6.2 (R1)
- new net: D29.1 (K), RN6.5 (R4)
- new net: D30.1 (K), RN6.6 (R5)
- new net: D39.1 (K), RN8.5 (R4)
- new net: D39.2 (A), U11.2 (Q0)
- new net: D14.1 (K), RN3.5 (R4)
- new net: D14.2 (A), U7.9 (Q3)
- new net: D25.1 (K), RN5.6 (R5)
- new net: D25.2 (A), U8.5 (Q1)
- new net: D15.1 (K), RN3.6 (R5)
- new net: D15.2 (A), U7.12 (Q4)
- new net: D2.2 (A), U5.4
- new net: D3.1 (K), RN2.4 (R3)
- new net: D3.2 (A), U5.6
- new net: D4.1 (K), RN2.5 (R4)
- new net: D16.1 (K), RN4.2 (R1)
- new net: D11.1 (K), RN3.2 (R1)
- new net: D11.2 (A), U7.2 (Q0)
- new net: D2.1 (K), RN2.3 (R2)
- new net: D5.1 (K), RN2.6 (R5)
- new net: D17.1 (K), RN4.3 (R2)
- new net: D18.1 (K), RN4.4 (R3)
- new net: D19.1 (K), RN4.5 (R4)
- new net: D20.1 (K), RN4.6 (R5)
- new net: D29.2 (A), U8.15 (Q5)
- new net: D30.2 (A), U8.16 (Q6)
- new net: D24.2 (A), U8.2 (Q0)
- new net: D26.2 (A), U8.6 (Q2)
- new net: D44.2 (A), U11.15 (Q5)
- new net: D40.2 (A), U11.5 (Q1)
- new net: D41.2 (A), U11.6 (Q2)
- new net: D31.1 (K), RN7.2 (R1)
- new net: D33.1 (K), RN7.4 (R3)
- new net: D34.1 (K), RN7.5 (R4)
- new net: D35.1 (K), RN7.6 (R5)
- new net: D12.1 (K), RN3.3 (R2)
- new net: D24.1 (K), RN5.5 (R4)
- new net: D35.2 (A), U10.12 (Q4)
- new net: D37.2 (A), U10.16 (Q6)
- new net: D38.2 (A), U10.19 (Q7)
- new net: D31.2 (A), U10.2 (Q0)
- new net: D33.2 (A), U10.6 (Q2)
- new net: D34.2 (A), U10.9 (Q3)
- new net: D37.1 (K), RN8.3 (R2)
- new net: D38.1 (K), RN8.4 (R3)
- new net: D40.1 (K), RN8.6 (R5)
- new net: D21.1 (K), RN5.2 (R1)
- new net: D22.1 (K), RN5.3 (R2)
- new net: D23.1 (K), RN5.4 (R3)
- new net: D12.2 (A), U7.5 (Q1)
- new net *SELECT_SWR: J1.29 (Pin_29)
- no-connect marks 1 -> 26
Other:
- moved on the sheet: J1, U1, U2, U3A, U3B, U3C, U4

Commit message: Finish up front panel data schematic
Parts:
- added C20: 100 uF, Capacitor_THT:CP_Radial_D6.3mm_P2.50mm, symbol Device:C_Polarized
Connections:
- net +5V: now also C20.1
- net GND: now also C20.2
- no-connect marks 26 -> 27
Changed lines of the file:
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@@
   (junction (at 210.185 208.915) (diameter 0) (color 0 0 0 0)
   )
+  (no_connect (at -39.37 102.87))
   (no_connect (at 314.325 219.075))
   (no_connect (at 203.835 101.6))
@@
     )
   )
+  (symbol (lib_id "power:GND") (at 396.24 234.315 0) (mirror y) (unit 1)
+    (in_bom yes) (on_board yes) (dnp no) (fields_autoplaced)
+    (property "Reference" "#PWR095" (at 396.24 240.665 0)
+      (effects (font (size 1.27 1.27)) hide)
+    )
+    (property "Value" "GND" (at 396.24 238.76 0)
+      (effects (font (size 1.27 1.27)))
+    )
+    (property "Footprint" "" (at 396.24 234.315 0)
+      (effects (font (size 1.27 1.27)) hide)
+    )
+    (property "Datasheet" "" (at 396.24 234.315 0)
+      (effects (font (size 1.27 1.27)) hide)
+    )
+    (pin "1")
+    (instances
+      (project "Nabu_MEGAMAPPER"
+        (path "/08a88c4b-5d36-43ed-bafe-b5ff1ee4c2dd"
+          (reference "#PWR095") (unit 1)
+        )
+      )
+      (project "Front Panel Address"
+        (path "/a6d091a4-b7a7-4622-98da-a8652e256494"
+          (reference "#PWR084") (unit 1)
+        )
+      )
+      (project "ALU"
+        (path "/b26dce39-0c19-4808-8ddd-74847f21ad13"
+          (reference "#PWR0176") (unit 1)
+        )
+      )
+      (project "Memory"
+        (path "/b9764240-fb05-4333-bc5f-d2675d8c17cf"
+          (reference "#PWR0101") (unit 1)
+        )
+      )
+    )
+  )
   (symbol (lib_id "power:+5V") (at 298.45 244.475 0) (unit 1)
     (in_bom yes) (on_board yes) (dnp no) (fields_autoplaced)
@@
     )
   )
+  (symbol (lib_id "Device:C_Polarized") (at 392.43 234.315 90) (unit 1)
+    (in_bom yes) (on_board yes) (dnp no)
+    (property "Reference" "C20" (at 394.335 227.965 90)
+      (effects (font (size 1.27 1.27)))
+    )
+    (property "Value" "100 uF" (at 396.24 230.505 90)
+      (effects (font (size 1.27 1.27)))
+    )
+    (property "Footprint" "Capacitor_THT:CP_Radial_D6.3mm_P2.50mm" (at 396.24 233.3498 0)
+      (effects (font (size 1.27 1.27)) hide)
+    )
+    (property "Datasheet" "~" (at 392.43 234.315 0)
+      (effects (font (size 1.27 1.27)) hide)
+    )
+    (pin "1")
+    (pin "2")
+    (instances
+      (project "Nabu_MEGAMAPPER"
+        (path "/08a88c4b-5d36-43ed-bafe-b5ff1ee4c2dd"
+          (reference "C20") (unit 1)
+        )
+      )
+      (project "Front Panel Address"
+        (path "/a6d091a4-b7a7-4622-98da-a8652e256494"
+          (reference "C14") (unit 1)
+        )
+      )
+      (project "ALU"
+        (path "/b26dce39-0c19-4808-8ddd-74847f21ad13"
+          (reference "C40") (unit 1)
+        )
+      )
+      (project "Memory"
+        (path "/b9764240-fb05-4333-bc5f-d2675d8c17cf"
+          (reference "C21") (unit 1)
+        )
+      )
+    )
+  )
   (symbol (lib_id "Device:LED") (at 374.015 93.98 180) (unit 1)
     (in_bom yes) (on_board yes) (dnp no)
@@
         )
       )
+    )
+  )
+  (symbol (lib_id "power:+5V") (at 388.62 234.315 0) (mirror y) (unit 1)
+    (in_bom yes) (on_board yes) (dnp no) (fields_autoplaced)
+    (property "Reference" "#PWR048" (at 388.62 238.125 0)
+      (effects (font (size 1.27 1.27)) hide)
+    )
+    (property "Value" "+5V" (at 388.62 229.87 0)
+      (effects (font (size 1.27 1.27)))
+    )
+    (property "Footprint" "" (at 388.62 234.315 0)
+      (effects (font (size 1.27 1.27)) hide)
+    )
+    (property "Datasheet" "" (at 388.62 234.315 0)
+      (effects (font (size 1.27 1.27)) hide)
+    )
+    (pin "1")
+    (instances
+      (project "Nabu_MEGAMAPPER"
+        (path "/08a88c4b-5d36-43ed-bafe-b5ff1ee4c2dd"
+          (reference "#PWR048") (unit 1)
+        )
+      )
+      (project "Front Panel Address"
+        (path "/a6d091a4-b7a7-4622-98da-a8652e256494"
+          (reference "#PWR083") (unit 1)
+        )
+      )
+      (project "ALU"
+        (path "/b26dce39-0c19-4808-8ddd-74847f21ad13"
+          (reference "#PWR0175") (unit 1)
+        )
+      )
+      (project "Memory"
+        (path "/b9764240-fb05-4333-bc5f-d2675d8c17cf"
+          (reference "#PWR0100") (unit 1)
+        )
+      )

Commit message: Start work on front panel address layout
Parts:
- removed U2: 74LS147, symbol 74xx:74LS147
- added U2: 74LS147, Package_DIP:DIP-16_W7.62mm, symbol Custom:74LS147
- C1, C2: footprint (none) -> Capacitor_THT:C_Disc_D5.0mm_W2.5mm_P5.00mm
- D1, D10, D11, D12, D13, D14, D15, D16, D17, D18, D19, D2, D20, D21, D22, D23, D24, D25, D26, D27, D28, D29, D3, D30, D31, D32, D33, D34, D35, D36, D37, D38, D39, D4, D40, D41, D42, D43, D44, D45, D5, D6, D7, D8, D9: footprint (none) -> LED_THT:LED_D5.0mm
- J1: footprint (none) -> Connector_IDC:IDC-Header_2x25_P2.54mm_Vertical
- R5, R6: footprint (none) -> Resistor_THT:R_Axial_DIN0207_L6.3mm_D2.5mm_P7.62mm_Horizontal
- SW1, SW2, SW3, SW4, SW5, SW6, SW7, SW8, SW9: footprint (none) -> Custom:MTS-102
- U1, U10, U11, U6, U7, U8, U9: footprint (none) -> Package_DIP:DIP-20_W7.62mm
- U3, U5: footprint (none) -> Package_DIP:DIP-14_W7.62mm
Connections:
- net +5V: now also U2.16 (VCC)
- net FP0: now also U2.9 (S0)
- net FP1: now also U2.7 (S1)
- net FP2: now also U2.6 (S2)
- net FP3: now also U2.14 (S3)
- net GND: now also U2.8 (GND)
- net SYNC_CLK: now reaches J1.28 (Pin_28)
- net SYNC_CLK: now also U1.11 (CP), U3.3 (C), U3.9 (Q)
- net at U3.5 (Q): now also U2.10 (E9)
- net at U1.9 (Q3): now also U2.1 (E4)
- net at U1.2 (Q0): now also U2.11 (E1)
- net at U1.5 (Q1): now also U2.12 (E2)
- net at U1.6 (Q2): now also U2.13 (E3)
- net at U1.12 (Q4): now also U2.2 (E5)
- net at U1.15 (Q5): now also U2.3 (E6)
- net at U1.16 (Q6): now also U2.4 (E7)
- net at U1.19 (Q7): now also U2.5 (E8)
- no-connect marks 27 -> 26

Commit message: Continue work on front panel
Connections:
- net SYNC_CLK: now also U3.12 (D), U4.3 (Q); no longer U1.11 (CP), U3.3 (C), U3.9 (Q)
- new net: U1.11 (CP), U3.3 (C), U3.9 (Q)

Commit message: Continue work on backplane
Connections:
- net CLK_A: no longer U3.11 (C)
- net GND: no longer J1.27 (Pin_27)
- net SYNC_CLK: now also J1.27 (Pin_27), U3.11 (C); no longer J1.28 (Pin_28), U3.12 (D), U4.3 (Q)
- net DELAY_CLK: now reaches U1.11 (CP), U3.3 (C), U3.9 (Q)
- net DELAY_CLK: now also J1.28 (Pin_28)
- new net: U3.12 (D), U4.3 (Q)
Changed lines of the file:
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@@
   (junction (at 36.195 223.52) (diameter 0) (color 0 0 0 0)
-  )
-  (junction (at 48.895 95.885) (diameter 0) (color 0 0 0 0)
   )
   (junction (at 43.18 188.595) (diameter 0) (color 0 0 0 0)
@@
     (stroke (width 0) (type default))
   )
-  (wire (pts (xy 48.895 93.345) (xy 48.895 95.885))
-    (stroke (width 0) (type default))
-  )
   (wire (pts (xy 203.835 93.98) (xy 216.535 93.98))
     (stroke (width 0) (type default))
@@
     (effects (font (size 1.27 1.27)) (justify right bottom))
   )
+  (label "DELAY_CLK" (at 48.895 90.805 0) (fields_autoplaced)
+    (effects (font (size 1.27 1.27)) (justify left bottom))
+  )
   (label "*LATCH_MB" (at 48.895 75.565 0) (fields_autoplaced)
     (effects (font (size 1.27 1.27)) (justify left bottom))
@@
     (effects (font (size 1.27 1.27)) (justify right bottom))
   )
-  (label "SYNC_CLK" (at 55.245 208.28 0) (fields_autoplaced)
-    (effects (font (size 1.27 1.27)) (justify left bottom))
+  (label "SYNC_CLK" (at 66.675 210.82 180) (fields_autoplaced)
+    (effects (font (size 1.27 1.27)) (justify right bottom))
   )
   (label "D3" (at 332.74 43.18 180) (fields_autoplaced)
@@
     (effects (font (size 1.27 1.27)) (justify right bottom))
   )
-  (label "SYNC_CLK" (at 48.895 90.805 0) (fields_autoplaced)
+  (label "SYNC_CLK" (at 48.895 93.345 0) (fields_autoplaced)
     (effects (font (size 1.27 1.27)) (justify left bottom))
   )
@@
     (effects (font (size 1.27 1.27)) (justify left bottom))
   )
-  (label "CLK_A" (at 66.675 210.82 180) (fields_autoplaced)
-    (effects (font (size 1.27 1.27)) (justify right bottom))
-  )
   (label "D4" (at 250.19 45.72 180) (fields_autoplaced)
     (effects (font (size 1.27 1.27)) (justify right bottom))
   )
+  (label "DELAY_CLK" (at 89.535 208.28 0) (fields_autoplaced)
+    (effects (font (size 1.27 1.27)) (justify left bottom))
+  )
   (label "D3" (at 250.19 43.18 180) (fields_autoplaced)

Commit message: Continue work on routing
Parts:
- added H1, H2, H3, H4: MountingHole, MountingHole:MountingHole_2.2mm_M2_Pad, symbol Mechanical:MountingHole
Changed lines of the file:
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@@
+    )
+  )
+  (symbol (lib_id "Mechanical:MountingHole") (at 208.28 257.175 0) (unit 1)
+    (in_bom yes) (on_board yes) (dnp no) (fields_autoplaced)
+    (property "Reference" "H2" (at 210.82 255.9629 0)
+      (effects (font (size 1.27 1.27)) (justify left))
+    )
+    (property "Value" "MountingHole" (at 210.82 258.3871 0)
+      (effects (font (size 1.27 1.27)) (justify left))
+    )
+    (property "Footprint" "MountingHole:MountingHole_2.2mm_M2_Pad" (at 208.28 257.175 0)
+      (effects (font (size 1.27 1.27)) hide)
+    )
+    (property "Datasheet" "~" (at 208.28 257.175 0)
+      (effects (font (size 1.27 1.27)) hide)
+    )
+    (instances
+      (project "Front Panel Register"
+        (path "/43c9f2e1-b850-426e-8849-9d0baaf5e00b"
+          (reference "H2") (unit 1)
+        )
+      )
+      (project "Front Panel Address"
+        (path "/a6d091a4-b7a7-4622-98da-a8652e256494"
+          (reference "H2") (unit 1)
+        )
+      )
     )
   )
@@
     )
   )
+  (symbol (lib_id "Mechanical:MountingHole") (at 208.28 269.875 0) (unit 1)
+    (in_bom yes) (on_board yes) (dnp no) (fields_autoplaced)
+    (property "Reference" "H4" (at 210.82 268.6629 0)
+      (effects (font (size 1.27 1.27)) (justify left))
+    )
+    (property "Value" "MountingHole" (at 210.82 271.0871 0)
+      (effects (font (size 1.27 1.27)) (justify left))
+    )
+    (property "Footprint" "MountingHole:MountingHole_2.2mm_M2_Pad" (at 208.28 269.875 0)
+      (effects (font (size 1.27 1.27)) hide)
+    )
+    (property "Datasheet" "~" (at 208.28 269.875 0)
+      (effects (font (size 1.27 1.27)) hide)
+    )
+    (instances
+      (project "Front Panel Register"
+        (path "/43c9f2e1-b850-426e-8849-9d0baaf5e00b"
+          (reference "H4") (unit 1)
+        )
+      )
+      (project "Front Panel Address"
+        (path "/a6d091a4-b7a7-4622-98da-a8652e256494"
+          (reference "H4") (unit 1)
+        )
+      )
+    )
+  )
   (symbol (lib_id "power:GND") (at 334.01 244.475 0) (unit 1)
     (in_bom yes) (on_board yes) (dnp no) (fields_autoplaced)
@@
     )
   )
+  (symbol (lib_id "Mechanical:MountingHole") (at 208.28 250.825 0) (unit 1)
+    (in_bom yes) (on_board yes) (dnp no) (fields_autoplaced)
+    (property "Reference" "H1" (at 210.82 249.6129 0)
+      (effects (font (size 1.27 1.27)) (justify left))
+    )
+    (property "Value" "MountingHole" (at 210.82 252.0371 0)
+      (effects (font (size 1.27 1.27)) (justify left))
+    )
+    (property "Footprint" "MountingHole:MountingHole_2.2mm_M2_Pad" (at 208.28 250.825 0)
+      (effects (font (size 1.27 1.27)) hide)
+    )
+    (property "Datasheet" "~" (at 208.28 250.825 0)
+      (effects (font (size 1.27 1.27)) hide)
+    )
+    (instances
+      (project "Front Panel Register"
+        (path "/43c9f2e1-b850-426e-8849-9d0baaf5e00b"
+          (reference "H1") (unit 1)
+        )
+      )
+      (project "Front Panel Address"
+        (path "/a6d091a4-b7a7-4622-98da-a8652e256494"
+          (reference "H1") (unit 1)
+        )
+      )
+    )
+  )
   (symbol (lib_id "power:+5V") (at 336.55 244.475 0) (unit 1)
     (in_bom yes) (on_board yes) (dnp no) (fields_autoplaced)
@@
         )
       )
+    )
+  )
+  (symbol (lib_id "Mechanical:MountingHole") (at 208.28 263.525 0) (unit 1)
+    (in_bom yes) (on_board yes) (dnp no) (fields_autoplaced)
+    (property "Reference" "H3" (at 210.82 262.3129 0)
+      (effects (font (size 1.27 1.27)) (justify left))
+    )
+    (property "Value" "MountingHole" (at 210.82 264.7371 0)
+      (effects (font (size 1.27 1.27)) (justify left))
+    )
+    (property "Footprint" "MountingHole:MountingHole_2.2mm_M2_Pad" (at 208.28 263.525 0)
+      (effects (font (size 1.27 1.27)) hide)
+    )
+    (property "Datasheet" "~" (at 208.28 263.525 0)
+      (effects (font (size 1.27 1.27)) hide)
+    )
+    (instances
+      (project "Front Panel Register"
+        (path "/43c9f2e1-b850-426e-8849-9d0baaf5e00b"
+          (reference "H3") (unit 1)
+        )
+      )
+      (project "Front Panel Address"
+        (path "/a6d091a4-b7a7-4622-98da-a8652e256494"
+          (reference "H3") (unit 1)
+        )
+      )
