File: kicad/Front Panel Address/Front Panel Address.kicad_pcb (KiCad board)
At the start: 2 copper layers, 170.2 x 107.3 mm, 104 parts, among them J1 Front Panel Connector, SW1 HALT / STEP, SW2 CONTINUE, SW3 GOTO, SW4 EXAMINE, SW5 EXAM NEXT, SW6 DEPOSIT, SW7 DEP NEXT, SW8 READ IN, SW9 XCT, U1 74LS377, U10 74LS377, U11 74LS377, U2 74LS147, U3 74LS74, U4 NE555P, U5 74LS04, U6 74LS244, U7 74LS377, U8 74LS377, U9 74LS377

Commit message: Continue work on front panel
Parts:
- moved C3 12.7 mm to (127.6, 128.3)
- moved U1 12.7 mm to (130.8, 134.6)
- moved R1 6.35 mm to (109.9, 134.0)
- moved R2 6.35 mm to (109.9, 130.8)
- moved R3 6.35 mm to (109.9, 127.6)
- moved C5 6.35 mm to (86.4, 128.3)
- moved U3 6.35 mm to (89.5, 134.6)
Connections:
- U1 pad 11: /SYNC_CLK -> Net-(U1-CP)
- U3 pad 12: Net-(U3B-D) -> /SYNC_CLK
- U3 pad 3: /SYNC_CLK -> Net-(U1-CP)
- U3 pad 9: /SYNC_CLK -> Net-(U1-CP)
- U4 pad 3: Net-(U3B-D) -> /SYNC_CLK

Commit message: Continue work on backplane
Connections:
- J1 pad 27: GND -> /SYNC_CLK
- J1 pad 28: /SYNC_CLK -> /DELAY_CLK
- U3 pad 11: /CLK_A -> /SYNC_CLK
- U3 pad 12: /SYNC_CLK -> /DELAY_CLK
- U4 pad 3: /SYNC_CLK -> /DELAY_CLK
Changed lines of the file:
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@@
   (net 182 "/SYNC_CLK")
   (net 183 "Net-(U1-CP)")
+  (net 184 "/DELAY_CLK")
   (footprint "Resistor_THT:R_Axial_DIN0207_L6.3mm_D2.5mm_P7.62mm_Horizontal" (layer "F.Cu")
     (at 67.31 133.985)
@@
       (net 140 "Net-(U3B-~{S})") (pinfunction "~{S}") (pintype "input"))
     (pad "11" thru_hole oval (at 7.62 7.62 90) (size 1.6 1.6) (drill 0.8) (layers "*.Cu" "*.Mask")
-      (net 119 "/CLK_A") (pinfunction "C") (pintype "input"))
+      (net 182 "/SYNC_CLK") (pinfunction "C") (pintype "input"))
     (pad "12" thru_hole oval (at 7.62 5.08 90) (size 1.6 1.6) (drill 0.8) (layers "*.Cu" "*.Mask")
-      (net 182 "/SYNC_CLK") (pinfunction "D") (pintype "input"))
+      (net 184 "/DELAY_CLK") (pinfunction "D") (pintype "input"))
     (pad "13" thru_hole oval (at 7.62 2.54 90) (size 1.6 1.6) (drill 0.8) (layers "*.Cu" "*.Mask")
       (net 141 "Net-(U3B-~{R})") (pinfunction "~{R}") (pintype "input"))
@@
       (net 3 "Net-(U4-THR)") (pinfunction "TR") (pintype "input"))
     (pad "3" thru_hole oval (at 0 5.08 90) (size 1.6 1.6) (drill 0.8) (layers "*.Cu" "*.Mask")
-      (net 182 "/SYNC_CLK") (pinfunction "Q") (pintype "output"))
+      (net 184 "/DELAY_CLK") (pinfunction "Q") (pintype "output"))
     (pad "4" thru_hole oval (at 0 7.62 90) (size 1.6 1.6) (drill 0.8) (layers "*.Cu" "*.Mask")
       (net 4 "+5V") (pinfunction "R") (pintype "input"))
@@
       (net 2 "GND") (pinfunction "Pin_26") (pintype "passive"))
     (pad "27" thru_hole circle (at 0 -33.02 90) (size 1.7 1.7) (drill 1) (layers "*.Cu" "*.Mask")
-      (net 2 "GND") (pinfunction "Pin_27") (pintype "passive"))
+      (net 182 "/SYNC_CLK") (pinfunction "Pin_27") (pintype "passive"))
     (pad "28" thru_hole circle (at 2.54 -33.02 90) (size 1.7 1.7) (drill 1) (layers "*.Cu" "*.Mask")
-      (net 182 "/SYNC_CLK") (pinfunction "Pin_28") (pintype "passive"))
+      (net 184 "/DELAY_CLK") (pinfunction "Pin_28") (pintype "passive"))
     (pad "29" thru_hole circle (at 0 -35.56 90) (size 1.7 1.7) (drill 1) (layers "*.Cu" "*.Mask")
       (net 117 "/*SELECT_SWR") (pinfunction "Pin_29") (pintype "passive+no_connect"))

Commit message: Continue work on routing
Parts:
- added H1: MountingHole, MountingHole:MountingHole_2.2mm_M2_Pad, F.Cu at (40.0, 71.1)
- added H2: MountingHole, MountingHole:MountingHole_2.2mm_M2_Pad, F.Cu at (40.0, 131.4)
- added H3: MountingHole, MountingHole:MountingHole_2.2mm_M2_Pad, F.Cu at (202.6, 71.1)
- added H4: MountingHole, MountingHole:MountingHole_2.2mm_M2_Pad, F.Cu at (202.6, 131.4)
Connections:
- U1 pad 11: Net-(U1-CP) -> /DELAY_CLK
- U3 pad 12: /DELAY_CLK -> Net-(U3B-D)
- U3 pad 3: Net-(U1-CP) -> /DELAY_CLK
- U3 pad 9: Net-(U1-CP) -> /DELAY_CLK
- U4 pad 3: /DELAY_CLK -> Net-(U3B-D)
Changed lines of the file:
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@@
   (net 181 "unconnected-(U11-Q7-Pad19)")
   (net 182 "/SYNC_CLK")
-  (net 183 "Net-(U1-CP)")
+  (net 183 "Net-(U3B-D)")
   (net 184 "/DELAY_CLK")
   (footprint "Resistor_THT:R_Axial_DIN0207_L6.3mm_D2.5mm_P7.62mm_Horizontal" (layer "F.Cu")
@@
     )
   )
+  (footprint "MountingHole:MountingHole_2.2mm_M2_Pad" (layer "F.Cu")
+    (at 202.565 131.445)
+    (descr "Mounting Hole 2.2mm, M2")
+    (tags "mounting hole 2.2mm m2")
+    (property "Sheetfile" "Front Panel Address.kicad_sch")
+    (property "Sheetname" "")
+    (property "ki_description" "Mounting Hole without connection")
+    (property "ki_keywords" "mounting hole")
+    (attr exclude_from_pos_files)
+    (fp_text reference "H4" (at 0 -3.2) (layer "F.Fab")
+        (effects (font (size 1 1) (thickness 0.15)))
+    )
+    (fp_text value "MountingHole" (at 0 3.2) (layer "F.Fab")
+        (effects (font (size 1 1) (thickness 0.15)))
+    )
+    (fp_text user "${REFERENCE}" (at 0 0) (layer "F.Fab")
+        (effects (font (size 1 1) (thickness 0.15)))
+    )
+    (fp_circle (center 0 0) (end 2.2 0)
+      (stroke (width 0.15) (type solid)) (fill none) (layer "Cmts.User"))
+    (fp_circle (center 0 0) (end 2.45 0)
+      (stroke (width 0.05) (type solid)) (fill none) (layer "F.CrtYd"))
+    (pad "1" thru_hole circle (at 0 0) (size 4.4 4.4) (drill 2.2) (layers "*.Cu" "*.Mask"))
+  )
   (footprint "Capacitor_THT:C_Disc_D5.0mm_W2.5mm_P5.00mm" (layer "F.Cu")
     (at 127.635 128.31 -90)
@@
       (net 151 "Net-(SW9-B)") (pinfunction "D") (pintype "input"))
     (pad "3" thru_hole oval (at 0 5.08 90) (size 1.6 1.6) (drill 0.8) (layers "*.Cu" "*.Mask")
-      (net 183 "Net-(U1-CP)") (pinfunction "C") (pintype "input"))
+      (net 184 "/DELAY_CLK") (pinfunction "C") (pintype "input"))
     (pad "4" thru_hole oval (at 0 7.62 90) (size 1.6 1.6) (drill 0.8) (layers "*.Cu" "*.Mask")
       (net 138 "Net-(U3A-~{S})") (pinfunction "~{S}") (pintype "input"))
@@
       (net 172 "unconnected-(U3B-~{Q}-Pad8)") (pinfunction "~{Q}") (pintype "output+no_connect"))
     (pad "9" thru_hole oval (at 7.62 12.7 90) (size 1.6 1.6) (drill 0.8) (layers "*.Cu" "*.Mask")
-      (net 183 "Net-(U1-CP)") (pinfunction "Q") (pintype "output"))
+      (net 184 "/DELAY_CLK") (pinfunction "Q") (pintype "output"))
     (pad "10" thru_hole oval (at 7.62 10.16 90) (size 1.6 1.6) (drill 0.8) (layers "*.Cu" "*.Mask")
       (net 140 "Net-(U3B-~{S})") (pinfunction "~{S}") (pintype "input"))
@@
       (net 182 "/SYNC_CLK") (pinfunction "C") (pintype "input"))
     (pad "12" thru_hole oval (at 7.62 5.08 90) (size 1.6 1.6) (drill 0.8) (layers "*.Cu" "*.Mask")
-      (net 184 "/DELAY_CLK") (pinfunction "D") (pintype "input"))
+      (net 183 "Net-(U3B-D)") (pinfunction "D") (pintype "input"))
     (pad "13" thru_hole oval (at 7.62 2.54 90) (size 1.6 1.6) (drill 0.8) (layers "*.Cu" "*.Mask")
       (net 141 "Net-(U3B-~{R})") (pinfunction "~{R}") (pintype "input"))
@@
     )
   )
+  (footprint "MountingHole:MountingHole_2.2mm_M2_Pad" (layer "F.Cu")
+    (at 202.565 71.12)
+    (descr "Mounting Hole 2.2mm, M2")
+    (tags "mounting hole 2.2mm m2")
+    (property "Sheetfile" "Front Panel Address.kicad_sch")
+    (property "Sheetname" "")
+    (property "ki_description" "Mounting Hole without connection")
+    (property "ki_keywords" "mounting hole")
+    (attr exclude_from_pos_files)
+    (fp_text reference "H3" (at 0 -3.2) (layer "F.Fab")
+        (effects (font (size 1 1) (thickness 0.15)))
+    )
+    (fp_text value "MountingHole" (at 0 3.2) (layer "F.Fab")
+        (effects (font (size 1 1) (thickness 0.15)))
+    )
+    (fp_text user "${REFERENCE}" (at 0 0) (layer "F.Fab")
+        (effects (font (size 1 1) (thickness 0.15)))
+    )
+    (fp_circle (center 0 0) (end 2.2 0)
+      (stroke (width 0.15) (type solid)) (fill none) (layer "Cmts.User"))
+    (fp_circle (center 0 0) (end 2.45 0)
+      (stroke (width 0.05) (type solid)) (fill none) (layer "F.CrtYd"))
+    (pad "1" thru_hole circle (at 0 0) (size 4.4 4.4) (drill 2.2) (layers "*.Cu" "*.Mask"))
+  )
   (footprint "Package_DIP:DIP-20_W7.62mm" (layer "F.Cu")
     (at 130.81 134.62 90)
@@
       (net 2 "GND") (pinfunction "GND") (pintype "power_in"))
     (pad "11" thru_hole oval (at 7.62 22.86 90) (size 1.6 1.6) (drill 0.8) (layers "*.Cu" "*.Mask")
-      (net 183 "Net-(U1-CP)") (pinfunction "CP") (pintype "input"))
+      (net 184 "/DELAY_CLK") (pinfunction "CP") (pintype "input"))
     (pad "12" thru_hole oval (at 7.62 20.32 90) (size 1.6 1.6) (drill 0.8) (layers "*.Cu" "*.Mask")
       (net 165 "Net-(U1-Q4)") (pinfunction "Q4") (pintype "output"))
@@
     )
   )
+  (footprint "MountingHole:MountingHole_2.2mm_M2_Pad" (layer "F.Cu")
+    (at 40.005 71.12)
+    (descr "Mounting Hole 2.2mm, M2")
+    (tags "mounting hole 2.2mm m2")
+    (property "Sheetfile" "Front Panel Address.kicad_sch")
+    (property "Sheetname" "")
+    (property "ki_description" "Mounting Hole without connection")
+    (property "ki_keywords" "mounting hole")
+    (attr exclude_from_pos_files)
+    (fp_text reference "H1" (at 0 -3.2) (layer "F.Fab")
+        (effects (font (size 1 1) (thickness 0.15)))
+    )
+    (fp_text value "MountingHole" (at 0 3.2) (layer "F.Fab")
+        (effects (font (size 1 1) (thickness 0.15)))
+    )
+    (fp_text user "${REFERENCE}" (at 0 0) (layer "F.Fab")
+        (effects (font (size 1 1) (thickness 0.15)))
+    )
+    (fp_circle (center 0 0) (end 2.2 0)
+      (stroke (width 0.15) (type solid)) (fill none) (layer "Cmts.User"))
+    (fp_circle (center 0 0) (end 2.45 0)
+      (stroke (width 0.05) (type solid)) (fill none) (layer "F.CrtYd"))
+    (pad "1" thru_hole circle (at 0 0) (size 4.4 4.4) (drill 2.2) (layers "*.Cu" "*.Mask"))
+  )
   (footprint "Resistor_THT:R_Array_SIP6" (layer "F.Cu")
     (at 137.795 80.645 180)
@@
       (net 3 "Net-(U4-THR)") (pinfunction "TR") (pintype "input"))
     (pad "3" thru_hole oval (at 0 5.08 90) (size 1.6 1.6) (drill 0.8) (layers "*.Cu" "*.Mask")
-      (net 184 "/DELAY_CLK") (pinfunction "Q") (pintype "output"))
+      (net 183 "Net-(U3B-D)") (pinfunction "Q") (pintype "output"))
     (pad "4" thru_hole oval (at 0 7.62 90) (size 1.6 1.6) (drill 0.8) (layers "*.Cu" "*.Mask")
       (net 4 "+5V") (pinfunction "R") (pintype "input"))
@@
     )
   )
+  (footprint "MountingHole:MountingHole_2.2mm_M2_Pad" (layer "F.Cu")
+    (at 40.005 131.445)
+    (descr "Mounting Hole 2.2mm, M2")
+    (tags "mounting hole 2.2mm m2")
+    (property "Sheetfile" "Front Panel Address.kicad_sch")
+    (property "Sheetname" "")
+    (property "ki_description" "Mounting Hole without connection")
+    (property "ki_keywords" "mounting hole")
+    (attr exclude_from_pos_files)
+    (fp_text reference "H2" (at 0 -3.2) (layer "F.Fab")
+        (effects (font (size 1 1) (thickness 0.15)))
+    )
+    (fp_text value "MountingHole" (at 0 3.2) (layer "F.Fab")
+        (effects (font (size 1 1) (thickness 0.15)))
+    )
+    (fp_text user "${REFERENCE}" (at 0 0) (layer "F.Fab")
+        (effects (font (size 1 1) (thickness 0.15)))
+    )
+    (fp_circle (center 0 0) (end 2.2 0)
+      (stroke (width 0.15) (type solid)) (fill none) (layer "Cmts.User"))
+    (fp_circle (center 0 0) (end 2.45 0)
+      (stroke (width 0.05) (type solid)) (fill none) (layer "F.CrtYd"))
+    (pad "1" thru_hole circle (at 0 0) (size 4.4 4.4) (drill 2.2) (layers "*.Cu" "*.Mask"))
+  )
   (footprint "LED_THT:LED_D5.0mm" (layer "F.Cu")

Commit message: Gerber creation marathon
Routing:
- net GND: track 0.00 -> 765.7 mm
- net +5V: track 0.00 -> 556.1 mm
- net /D8: track 0.00 -> 181.6 mm, vias 0 -> 2
- net /CLK_A: track 0.00 -> 174.6 mm
- net /D5: track 0.00 -> 168.7 mm, vias 0 -> 1
- net /D9: track 0.00 -> 153.5 mm
- net /D7: track 0.00 -> 143.2 mm, vias 0 -> 1
- net /D1: track 0.00 -> 138.3 mm
- net /D10: track 0.00 -> 136.6 mm
- net /D12: track 0.00 -> 133.5 mm, vias 0 -> 1
- net /D0: track 0.00 -> 132.8 mm
- net /D11: track 0.00 -> 129.9 mm
- net /D4: track 0.00 -> 114.5 mm, vias 0 -> 1
- net Net-(SW9-B): track 0.00 -> 114.4 mm, vias 0 -> 1
- net /D3: track 0.00 -> 109.7 mm, vias 0 -> 2
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- added copper zone on B.Cu, net GND
- added copper zone on F.Cu, net GND
Other:
- board text added: "Gavin Tersteeg, 2026"
- board text added: "RDP-9A-FPA-0"
