File: kicad/Front Panel Register/Front Panel Register.kicad_sch (KiCad schematic)
At the start: 127 parts, among them J1 Front Panel Connector, SW1 SWR0, SW10 SWR9, SW11 SWR10, SW12 SWR11, SW13 SWR12, SW14 SWR13, SW15 SWR14, SW16 SWR15, SW17 SWR16, SW18 SWR17, SW2 SWR1, SW3 SWR2, SW4 SWR3, SW5 SWR4, SW6 SWR5, SW7 SWR6, SW8 SWR7, SW9 SWR8, U1 74LS244, U10 74LS377, U11 74LS377, U12 74LS377, U2 74LS244, U3 74LS244, U4 74LS377, U5 74LS377, U6 74LS377, U7 74LS377, U8 74LS377, U9 74LS377

Commit message: Start work on front panel register layout
Parts:
- D1, D10, D11, D12, D13, D14, D15, D16, D17, D18, D19, D2, D20, D21, D22, D23, D24, D25, D26, D27, D28, D29, D3, D30, D31, D32, D33, D34, D35, D36, D37, D38, D39, D4, D40, D41, D42, D43, D44, D45, D46, D47, D48, D49, D5, D50, D51, D52, D53, D54, D6, D7, D8, D9: footprint (none) -> LED_THT:LED_D5.0mm
- J1: footprint (none) -> Connector_IDC:IDC-Header_2x25_P2.54mm_Vertical
- SW1, SW10, SW11, SW12, SW13, SW14, SW15, SW16, SW17, SW18, SW2, SW3, SW4, SW5, SW6, SW7, SW8, SW9: footprint (none) -> Custom:MTS-102
- U1, U10, U11, U12, U2, U3, U4, U5, U6, U7, U8, U9: footprint (none) -> Package_DIP:DIP-20_W7.62mm

Commit message: Continue work on backplane
Connections:
- net GND: no longer J1.27 (Pin_27)
- net DELAY_CLK: now reaches J1.28 (Pin_28)
- new net SYNC_CLK: J1.27 (Pin_27)
- no-connect marks 64 -> 65
Changed lines of the file:
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@@
   (junction (at 249.555 220.98) (diameter 0) (color 0 0 0 0)
-  )
-  (junction (at 53.34 95.25) (diameter 0) (color 0 0 0 0)
   )
   (junction (at 123.19 149.86) (diameter 0) (color 0 0 0 0)
@@
   (no_connect (at 170.815 114.3))
   (no_connect (at 53.34 39.37))
+  (no_connect (at 53.34 90.17))
   (no_connect (at 214.63 270.51))
   (no_connect (at 300.99 149.86))
@@
   (no_connect (at 300.99 147.32))
   (no_connect (at 28.575 271.78))
+  (no_connect (at 53.34 92.71))
   (no_connect (at 40.64 85.09))
   (no_connect (at 148.59 142.24))
@@
   (no_connect (at 201.295 270.51))
   (no_connect (at 257.175 195.58))
-  (no_connect (at 53.34 90.17))
   (no_connect (at 224.79 154.94))
   (no_connect (at 134.62 270.51))
@@
     (stroke (width 0) (type default))
   )
-  (wire (pts (xy 53.34 92.71) (xy 53.34 95.25))
-    (stroke (width 0) (type default))
-  )
   (wire (pts (xy 269.24 139.7) (xy 275.59 139.7))
     (stroke (width 0) (type default))
@@
     (effects (font (size 1.27 1.27)) (justify right bottom))
   )
+  (label "SYNC_CLK" (at 53.34 92.71 0) (fields_autoplaced)
+    (effects (font (size 1.27 1.27)) (justify left bottom))
+  )
   (label "D8" (at 199.39 86.36 180) (fields_autoplaced)
     (effects (font (size 1.27 1.27)) (justify right bottom))
@@
     (effects (font (size 1.27 1.27)) (justify left bottom))
   )
+  (label "DELAY_CLK" (at 53.34 90.17 0) (fields_autoplaced)
+    (effects (font (size 1.27 1.27)) (justify left bottom))
+  )

Commit message: Continue work on routing
Parts:
- added H1, H2, H3, H4: MountingHole, MountingHole:MountingHole_2.2mm_M2_Pad, symbol Mechanical:MountingHole
Changed lines of the file:
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@@
     )
   )
+  (symbol (lib_id "Mechanical:MountingHole") (at 389.89 29.845 0) (unit 1)
+    (in_bom yes) (on_board yes) (dnp no) (fields_autoplaced)
+    (property "Reference" "H3" (at 392.43 28.6329 0)
+      (effects (font (size 1.27 1.27)) (justify left))
+    )
+    (property "Value" "MountingHole" (at 392.43 31.0571 0)
+      (effects (font (size 1.27 1.27)) (justify left))
+    )
+    (property "Footprint" "MountingHole:MountingHole_2.2mm_M2_Pad" (at 389.89 29.845 0)
+      (effects (font (size 1.27 1.27)) hide)
+    )
+    (property "Datasheet" "~" (at 389.89 29.845 0)
+      (effects (font (size 1.27 1.27)) hide)
+    )
+    (instances
+      (project "Front Panel Register"
+        (path "/43c9f2e1-b850-426e-8849-9d0baaf5e00b"
+          (reference "H3") (unit 1)
+        )
+      )
+    )
+  )
   (symbol (lib_id "Switch:SW_SPDT") (at 257.175 265.43 270) (unit 1)
     (in_bom yes) (on_board yes) (dnp no)
@@
     )
   )
+  (symbol (lib_id "Mechanical:MountingHole") (at 389.89 23.495 0) (unit 1)
+    (in_bom yes) (on_board yes) (dnp no) (fields_autoplaced)
+    (property "Reference" "H2" (at 392.43 22.2829 0)
+      (effects (font (size 1.27 1.27)) (justify left))
+    )
+    (property "Value" "MountingHole" (at 392.43 24.7071 0)
+      (effects (font (size 1.27 1.27)) (justify left))
+    )
+    (property "Footprint" "MountingHole:MountingHole_2.2mm_M2_Pad" (at 389.89 23.495 0)
+      (effects (font (size 1.27 1.27)) hide)
+    )
+    (property "Datasheet" "~" (at 389.89 23.495 0)
+      (effects (font (size 1.27 1.27)) hide)
+    )
+    (instances
+      (project "Front Panel Register"
+        (path "/43c9f2e1-b850-426e-8849-9d0baaf5e00b"
+          (reference "H2") (unit 1)
+        )
+      )
+    )
+  )
   (symbol (lib_id "74xx:74LS377") (at 135.89 48.26 0) (unit 1)
     (in_bom yes) (on_board yes) (dnp no) (fields_autoplaced)
@@
     )
   )
+  (symbol (lib_id "Mechanical:MountingHole") (at 389.89 17.145 0) (unit 1)
+    (in_bom yes) (on_board yes) (dnp no) (fields_autoplaced)
+    (property "Reference" "H1" (at 392.43 15.9329 0)
+      (effects (font (size 1.27 1.27)) (justify left))
+    )
+    (property "Value" "MountingHole" (at 392.43 18.3571 0)
+      (effects (font (size 1.27 1.27)) (justify left))
+    )
+    (property "Footprint" "MountingHole:MountingHole_2.2mm_M2_Pad" (at 389.89 17.145 0)
+      (effects (font (size 1.27 1.27)) hide)
+    )
+    (property "Datasheet" "~" (at 389.89 17.145 0)
+      (effects (font (size 1.27 1.27)) hide)
+    )
+    (instances
+      (project "Front Panel Register"
+        (path "/43c9f2e1-b850-426e-8849-9d0baaf5e00b"
+          (reference "H1") (unit 1)
+        )
+      )
+    )
+  )
   (symbol (lib_id "power:GND") (at 290.83 264.795 0) (mirror y) (unit 1)
     (in_bom yes) (on_board yes) (dnp no) (fields_autoplaced)
@@
         )
       )
+    )
+  )
+  (symbol (lib_id "Mechanical:MountingHole") (at 389.89 36.195 0) (unit 1)
+    (in_bom yes) (on_board yes) (dnp no) (fields_autoplaced)
+    (property "Reference" "H4" (at 392.43 34.9829 0)
+      (effects (font (size 1.27 1.27)) (justify left))
+    )
+    (property "Value" "MountingHole" (at 392.43 37.4071 0)
+      (effects (font (size 1.27 1.27)) (justify left))
+    )
+    (property "Footprint" "MountingHole:MountingHole_2.2mm_M2_Pad" (at 389.89 36.195 0)
+      (effects (font (size 1.27 1.27)) hide)
+    )
+    (property "Datasheet" "~" (at 389.89 36.195 0)
+      (effects (font (size 1.27 1.27)) hide)
+    )
+    (instances
+      (project "Front Panel Register"
+        (path "/43c9f2e1-b850-426e-8849-9d0baaf5e00b"
+          (reference "H4") (unit 1)
+        )
+      )
