File: kicad/Front Panel Register/Front Panel Register.kicad_pcb (KiCad board)
At the start: 2 copper layers, 127 parts, among them J1 Front Panel Connector, SW1 SWR0, SW10 SWR9, SW11 SWR10, SW12 SWR11, SW13 SWR12, SW14 SWR13, SW15 SWR14, SW16 SWR15, SW17 SWR16, SW18 SWR17, SW2 SWR1, SW3 SWR2, SW4 SWR3, SW5 SWR4, SW6 SWR5, SW7 SWR6, SW8 SWR7, SW9 SWR8, U1 74LS244, U10 74LS377, U11 74LS377, U12 74LS377, U2 74LS244, U3 74LS244, U4 74LS377, U5 74LS377, U6 74LS377, U7 74LS377, U8 74LS377, U9 74LS377

Commit message: Start work on front panel address layout
Parts:
- added REF**: MountingHole_2.2mm_M2_Pad, MountingHole:MountingHole_2.2mm_M2_Pad, F.Cu at (236.9, 131.4)
- added REF**: MountingHole_2.2mm_M2_Pad, MountingHole:MountingHole_2.2mm_M2_Pad, F.Cu at (40.0, 71.1)
- added REF**: MountingHole_2.2mm_M2_Pad, MountingHole:MountingHole_2.2mm_M2_Pad, F.Cu at (236.9, 71.1)
- added REF**: MountingHole_2.2mm_M2_Pad, MountingHole:MountingHole_2.2mm_M2_Pad, F.Cu at (40.0, 131.4)
- C13, J1: moved to B.Cu
- moved R18 378.1 mm to (38.1, 139.1)
- moved R17 367.7 mm to (48.9, 139.1)
- moved U12 366.0 mm to (71.8, 106.7), turned to 90 degrees
- moved R16 357.4 mm to (59.7, 139.1)
- moved R15 345.3 mm to (72.4, 139.1)
- moved C6 340.8 mm to (44.5, 68.6), turned to -90 degrees
- moved D18 337.9 mm to (40.6, 55.2)
- moved R14 335.8 mm to (82.5, 139.1)
- moved C3 335.6 mm to (59.7, 128.3), turned to -90 degrees
- moved RN8 328.7 mm to (65.4, 80.6), turned to 180 degrees
- moved RN4 328.6 mm to (65.4, 62.2), turned to 180 degrees
- moved R13 325.2 mm to (94.0, 139.1)
- moved U11 322.6 mm to (106.0, 106.7), turned to 90 degrees
- moved D17 319.6 mm to (51.4, 55.2)
- moved U9 318.9 mm to (80.0, 74.9), turned to 90 degrees
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Other:
- board outline added: 204.5 x 107.3 mm

Commit message: Continue work on backplane
Connections:
- J1 pad 27: GND -> /SYNC_CLK
- J1 pad 28: unconnected-(J1-Pin_28-Pad28) -> /DELAY_CLK
Changed lines of the file:
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@@
   (net 131 "/FP2")
   (net 132 "/FP3")
-  (net 133 "unconnected-(J1-Pin_28-Pad28)")
+  (net 133 "/SYNC_CLK")
   (net 134 "/*SELECT_SWR")
   (net 135 "/CLK_B")
@@
   (net 214 "unconnected-(U12-Q6-Pad16)")
   (net 215 "unconnected-(U12-Q7-Pad19)")
+  (net 216 "/DELAY_CLK")
   (footprint "LED_THT:LED_D5.0mm" (layer "F.Cu")
     (at 222.885 55.245)
@@
       (net 2 "GND") (pinfunction "Pin_26") (pintype "passive"))
     (pad "27" thru_hole circle (at 0 -33.02 90) (size 1.7 1.7) (drill 1) (layers "*.Cu" "*.Mask")
-      (net 2 "GND") (pinfunction "Pin_27") (pintype "passive"))
+      (net 133 "/SYNC_CLK") (pinfunction "Pin_27") (pintype "passive+no_connect"))
     (pad "28" thru_hole circle (at 2.54 -33.02 90) (size 1.7 1.7) (drill 1) (layers "*.Cu" "*.Mask")
-      (net 133 "unconnected-(J1-Pin_28-Pad28)") (pinfunction "Pin_28") (pintype "passive+no_connect"))
+      (net 216 "/DELAY_CLK") (pinfunction "Pin_28") (pintype "passive+no_connect"))
     (pad "29" thru_hole circle (at 0 -35.56 90) (size 1.7 1.7) (drill 1) (layers "*.Cu" "*.Mask")
       (net 134 "/*SELECT_SWR") (pinfunction "Pin_29") (pintype "passive"))

Commit message: Continue work on routing
Parts:
- removed REF** (x4): MountingHole_2.2mm_M2_Pad, MountingHole:MountingHole_2.2mm_M2_Pad
- added H1: MountingHole, MountingHole:MountingHole_2.2mm_M2_Pad, F.Cu at (40.0, 71.1)
- added H2: MountingHole, MountingHole:MountingHole_2.2mm_M2_Pad, F.Cu at (40.0, 131.4)
- added H3: MountingHole, MountingHole:MountingHole_2.2mm_M2_Pad, F.Cu at (236.9, 71.1)
- added H4: MountingHole, MountingHole:MountingHole_2.2mm_M2_Pad, F.Cu at (236.9, 131.4)
Routing:
- net GND: track 0.00 -> 857.2 mm
- net +5V: track 0.00 -> 676.7 mm
- net /CLK_B: track 0.00 -> 313.7 mm, vias 0 -> 1
- net /D16: track 0.00 -> 236.9 mm
- net /D15: track 0.00 -> 229.1 mm
- net /D17: track 0.00 -> 228.1 mm
- net /D14: track 0.00 -> 218.8 mm
- net /D13: track 0.00 -> 214.2 mm
- net /*LATCH_MB: track 0.00 -> 210.5 mm, vias 0 -> 1
- net /D9: track 0.00 -> 201.9 mm, vias 0 -> 1
- net /D2: track 0.00 -> 199.1 mm
- net /D6: track 0.00 -> 198.1 mm
- net /D12: track 0.00 -> 193.5 mm, vias 0 -> 2
- net /*SELECT_SWR: track 0.00 -> 189.1 mm
- net /D0: track 0.00 -> 183.4 mm, vias 0 -> 2
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- added copper zone on B.Cu, net GND
- added copper zone on F.Cu, net GND
Other:
- board text added: "Gavin Tersteeg, 2026"
- board text added: "JLCJLCJLCJLC"
- board text added: "RDP-9A-FPR-0"

Commit message: Gerber creation marathon
Routing:
- net /D1: track 166.8 -> 188.9 mm, vias 3 -> 1
- net /D9: track 201.9 -> 181.1 mm, vias 1 -> 0
- net /D12: track 193.5 -> 213.8 mm, vias 2 -> 0
- net /*LATCH_MB: track 210.5 -> 191.4 mm
- net Net-(D35-A): track 33.8 -> 52.8 mm, vias 1 -> 0
- net /D6: track 198.1 -> 179.7 mm
- net Net-(D12-A): track 54.6 -> 36.7 mm, vias 0 -> 1
- net /D15: track 229.1 -> 212.9 mm
- net Net-(D21-A): track 46.9 -> 32.1 mm, vias 0 -> 1
- net +5V: track 676.7 -> 662.0 mm
- net /D5: track 171.7 -> 186.2 mm, vias 1 -> 3
- net Net-(D47-A): track 17.0 -> 31.5 mm, vias 1 -> 0
- net Net-(D31-A): track 82.5 -> 94.9 mm, vias 1 -> 0
- net Net-(D38-A): track 84.9 -> 95.6 mm
- net GND: track 857.2 -> 867.5 mm
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Other:
- board text removed: "JLCJLCJLCJLC"
