File: kicad/TTY Clock/TTY Clock.kicad_sch (KiCad schematic)
At the start: 22 parts, among them J1 I/O Connector, J2 Custom Clock, SW1 UART 1 Settings, SW2 UART 2 Settings, U1 74LS169, U2 74LS169, U3 74LS169, U4 74LS169, U5 74LS00, U6 74LS151, U7 74LS151, U8 TR1863, U9 TR1863, X1 2.4576 Mhz Oscillator

Commit message: Continue work on TTY clock schematic
Parts:
- added C1, C2, C3, C4: 1.0 uF, Capacitor_THT:CP_Radial_D5.0mm_P2.00mm, symbol Device:C_Polarized
- added J3: TTL Serial 0, Connector_PinHeader_2.54mm:PinHeader_1x06_P2.54mm_Horizontal, symbol Connector:Conn_01x06_Male
- added J4: TTL Serial 1, Connector_PinHeader_2.54mm:PinHeader_1x06_P2.54mm_Horizontal, symbol Connector:Conn_01x06_Male
- added J5: RS232 Serial 0, Connector_IDC:IDC-Header_2x05_P2.54mm_Vertical, symbol Connector_Generic:Conn_02x05_Counter_Clockwise
- added J6: RS232 Serial 1, Connector_IDC:IDC-Header_2x05_P2.54mm_Vertical, symbol Connector_Generic:Conn_02x05_Counter_Clockwise
- added JP1: RX0 Select, Connector_PinHeader_2.54mm:PinHeader_1x03_P2.54mm_Vertical, symbol Jumper:Jumper_3_Bridged12
- added JP2: RX1 Select, Connector_PinHeader_2.54mm:PinHeader_1x03_P2.54mm_Vertical, symbol Jumper:Jumper_3_Bridged12
- added R10, R11, R12, R13, R14, R15, R16, R17, R18, R19, R20, R21, R22, R23, R24, R9: 4.7K, symbol Device:R
- added U10: MAX232, Package_DIP:DIP-16_W7.62mm, symbol Interface_UART:MAX232
Connections:
- net +5V: now also C2.2, R10.1, R11.1, R12.1, R13.1, R14.1, R15.2, R16.2, R17.2, R18.2, R19.2, R20.2, R21.2, R22.2, R23.2, R24.2, R9.1, U10.16 (VCC)
- net GND: now also U8.16 (SFD), U9.16 (SFD), C3.1, J3.1 (Pin_1), J4.1 (Pin_1), J5.5 (Pin_5), J6.5 (Pin_5), U10.15 (GND)
- net at U7.10 (S1): now also SW2.2, R13.2
- net at U7.11 (S0): now also SW2.1, R12.2
- net at U7.9 (S2): now also SW2.3, R14.2
- net at U8.20 (RI): now also JP1.2 (C)
- net at U8.25 (TRO): now also J3.4 (Pin_4), U10.11 (T1IN)
- net at U8.35 (PI): now also SW1.8, R19.1
- net at U8.36 (SBS): now also SW1.7, R18.1
- net at U8.37 (WLS2): now also SW1.6, R17.1
- net at U8.38 (WLS1): now also SW1.5, R16.1
- net at U8.39 (EPE): now also SW1.4, R15.1
- net at SW1.1, U6.11 (S0): now also R9.2
- net at SW1.2, U6.10 (S1): now also R10.2
- net at SW1.3, U6.9 (S2): now also R11.2
- net at SW2.4: now also U9.39 (EPE), R20.1
- net at SW2.5: now also U9.38 (WLS1), R21.1
- net at SW2.6: now also U9.37 (WLS2), R22.1
- net at SW2.7: now also U9.36 (SBS), R23.1
- net at SW2.8: now also U9.35 (PI), R24.1
- net at U9.20 (RI): now also JP2.2 (C)
- net at U9.25 (TRO): now also J4.4 (Pin_4), U10.10 (T2IN)
- new net: JP1.1 (A), U10.12 (R1OUT)
- new net: J3.3 (Pin_3), JP1.3 (B)
- new net: C2.1, U10.2 (VS+)
- new net: C3.2, U10.6 (VS-)
- new net: C1.1, U10.1 (C1+)
- new net: J5.2 (Pin_2), U10.13 (R1IN)
- new net: J5.3 (Pin_3), U10.14 (T1OUT)
- new net: C1.2, U10.3 (C1-)
- new net: C4.1, U10.4 (C2+)
- new net: C4.2, U10.5 (C2-)
- new net: J6.3 (Pin_3), U10.7 (T2OUT)
- new net: J6.2 (Pin_2), U10.8 (R2IN)
- new net: JP2.1 (A), U10.9 (R2OUT)
- new net: J4.3 (Pin_3), JP2.3 (B)
- no-connect marks 14 -> 34
Other:
- moved on the sheet: SW1, SW2

Commit message: Continue work on TTY / clock
Parts:
- added R25, R26: 4.7K, symbol Device:R
- added U11, U12, U13: 74LS240, symbol 74xx:74LS240
- added U14, U15: 74LS244, symbol 74xx:74LS244
- added U16, U17, U18: 74LS32, symbol 74xx:74LS32
- added U19: 74LS06, symbol 74xx:74LS06
Connections:
- net *DRQ_GRANT: now also U5.12, U5.13
- net *IOT_PULSE: now also U16.5
- net *PI_ENABLE: now also U13.4 (I1a)
- net *PTP_FLAG: now also U12.17 (I3b)
- net *PTP_TAPE: now also U12.2 (I0a)
- net *PTR_FLAG: now also U13.2 (I0a)
- net *PTR_TAPE: now also U12.4 (I1a)
- net +5V: now also R25.1, R26.1, U11.20 (VCC), U12.20 (VCC), U13.20 (VCC), U14.20 (VCC), U15.20 (VCC)
- net A_DEVICE0: now also U5.9, U16.9
- net A_DEVICE1: now also U5.10, U16.10
- net A_DEVICE2: now also U5.4, U5.5, U17.2
- net A_DEVICE3: now also U16.1
- net A_DEVICE4: now also U16.2
- net A_DEVICE5: now also U16.4
- net D0: now also U11.18 (O0a), U14.18 (O0a)
- net D1: now also U11.16 (O1a), U14.16 (O1a)
- net D10: now also U12.14 (O2a), U15.14 (O2a)
- net D11: now also U12.12 (O3a), U15.12 (O3a)
- net D12: now also U12.9 (O0b), U15.9 (O0b)
- net D13: now also U12.7 (O1b), U15.7 (O1b)
- net D14: now also U12.5 (O2b), U15.5 (O2b)
- net D15: now also U12.3 (O3b), U15.3 (O3b)
- net D16: now also U13.18 (O0a), U13.9 (O0b)
- net D17: now also U13.16 (O1a), U13.7 (O1b)
- net D2: now also U11.14 (O2a), U14.14 (O2a)
- net D3: now also U11.12 (O3a), U14.12 (O3a)
- net D4: now also U11.9 (O0b), U14.9 (O0b)
- net D5: now also U11.7 (O1b), U14.7 (O1b)
- net D6: now also U11.5 (O2b), U14.5 (O2b)
- net D7: now also U11.3 (O3b), U14.3 (O3b)
- net D8: now also U12.18 (O0a), U15.18 (O0a)
- net D9: now also U12.16 (O1a), U15.16 (O1a)
- net GND: now also U11.10 (GND), U12.10 (GND), U13.10 (GND), U13.15 (I2b), U13.17 (I3b), U13.6 (I2a), U13.8 (I3a), U14.10 (GND), U14.11 (I0b), U14.13 (I1b), U14.15 (I2b), U14.17 (I3b), U14.8 (I3a), U15.10 (GND), U15.11 (I0b), U15.13 (I1b), U15.15 (I2b), U15.17 (I3b), U15.2 (I0a), U15.4 (I1a), U15.6 (I2a), U15.8 (I3a)
- net at U5.8: now also U18.2
- net at U5.6: now also U17.10
- net at U5.11: now also U14.2 (I0a), U14.4 (I1a), U14.6 (I2a)
- new net: U17.3, U17.5, U18.1
- new net: U16.11, U17.1, U17.9
- new net: U16.12, U16.3
- new net: U16.13, U16.6
- new net: U14.1 (OEa), U14.19 (OEb)
- new net: R25.2, U13.11 (I0b)
- new net: U16.8, U17.12, U17.4
- new net: U17.13, U17.8
- new net: U15.1 (OEa), U15.19 (OEb)
- new net: R26.2, U13.13 (I1b)
- new net: U11.1 (OEa), U11.19 (OEb)
- new net: U12.1 (OEa), U12.19 (OEb)
- new net *KEYBD_EN: U18.3
- new net *PRINT_EN: U17.11
- new net *RTC_EN: U17.6
- no-connect marks 34 -> 48
Other:
- moved on the sheet: C1, C2, C3, C4, J1, J2, J3, J4, J5, J6, JP1, JP2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

Commit message: Continue work on TTY clock card
Parts:
- added R27, R28, R29, R30: 4.7K, symbol Device:R
Connections:
- net *DRQ_GRANT: now also U14.1 (OEa), U14.19 (OEb), U18.4; no longer U5.12, U5.13
- net *EXTERNAL: now also U19.2
- net +5V: now also R27.1, R28.1, R29.1, R30.1
- net at U15.1 (OEa), U15.19 (OEb): now also U13.19 (OEb), U18.6, U18.9
- net at U13.1 (OEa): now also U11.1 (OEa), U11.19 (OEb), U12.1 (OEa), U12.19 (OEb), U18.10
- net at U18.8: now also U19.3
- net at U19.1: now also U19.4, R30.2
- new net: R27.2, U14.2 (I0a)
- new net: R28.2, U14.4 (I1a)
- new net: R29.2, U14.6 (I2a)
- now unconnected: U5.11
Other:
- moved on the sheet: U18B, U18C, U19A, U19B, U5D

Commit message: Continue work on TTY clock
Parts:
- added U20: 74LS04, symbol 74xx:74LS04
- added U21: 74LS32, symbol 74xx:74LS32
Connections:
- net *CAF: now also U20.9
- net *KEYBD_EN: now also U18.12
- net A_PULSE0: now also U20.1
- net A_PULSE1: now also U20.3
- net A_PULSE2: now also U20.5
- net CAF: now reaches U8.21 (MR)
- net CAF: now also U9.21 (MR), U20.8
- net at U11.1 (OEa), U11.19 (OEb), U12.1 (OEa)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: now also U18.11
- net *A_PULSE2: now reaches U18.13
- net *A_PULSE2: now also U20.6
- new net *A_PULSE0: U20.2
- new net *A_PULSE1: U20.4
Other:
- moved on the sheet: U18D, U19C, U5D

Commit message: Continue work on TTY clock
Parts:
- added R31, R32, R33, R34, R35: 4.7K, symbol Device:R
- added U22, U27, U28, U29, U30: 74LS74, symbol 74xx:74LS74
- added U23, U26: 74LS32, symbol 74xx:74LS32
- added U24: 74LS02, symbol 74xx:74LS02
- added U25: 74LS257, symbol 74xx:74LS257
Connections:
- net *A_PULSE0: now also U24.3, U24.8
- net *A_PULSE1: now also U23.10, U26.1
- net *A_PULSE2: now also U23.12
- net *CAF: now also U23.1, U23.4
- net *IOT_SKIP: now also U19.10, U19.8
- net *KEYBD_EN: now also U23.9, U24.2
- net *PRINT_EN: now also U23.13, U24.9, U26.2
- net *RTC_EN: now also U26.5
- net +5V: now also R31.1, R32.1, R33.1, R34.1, R35.1, U25.16 (VCC)
- net A_DEVICE2: now also U24.5; no longer U5.4, U5.5
- net A_SUBDEV0: now also U20.11, U21.1, U21.5, U25.1 (S)
- net GND: now also U25.10 (I1d), U25.11 (I0d), U25.13 (I1c), U25.14 (I0c), U25.15 (OE), U25.8 (GND)
- net at U19.11: now also U20.12
- net at U21.11: now also U9.23 (~{THRL})
- net *PRINT_WR: now reaches U21.12
- net *PRINT_WR: now also U21.4, U23.11
- net *A_SUBDEV0: now reaches U21.13
- net *A_SUBDEV0: now also U20.10, U21.9
- net 60_HZ: now reaches U4.9 (~{PE}), U5.3
- net at U8.18 (~{DRR}): now also U21.3, U8.4 (RRD)
- net RECV_FLAG_0: now reaches U8.19 (DR)
- net RECV_FLAG_0: now also U25.2 (I0a)
- net at U8.22 (THRE): now also U22.3 (C)
- net at U8.23 (~{THRL}): now also U21.6
- net at U17.10: now also U24.4; no longer U5.6
- net at U5.11: now also U20.13
- net at U5.12: now also U25.7 (Zb)
- net PRINT_SKIP: now reaches U5.13
- net PRINT_SKIP: now also U24.10
- net *KEYBD_RD: now reaches U18.5
- net *KEYBD_RD: now also U21.10, U21.2, U23.8
- net at U21.8: now also U9.4 (RRD)
- net at U19.5: now also U5.6
- net at U19.6: now also U19.9, R35.2
- net RECV_FLAG_1: now reaches U9.19 (DR)
- net RECV_FLAG_1: now also U25.3 (I1a)
- net at U9.22 (THRE): now also U22.11 (C)
- new net: R32.2, U22.4 (~{S})
- new net: R34.2, U22.10 (~{S})
- new net: R33.2, U22.12 (D)
- new net: U22.13 (~{R}), U23.6
- new net: U25.4 (Za), U5.4
- new net: U22.1 (~{R}), U23.3
- new net: R31.2, U22.2 (D)
- new net *PRINT_RES: U23.2, U23.5, U26.3
- new net KEYBD_SKIP: U24.1, U5.5
- new net TRNS_FLAG_0: U22.5 (Q), U25.5 (I0b)
- new net TRNS_FLAG_1: U22.9 (Q), U25.6 (I1b)
- no-connect marks 48 -> 53
Other:
- moved on the sheet: U19C, U19D, U19E, U19F, U20E, U20F, U21A, U21B, U21C, U21D, U5B, U5D
