File: kicad/TTY Clock/TTY Clock.kicad_sch (KiCad schematic)
At the start: 80 parts, among them J1 I/O Connector, J2 Custom Clock, J3 TTL Serial 0, J4 TTL Serial 1, J5 RS232 Serial 0, J6 RS232 Serial 1, SW1 UART 1 Settings, SW2 UART 2 Settings, U1 74LS169, U10 MAX232, U11 74LS240, U12 74LS240, U13 74LS240, U14 74LS244, U15 74LS244, U16 74LS32, U17 74LS32, U18 74LS32, U19 74LS06, U2 74LS169, U20 74LS04, U21 74LS32, U22 74LS74, U23 74LS32, U24 74LS02, U25 74LS257, U26 74LS32, U27 74LS74, U28 74LS74, U29 74LS74, U3 74LS169, U30 74LS74, U4 74LS169, U5 74LS00, U6 74LS151, U7 74LS151, U8 TR1863, U9 TR1863, X1 2.4576 Mhz Oscillator

Commit message: Continue work on TTY clock card
Connections:
- net RECV_FLAG_0: now also U12.15 (I2b)
- net TRNS_FLAG_0: now also U12.13 (I1b)
Other:
- moved on the sheet: R35, U19C, U19D, U19E, U20F, U25, U5B, U5D

Commit message: Continue work on Clock TTY card
Parts:
- added R36, R37, R38, R39, R40, R41, R42, R43, R44, R45, R46, R47: 4.7K, symbol Device:R
- added SW3: IORS 0 Settings, symbol Switch:SW_DIP_x08
- added SW4: IORS 1 Settings, symbol Switch:SW_DIP_x08
- added SW5: IORS 2 Settings, symbol Switch:SW_DIP_x08
- added SW6: IORS 3 Settings, symbol Switch:SW_DIP_x08
- added U31: 74LS32, symbol 74xx:74LS32
- added U32: 74LS08, symbol 74xx:74LS08
Connections:
- net *CHAN_REQ is gone; now on net *RTC_PENDING: J1.b27 (Pin_b27)
- net *DMA_REQ is gone; now on net *RTC_PENDING: J1.b26 (Pin_b26)
- net *A_PULSE1: now also U26.4
- net *A_PULSE2: now also U26.9
- net *CAF: now also U32.2
- net *DRQ_GRANT: now also U26.12, U27.10 (~{S})
- net *INCREMENT_ZERO: now also U26.13
- net *IORS_FLAG0: now also SW3.10, SW3.11, SW3.12, SW3.13, SW3.14, SW3.15, SW3.16, SW3.9
- net *IORS_FLAG1: now also SW4.10, SW4.11, SW4.12, SW4.13, SW4.14, SW4.15, SW4.16, SW4.9
- net *IORS_FLAG2: now also SW5.10, SW5.11, SW5.12, SW5.13, SW5.14, SW5.15, SW5.16, SW5.9
- net *IORS_FLAG3: now also SW6.10, SW6.11, SW6.12, SW6.13, SW6.14, SW6.15, SW6.16, SW6.9
- net *PI_ENABLE: now also U27.6 (~{Q})
- net *RESET: now also U28.1 (~{R})
- net *RTC_EN: now also U26.10
- net +5V: now also R36.1, R37.1, R38.1, R39.1, R40.1, R41.1, R42.1, R43.1, R44.1, R45.1, R46.1, R47.1
- net 60_HZ: now also U31.2
- net A_DEVICE0: now also U32.4; no longer U5.9
- net A_DEVICE1: now also U32.5; no longer U5.10
- net A_DEVICE3: now also U32.9
- net A_DEVICE4: now also U32.10
- net A_SUBDEV1: now also U27.2 (D), U28.2 (D)
- net GND: now also U27.11 (C), U27.12 (D), U28.11 (C), U28.12 (D)
- net at U18.2: now also U24.13; no longer U5.8
- net at U28.10 (~{S}): now also U26.11
- net at U28.13 (~{R}): now also U32.3
- net *RTC_FLAG: now reaches U28.8 (~{Q})
- net *RTC_FLAG: now also U12.8 (I3a)
- net at U24.12: now also U32.6
- net *SET_RTC_EN: now reaches U28.3 (C)
- net *SET_RTC_EN: now also U12.6 (I2a), U26.8, U32.1
- net at U28.4 (~{S}): now also R47.2
- net *RTC_ENABLE: now reaches U28.6 (~{Q})
- net *RTC_ENABLE: now also U31.1
- net *SET_PI: now reaches U26.6
- net *SET_PI: now also U27.3 (C)
- net at U27.13 (~{R}): now also U31.3
- net *RTC_PENDING: now reaches U27.9 (Q)
- net at U27.1 (~{R}): now also R46.2
- net at U27.4 (~{S}): now also R45.2
- net IORS4: now reaches U11.11 (I0b)
- net IORS4: now also R40.2, SW3.5, SW4.5, SW5.5, SW6.5
- net IORS5: now reaches U11.13 (I1b)
- net IORS5: now also R41.2, SW3.6, SW4.6, SW5.6, SW6.6
- net IORS6: now reaches U11.15 (I2b)
- net IORS6: now also R42.2, SW3.7, SW4.7, SW5.7, SW6.7
- net IORS7: now reaches U11.17 (I3b)
- net IORS7: now also R43.2, SW3.8, SW4.8, SW5.8
- net IORS0: now reaches U11.2 (I0a)
- net IORS0: now also R36.2, SW3.1, SW4.1, SW5.1, SW6.1
- net IORS1: now reaches U11.4 (I1a)
- net IORS1: now also R37.2, SW3.2, SW4.2, SW5.2, SW6.2
- net IORS2: now reaches U11.6 (I2a)
- net IORS2: now also R38.2, SW3.3, SW4.3, SW5.3, SW6.3
- net IORS3: now reaches U11.8 (I3a)
- net IORS3: now also R39.2, SW3.4, SW4.4, SW5.4, SW6.4
- net at U12.11 (I0b): now also R44.2, SW6.8
- no-connect marks 53 -> 57
Other:
- moved on the sheet: U24D, U26C, U26D, U27A, U27B, U28A, U28B, U5C

Commit message: Continue work on Clock TTY card
Parts:
- removed R46: 4.7K, symbol Device:R
- added U33: 74LS08, symbol 74xx:74LS08
- added U34: 74LS04, symbol 74xx:74LS04
Connections:
- net *CAF_REQ: now also U34.8
- net *INT_DETECT: now also U27.1 (~{R})
- net *IOT_PULSE: now also U31.10
- net *IOT_SKIP: now also U19.6
- net *JMP_I_DETECT: now also U29.3 (C)
- net *REST_PEND: now also U29.6 (~{Q})
- net +5V: now also R35.2; no longer R35.1
- net A_DEVICE2: now also U31.4, U32.12, U34.5; no longer U24.5
- net A_DEVICE5: now also U31.5, U32.13
- net A_PULSE0: now also U33.2
- net A_PULSE1: now also U33.4
- net A_PULSE2: now also U33.9
- net A_SUBDEV0: no longer U20.11, U21.1, U21.5
- net A_SUBDEV1: now also U20.11, U21.1, U21.5, U33.10
- net GND: now also U29.2 (D)
- net at U18.2: now also U34.12; no longer U24.13
- net *MEM_EN: now reaches U31.11
- net at U31.12: now also U24.5, U31.8
- net at U31.13: now also U34.4
- net at U32.6: now also U5.9, U34.13; no longer U24.12
- net at U17.10: now also U34.6; no longer U24.4
- net at U24.6: now also U31.6
- net at U31.9: now also U5.8
- net at U32.11: now also U34.3
- net at U5.10: now also U32.8
- net at U19.5: now also U33.3; no longer U5.6
- net at U29.1 (~{R}): now also R35.1
- net at U29.4 (~{S}): now also U34.10
- net *A_SUBDEV0 renamed *A_SUBDEV1
- new net: U33.11, U34.11
- new net: U34.1, U5.6
- new net: U33.6, U34.9
- new net: U19.9, U34.2
- new net: U33.12, U33.8
- new net API_EN: U24.4, U33.1, U33.13, U33.5
- no-connect marks 57 -> 58
Other:
- moved on the sheet: U19C, U24B, U24D, U29A, U31B, U31C, U31D, U32D, U5C

Commit message: Continue work on TTY clock card
Parts:
- removed U17, U26, U31: 74LS32, symbol 74xx:74LS32
- removed U24: 74LS02, symbol 74xx:74LS02
- removed U33: 74LS08, symbol 74xx:74LS08
- removed unit 2 of U34
- removed unit 5 of U34
- removed unit 6 of U34
- removed unit 7 of U34
- removed unit 3 of U34
- removed unit 4 of U34
- added R47, R48: 4.7K, symbol Device:R
- added U32, U34: 74LS32, symbol 74xx:74LS32
- added U33: 74LS02, symbol 74xx:74LS02
- added U8, U9: 74LS138, symbol 74xx:74LS138
- renumbered R36 to R1, R30 to R10, R25 to R11, R26 to R12, R2 to R13, R1 to R14, R27 to R15, R28 to R16, R29 to R17, R3 to R18, R4 to R19, R37 to R2, R45 to R20, R5 to R21, R6 to R22, R35 to R23, R9 to R24, R10 to R25, R11 to R26, R12 to R27, R13 to R28, R14 to R29, R38 to R3, R8 to R30, R7 to R31, R15 to R32, R16 to R33, R17 to R34, R18 to R35, R19 to R36, R20 to R37, R21 to R38, R22 to R39, R39 to R4, R23 to R40, R24 to R41, R47 to R42, R31 to R43, R33 to R44, R32 to R45, R34 to R46, R40 to R5, R41 to R6, R42 to R7, R43 to R8, R44 to R9, SW3 to SW1, SW4 to SW2, SW5 to SW3, SW6 to SW4, SW1 to SW5, SW2 to SW6, U18 to U1, U13 to U10, U1 to U11, U14 to U12, U27 to U13, U2 to U14, U30 to U15, U15 to U16, U29 to U17, U3 to U18, U5 to U19, U20 to U2, U4 to U20, U6 to U21, U7 to U22, U21 to U23, U23 to U24, U22 to U25, U8 to U26, U9 to U27, U25 to U29, U11 to U3, U10 to U30, U34 to U31, U16 to U4, U32 to U5, U12 to U6, U19 to U7
Connections:
- net *A_PULSE0: now also U33.12, U33.3, U33.6, U33.9, U34.13
- net *A_PULSE1: now also U5.9, U32.10, U32.13, U32.2, U34.5; no longer U24.10
- net *A_PULSE2: now also U5.10, U32.5, U34.10, U34.2; no longer U24.12
- net *CAF_REQ: now also U34.6
- net *DRQ_GRANT: now also U24.9
- net *INCREMENT_ZERO: now also U24.10
- net *IOT_PULSE: now also U8.4 (E1), U9.4 (E1); no longer U4.5
- net *IOT_SKIP: now also U7.12
- net *KEYBD_EN: now also U4.6, U32.9, U33.5; no longer U1.3, U24.9
- net *KEYBD_RD: now also U32.8; no longer U24.8
- net *MEMM_ENABLE: now also U17.8 (~{Q})
- net *MEM_EN: now also U1.3, U34.12
- net *PRINT_EN: now also U4.8, U32.12, U33.8, U34.1; no longer U24.13
- net *PRINT_RES: now also U32.11
- net *PRINT_WR: now also U34.3; no longer U24.11
- net *RTC_EN: now also U4.3, U32.1, U32.4, U33.2
- net *RTC_ENABLE: now also U24.12
- net *SET_PI: now also U32.3
- net *SET_RTC_EN: now also U32.6
- net +5V: now also R47.1, R48.1, U8.16 (VCC), U9.16 (VCC)
- net 60_HZ: now also U24.13
- net A_DEVICE0: now also U9.1 (A0); no longer U4.9, U5.4
- net A_DEVICE1: now also U9.2 (A1); no longer U4.10, U5.5
- net A_DEVICE2: now also U9.3 (A2); no longer U5.12
- net A_DEVICE3: now also U8.1 (A0); no longer U4.1, U5.9
- net A_DEVICE4: now also U8.2 (A1); no longer U4.2, U5.10
- net A_DEVICE5: now also U8.3 (A2); no longer U4.4, U5.13
- net A_SUBDEV0: no longer U29.1 (S)
- net A_SUBDEV1: now also U29.1 (S)
- net GND: now also U8.5 (E2), U8.8 (GND), U9.5 (E2), U9.8 (GND)
- net KEYBD_SKIP: now also U33.4
- net PRINT_SKIP: now also U33.10
- net at U1.1: now also U9.7 (O7)
- net at U1.2: now also U8.7 (O7)
- net *API_EN: now reaches U4.11
- net *API_EN: now also U33.11, U34.4, U34.9
- net MEMM_ENABLE: now reaches U17.9 (Q)
- net MEMM_ENABLE: now also U5.13
- net at U5.6: now also U7.13; no longer U19.9
- net at U4.12: now also U4.4, U9.12 (O3); no longer U4.3
- net at U4.13: now also U8.12 (O3); no longer U4.6
- net at U7.5: now also U33.13
- net at U19.8: now also U5.12
- net at U28.10 (~{S}): now also U24.8
- net RTC_FLAG: now reaches U28.9 (Q)
- net RTC_FLAG: now also U5.4
- net *REST_SET: now reaches U17.4 (~{S})
- net *REST_SET: now also U34.8
- net at U19.10: now also U19.9, U34.11; no longer U5.8
- net at U13.13 (~{R}): now also U24.11
- new net: R47.2, U9.6 (E3)
- new net: U33.1, U5.5
- new net: U4.10, U4.2, U4.5, U8.15 (O0)
- new net: R48.2, U8.6 (E3)
- new net: U4.1, U9.15 (O0)
- new net: U4.9, U9.11 (O4)
- new net *A_PULSE12: U5.8
- no-connect marks 58 -> 66
Other:
- moved on the sheet: U15A, U17B, U19C, U1A, U24C, U24D, U4A, U4B, U4C, U4D, U4E, U5B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

Commit message: Finish initial TTY clock schematic
Parts:
- removed J3: TTL Serial 0, Connector_PinHeader_2.54mm:PinHeader_1x06_P2.54mm_Horizontal, symbol Connector:Conn_01x06_Male
- removed J4: TTL Serial 1, Connector_PinHeader_2.54mm:PinHeader_1x06_P2.54mm_Horizontal, symbol Connector:Conn_01x06_Male
- removed U31: 74LS04, symbol 74xx:74LS04
- added C10, C11, C12, C13, C14, C15, C16, C17, C18, C19, C20, C21, C22, C23, C24, C25, C26, C27, C28, C29, C30, C31, C32, C33, C34, C35, C36, C37, C38, C39, C40, C5, C6, C7, C8, C9: 0.1uF, symbol Device:C
- added C20: 100 uF, Capacitor_THT:CP_Radial_D6.3mm_P2.50mm, symbol Device:C_Polarized
- added J3: TTL Serial 0, symbol Connector_Generic:Conn_01x06
- added J4: TTL Serial 1, symbol Connector_Generic:Conn_01x06
- added R49, R50: 4.7K, symbol Device:R
- added U20: 74LS02, symbol 74xx:74LS02
- added U23: 74LS32, symbol 74xx:74LS32
- added U36: 74LS06, symbol 74xx:74LS06
- renumbered R47 to R10, R48 to R11, R11 to R12, R12 to R13, R20 to R14, R13 to R15, R14 to R16, R15 to R17, R16 to R18, R17 to R19, R23 to R20, R18 to R21, R19 to R22, R10 to R23, R21 to R24, R22 to R25, R24 to R26, R25 to R27, R26 to R28, R27 to R29, R28 to R30, R29 to R31, R30 to R32, R31 to R33, R32 to R34, R33 to R35, R34 to R36, R35 to R37, R36 to R38, R37 to R39, R38 to R40, R39 to R41, R40 to R42, R41 to R43, R42 to R44, R43 to R45, R44 to R46, R45 to R47, R46 to R48, U7 to U10, U19 to U11, U4 to U12, U34 to U13, U10 to U14, U13 to U15, U11 to U16, U12 to U18, U14 to U19, U15 to U21, U16 to U22, U18 to U24, U23 to U25, U20 to U26, U21 to U27, U22 to U28, U24 to U29, U5 to U3, U25 to U30, U28 to U31, U26 to U32, U27 to U33, U29 to U34, U30 to U35, U3 to U4, U33 to U5, U32 to U6, U6 to U7, U9 to U8, U8 to U9
Connections:
- net *A_PULSE0: now also U20.3; no longer U13.13
- net *A_PULSE12: now also U13.13
- net *A_PULSE2: now also U17.12 (D)
- net *A_SUBDEV1: now also U1.10
- net *INT_REQ: now also U36.2, U36.4, U36.6
- net *IOT_SKIP: now also U10.4
- net *JMP_I_DETECT: now also U21.3 (C), U23.1
- net *MEM_EN: now also U1.9, U20.2
- net *REST_PEND: now also U23.5
- net +5V: now also U1.14 (VCC), U10.14 (VCC), U11.14 (VCC), U12.14 (VCC), U13.14 (VCC), U15.14 (VCC), U17.14 (VCC), U2.14 (VCC), U21.14 (VCC), U25.14 (VCC), U29.14 (VCC), U3.14 (VCC), U30.14 (VCC), U31.14 (VCC), U5.14 (VCC), U6.14 (VCC), C10.1, C11.1, C12.1, C13.1, C14.1, C15.1, C16.1, C17.1, C18.1, C19.1, C20.1, C20.1, C21.1, C22.1, C23.1, C24.1, C25.1, C26.1, C27.1, C28.1, C29.1, C30.1, C31.1, C32.1, C33.1, C34.1, C35.1, C36.1, C37.1, C38.1, C39.1, C40.1, C5.1, C6.1, C7.1, C8.1, C9.1, R49.1, R50.1, U20.14 (VCC), U23.14 (VCC), U36.14 (VCC)
- net D0: now also U32.12 (RR1), U32.26 (TR1), U33.12 (RR1), U33.26 (TR1)
- net D1: now also U32.11 (RR2), U32.27 (TR2), U33.11 (RR2), U33.27 (TR2)
- net D16: now also U23.12
- net D2: now also U32.10 (RR3), U32.28 (TR3), U33.10 (RR3), U33.28 (TR3)
- net D3: now also U32.29 (TR4), U32.9 (RR4), U33.29 (TR4), U33.9 (RR4)
- net D4: now also U32.30 (TR5), U32.8 (RR5), U33.30 (TR5), U33.8 (RR5)
- net D5: now also U32.31 (TR6), U32.7 (RR6), U33.31 (TR6), U33.7 (RR6)
- net D6: now also U32.32 (TR7), U32.6 (RR7), U33.32 (TR7), U33.6 (RR7)
- net D7: now also U32.33 (TR8), U32.5 (RR8), U33.33 (TR8), U33.5 (RR8)
- net GND: now also U1.7 (GND), U10.7 (GND), U11.7 (GND), U12.7 (GND), U13.7 (GND), U15.7 (GND), U17.7 (GND), U2.7 (GND), U21.11 (C), U21.12 (D), U21.2 (D), U21.7 (GND), U25.7 (GND), U29.7 (GND), U3.7 (GND), U30.7 (GND), U31.7 (GND), U5.7 (GND), U6.7 (GND), C10.2, C11.2, C12.2, C13.2, C14.2, C15.2, C16.2, C17.2, C18.2, C19.2, C20.2, C20.2, C21.2, C22.2, C23.2, C24.2, C25.2, C26.2, C27.2, C28.2, C29.2, C30.2, C31.2, C32.2, C33.2, C34.2, C35.2, C36.2, C37.2, C38.2, C39.2, C40.2, C5.2, C6.2, C7.2, C8.2, C9.2, J3.1 (Pin_1), J4.1 (Pin_1), U20.7 (GND), U23.13, U23.7 (GND), U36.11, U36.13, U36.7 (GND), U36.9
- net RECV_FLAG_0: now also U36.5
- net RTC_FLAG: now also U36.1
- net TRNS_FLAG_0: now also U36.3
- net at U17.10 (~{S}): now also U23.6
- net *MEMM_SET: now reaches U17.11 (C)
- net *MEMM_SET: now also U13.11
- net at U17.13 (~{R}): now also U23.8
- net at JP1.3 (B): now also J3.3 (Pin_3)
- net at U32.25 (TRO), U35.11 (T1IN): now also J3.4 (Pin_4)
- net at U3.11: now also U10.3
- net at U3.12: now also U20.1; no longer U11.8
- net at U33.25 (TRO), U35.10 (T2IN): now also J4.4 (Pin_4)
- net at U1.6, U14.19 (OEb), U22.1 (OEa)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: now also U11.9; no longer U1.9
- net at U11.6: now also U20.8, U20.9
- net at U1.11, U14.1 (OEa), U4.1 (OEa)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: now also U11.10; no longer U1.10
- net at U25.8, U33.4 (RRD): now also U33.18 (~{DRR})
- net at JP2.3 (B): now also J4.3 (Pin_3)
- net at U10.9: now also U20.10
- net at U21.1 (~{R}): now also R23.2
- net *EMIR_SET: now reaches U21.4 (~{S})
- net *EMIR_SET: now also U1.8
- net EMIR_PEND: now reaches U21.5 (Q)
- net EMIR_PEND: now also U20.11
- net REST_PEND: now reaches U17.5 (Q)
- net REST_PEND: now also U20.12
- net at U21.10 (~{S}): now also R49.2
- net at U21.13 (~{R}): now also R50.2
- net *SET_PI renamed *PI_SET
- new net: U10.1, U11.8
- new net: U20.13, U23.9
- new net: U20.4, U23.4
- new net: U20.5, U20.6, U23.11, U23.2
- new net: U23.10, U23.3
- no-connect marks 66 -> 76
Other:
- moved on the sheet: R14, R20, R23, U10A, U10B, U10G, U11C, U11E, U12E, U13D, U13E, U15A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

Commit message: The great PCB layout-athon
Parts:
- removed R1, R15, R16, R2, R21, R22, R24, R25, R26, R27, R28, R29, R3, R30, R31, R32, R33, R34, R35, R36, R37, R38, R39, R4, R40, R41, R42, R43, R5, R6, R7, R8: 4.7K, symbol Device:R
- added C41, C43: 0.1uF, Capacitor_THT:C_Disc_D5.0mm_W2.5mm_P5.00mm, symbol Device:C
- added JP3: TRNS1 INT, Connector_PinHeader_2.54mm:PinHeader_1x03_P2.54mm_Vertical, symbol Jumper:Jumper_3_Bridged12
- added JP4: RECV1 INT, Connector_PinHeader_2.54mm:PinHeader_1x03_P2.54mm_Vertical, symbol Jumper:Jumper_3_Bridged12
- added R19: 4.7K, Resistor_THT:R_Axial_DIN0207_L6.3mm_D2.5mm_P7.62mm_Horizontal, symbol Device:R
- added RN1, RN2, RN3, RN4: 4.7K, Resistor_THT:R_Array_SIP9, symbol Device:R_Network08
- added U37: 74LS08, Package_DIP:DIP-14_W7.62mm, symbol 74xx:74LS08
- C10, C11, C12, C13, C14, C15, C16, C17, C18, C19, C20, C21, C22, C23, C24, C25, C26, C27, C28, C29, C30, C31, C32, C33, C34, C35, C36, C37, C38, C39, C40, C5, C6, C7, C8, C9: footprint (none) -> Capacitor_THT:C_Disc_D5.0mm_W2.5mm_P5.00mm
- J1: footprint Connector_DIN:DIN41612_B_2x32_Female_Vertical_THT -> Connector_DIN:DIN41612_B_2x32_Male_Horizontal_THT
- J2: footprint (none) -> Connector_PinHeader_2.54mm:PinHeader_1x04_P2.54mm_Horizontal
- J3, J4: footprint (none) -> Connector_PinHeader_2.54mm:PinHeader_1x06_P2.54mm_Horizontal
- J5, J6: footprint Connector_IDC:IDC-Header_2x05_P2.54mm_Vertical -> Connector_IDC:IDC-Header_2x05_P2.54mm_Horizontal
- R1: renamed from R9; footprint (none) -> Resistor_THT:R_Axial_DIN0207_L6.3mm_D2.5mm_P7.62mm_Horizontal
- R10: renamed from R20; footprint (none) -> Resistor_THT:R_Axial_DIN0207_L6.3mm_D2.5mm_P7.62mm_Horizontal
- R11: renamed from R23; footprint (none) -> Resistor_THT:R_Axial_DIN0207_L6.3mm_D2.5mm_P7.62mm_Horizontal
- R12: renamed from R44; footprint (none) -> Resistor_THT:R_Axial_DIN0207_L6.3mm_D2.5mm_P7.62mm_Horizontal
- R13: renamed from R45; footprint (none) -> Resistor_THT:R_Axial_DIN0207_L6.3mm_D2.5mm_P7.62mm_Horizontal
- R14: renamed from R47; footprint (none) -> Resistor_THT:R_Axial_DIN0207_L6.3mm_D2.5mm_P7.62mm_Horizontal
- R15: renamed from R46; footprint (none) -> Resistor_THT:R_Axial_DIN0207_L6.3mm_D2.5mm_P7.62mm_Horizontal
- R16: renamed from R48; footprint (none) -> Resistor_THT:R_Axial_DIN0207_L6.3mm_D2.5mm_P7.62mm_Horizontal
- R17: renamed from R49; footprint (none) -> Resistor_THT:R_Axial_DIN0207_L6.3mm_D2.5mm_P7.62mm_Horizontal
- R18: renamed from R50; footprint (none) -> Resistor_THT:R_Axial_DIN0207_L6.3mm_D2.5mm_P7.62mm_Horizontal
- R2: renamed from R10; footprint (none) -> Resistor_THT:R_Axial_DIN0207_L6.3mm_D2.5mm_P7.62mm_Horizontal
- R3: renamed from R11; footprint (none) -> Resistor_THT:R_Axial_DIN0207_L6.3mm_D2.5mm_P7.62mm_Horizontal
- R4: renamed from R12; footprint (none) -> Resistor_THT:R_Axial_DIN0207_L6.3mm_D2.5mm_P7.62mm_Horizontal
- R5: renamed from R13; footprint (none) -> Resistor_THT:R_Axial_DIN0207_L6.3mm_D2.5mm_P7.62mm_Horizontal
- R6: renamed from R14; footprint (none) -> Resistor_THT:R_Axial_DIN0207_L6.3mm_D2.5mm_P7.62mm_Horizontal
- R7: renamed from R17; footprint (none) -> Resistor_THT:R_Axial_DIN0207_L6.3mm_D2.5mm_P7.62mm_Horizontal
- R8: renamed from R18; footprint (none) -> Resistor_THT:R_Axial_DIN0207_L6.3mm_D2.5mm_P7.62mm_Horizontal
- R9: renamed from R19; footprint (none) -> Resistor_THT:R_Axial_DIN0207_L6.3mm_D2.5mm_P7.62mm_Horizontal
- SW1, SW2, SW3, SW4: footprint (none) -> Button_Switch_THT:SW_DIP_SPSTx08_Slide_9.78x22.5mm_W7.62mm_P2.54mm
- SW5: value UART 1 Settings -> UART 0 Settings; footprint (none) -> Button_Switch_THT:SW_DIP_SPSTx08_Slide_9.78x22.5mm_W7.62mm_P2.54mm
- SW6: value UART 2 Settings -> UART 1 Settings; footprint (none) -> Button_Switch_THT:SW_DIP_SPSTx08_Slide_9.78x22.5mm_W7.62mm_P2.54mm
- U1, U10, U11, U12, U13, U15, U17, U2, U20, U21, U23, U25, U29, U3, U30, U31, U36, U5, U6: footprint (none) -> Package_DIP:DIP-14_W7.62mm
- U14, U18, U22, U4, U7: footprint (none) -> Package_DIP:DIP-20_W7.62mm
- U16, U19, U24, U26, U27, U28, U34, U8, U9: footprint (none) -> Package_DIP:DIP-16_W7.62mm
- U32, U33: footprint (none) -> Package_DIP:DIP-40_W15.24mm
Connections:
- net *A_SUBDEV1: now also U29.2
- net *CAF: now also U37.4, U37.9; no longer U29.1, U29.4
- net *DRQ_GRANT: now also U37.1; no longer U29.9
- net *INCREMENT_ZERO: now also U1.5; no longer U29.10
- net *INT_REQ: now also U36.10, U36.8
- net *JMP_I_DETECT: now also U29.4
- net *KEYBD_RD: now also U37.2; no longer U1.5
- net *PRINT_RES: now also U37.10, U37.5; no longer U29.2, U29.5
- net *REST_PEND: now also U29.5; no longer U23.5
- net *RTC_ENABLE: now also U7.6 (I2a)
- net *SET_RTC_EN: no longer U7.6 (I2a)
- net +5V: now also C41.1, C43.1, R19.1, RN1.1 (common), RN2.1 (common), RN3.1 (common), RN4.1 (common), U37.14 (VCC)
- net GND: now also SW5.10, SW5.11, SW5.12, SW5.13, SW5.14, SW5.15, SW5.16, SW5.9, SW6.10, SW6.11, SW6.12, SW6.13, SW6.14, SW6.15, SW6.16, SW6.9, U29.10, U29.9, C41.2, C43.2, JP3.3 (B), JP4.3 (B), U37.12, U37.13, U37.7 (GND); no longer U36.11, U36.13, U36.9
- net IORS0: now also RN1.9 (R8)
- net IORS1: now also RN1.8 (R7)
- net IORS2: now also RN1.7 (R6)
- net IORS3: now also RN1.6 (R5)
- net IORS4: now also RN1.5 (R4)
- net IORS5: now also RN1.4 (R3)
- net IORS6: now also RN1.3 (R2)
- net IORS7: now also RN1.2 (R1)
- net RECV_FLAG_0: now also U36.13; no longer U7.15 (I2b)
- net RECV_FLAG_1: now also JP4.1 (A)
- net TRNS_FLAG_0: no longer U7.13 (I1b)
- net TRNS_FLAG_1: now also JP3.1 (A)
- net at U19.9 (~{PE}): now also RN2.4 (R3)
- net at SW5.2, U27.10 (S1): now also RN3.8 (R7)
- net at U19.1 (U/~{D}): now also RN2.5 (R4)
- net at U16.1 (U/~{D}): now also RN2.3 (R2)
- net at U16.9 (~{PE}): now also RN2.2 (R1)
- net at SW5.5, U32.38 (WLS1): now also RN4.6 (R5)
- net at SW6.2, U28.10 (S1): now also RN3.5 (R4)
- net at SW6.1, U28.11 (S0): now also RN3.6 (R5)
- net at J2.2 (Pin_2), U27.12 (I7), U28.12 (I7): now also RN2.8 (R7)
- net at SW6.3, U28.9 (S2): now also RN3.4 (R3)
- net at SW5.6, U32.37 (WLS2): now also RN4.7 (R6)
- net at SW5.8, U32.35 (PI): now also RN4.9 (R8)
- net at SW5.7, U32.36 (SBS): now also RN4.8 (R7)
- net at SW5.4, U32.39 (EPE): now also RN4.5 (R4)
- net at U31.10 (~{S}): now also U1.6; no longer U29.8
- net at SW6.7, U33.36 (SBS): now also RN4.3 (R2)
- net at U11.9, U14.19 (OEb), U22.1 (OEa)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: now also U37.3; no longer U1.6
- net at U30.13 (~{R}): now also U37.6; no longer U29.6
- net at SW6.8, U33.35 (PI): now also RN4.4 (R3)
- net at U24.9 (~{PE}): now also RN2.6 (R5)
- net at SW5.3, U27.9 (S2): now also RN3.7 (R6)
- net at U36.12: now also U7.15 (I2b), R19.2
- net at U20.4: now also U23.5; no longer U23.4
- net at U24.1 (U/~{D}): now also RN2.7 (R6)
- net at SW5.1, U27.11 (S0): now also RN3.9 (R8)
- net at U30.1 (~{R}): now also U37.8; no longer U29.3
- net at SW6.4, U33.39 (EPE): now also RN3.2 (R1)
- net at SW6.5, U33.38 (WLS1): now also RN3.3 (R2)
- net at SW6.6, U33.37 (WLS2): now also RN4.2 (R1)
- net at U26.1 (U/~{D}): now also RN2.9 (R8)
- net *TRNS_FLAG_0: now reaches U30.6 (~{Q})
- net *TRNS_FLAG_0: now also U7.13 (I1b)
- net *REST_SET: no longer names the net of U13.8
- net *REST_SET: now also U29.1; no longer U17.4 (~{S})
- new net: U23.4, U29.6
- new net: JP3.2 (C), U36.9
- new net: U17.4 (~{S}), U29.3
- new net: JP4.2 (C), U36.11
- no-connect marks 76 -> 74
Other:
- moved on the sheet: C20, U1B, U23B, U29A, U29B, U29C, U36A, U36B, U36C, U36D, U36E, U36F
