File: kicad/TTY Clock/TTY Clock.kicad_pcb (KiCad board)
At the start: 2 copper layers, 234.9 x 137.5 mm, 120 parts, among them J1 I/O Connector, J2 Custom Clock, J3 TTL Serial 0, J4 TTL Serial 1, J5 RS232 Serial 0, J6 RS232 Serial 1, SW1 IORS 0 Settings, SW2 IORS 1 Settings, SW3 IORS 2 Settings, SW4 IORS 3 Settings, SW5 UART 0 Settings, SW6 UART 1 Settings, U1 74LS32, U10 74LS06, U11 74LS00, U12 74LS32, U13 74LS32, U14 74LS240, U15 74LS74, U16 74LS169, U17 74LS74, U18 74LS244, U19 74LS169, U2 74LS04, U20 74LS02, U21 74LS74, U22 74LS244, U23 74LS32, U24 74LS169, U25 74LS32, U26 74LS169, U27 74LS151, U28 74LS151, U29 74LS32, U3 74LS08, U30 74LS74, U31 74LS74, U32 TR1863, U33 TR1863, U34 74LS257, U35 MAX232, U36 74LS06, U37 74LS08, U4 74LS240, U5 74LS02, U6 74LS32, U7 74LS240, U8 74LS138, U9 74LS138, X1 2.4576 Mhz Oscillator

Commit message: Gerber creation marathon
Routing:
- net GND: track 0.00 -> 1640.0 mm
- net +5V: track 0.00 -> 1271.0 mm
- net /*CAF: track 0.00 -> 369.8 mm, vias 0 -> 1
- net /*DRQ_GRANT: track 0.00 -> 327.9 mm, vias 0 -> 1
- net Net-(U14-OEb): track 0.00 -> 318.0 mm, vias 0 -> 3
- net /A_SUBDEV1: track 0.00 -> 296.9 mm, vias 0 -> 2
- net /CAF: track 0.00 -> 286.8 mm, vias 0 -> 1
- net /D7: track 0.00 -> 277.1 mm, vias 0 -> 1
- net /D6: track 0.00 -> 275.8 mm, vias 0 -> 1
- net /D0: track 0.00 -> 269.5 mm, vias 0 -> 2
- net /*A_PULSE2: track 0.00 -> 268.9 mm, vias 0 -> 1
- net /D1: track 0.00 -> 264.0 mm, vias 0 -> 2
- net /D5: track 0.00 -> 262.6 mm
- net /D2: track 0.00 -> 257.4 mm, vias 0 -> 1
- net /D4: track 0.00 -> 255.5 mm
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- added copper zone on B.Cu, net GND
- added copper zone on F.Cu, net GND
Other:
- board text removed: "JLCJLCJLCJLC"
