File: kicad/Memory/Memory.kicad_sch (KiCad schematic)
At the start: 12 parts, among them J1 Control Connector, J2 Data Connector, U1 CY62256-70PC, U10 74LS257, U2 CY62256-70PC, U3 CY62256-70PC, U4 74LS245, U5 74LS245, U6 74LS245, U7 74LS257, U8 74LS257, U9 74LS257

Commit message: Continue work on memory board
Connections:
- net A0: now also U7.4 (Za)
- net A1: now also U7.7 (Zb)
- net A10: now also U9.12 (Zc)
- net A11: now also U9.9 (Zd)
- net A12: now also U10.4 (Za)
- net A13: now also U10.7 (Zb)
- net A14: now also U10.12 (Zc)
- net A2: now also U7.12 (Zc)
- net A3: now also U7.9 (Zd)
- net A4: now also U8.4 (Za)
- net A5: now also U8.7 (Zb)
- net A6: now also U8.12 (Zc)
- net A7: now also U8.9 (Zd)
- net A8: now also U9.4 (Za)
- net A9: now also U9.7 (Zb)
- net D0: now also U4.2 (A0)
- net D1: now also U4.3 (A1)
- net D10: now also U5.4 (A2)
- net D11: now also U5.5 (A3)
- net D12: now also U5.6 (A4)
- net D13: now also U5.7 (A5)
- net D14: now also U5.8 (A6)
- net D15: now also U5.9 (A7)
- net D16: now also U6.2 (A0)
- net D17: now also U6.3 (A1)
- net D2: now also U4.4 (A2)
- net D3: now also U4.5 (A3)
- net D4: now also U4.6 (A4)
- net D5: now also U4.7 (A5)
- net D6: now also U4.8 (A6)
- net D7: now also U4.9 (A7)
- net D8: now also U5.2 (A0)
- net D9: now also U5.3 (A1)
- net GND: now also U10.15 (OE), U6.4 (A2), U6.5 (A3), U6.6 (A4), U6.7 (A5), U6.8 (A6), U6.9 (A7), U7.15 (OE), U8.15 (OE), U9.15 (OE)
- net M17: now reaches U6.17 (B1)
- net M16: now reaches U6.18 (B0)
- net M15: now reaches U5.11 (B7)
- net M14: now reaches U5.12 (B6)
- net M13: now reaches U5.13 (B5)
- net M12: now reaches U5.14 (B4)
- net M11: now reaches U5.15 (B3)
- net M10: now reaches U5.16 (B2)
- net M9: now reaches U5.17 (B1)
- net M8: now reaches U5.18 (B0)
- net M7: now reaches U4.11 (B7)
- net M6: now reaches U4.12 (B6)
- net M5: now reaches U4.13 (B5)
- net M4: now reaches U4.14 (B4)
- net M3: now reaches U4.15 (B3)
- net M2: now reaches U4.16 (B2)
- net M1: now reaches U4.17 (B1)
- net M0: now reaches U4.18 (B0)
- no-connect marks 86 -> 93

Commit message: Continue work on memory board
Parts:
- added R2 (x18): 4.7K, symbol Device:R
- added U11, U12, U13, U14: 74LS377, symbol 74xx:74LS377
- added U15: 74LS32, symbol 74xx:74LS32
- added U16: 74LS257, symbol 74xx:74LS257
- added U17: 74LS08, symbol 74xx:74LS08
- added U18: 74LS00, symbol 74xx:74LS00
Connections:
- net *MEMM_ENABLE: now also U18.10, U18.9
- net *SELECT_CORE: now also U1.22 (~{OE}), U2.22 (~{OE}), U3.22 (~{OE}), U4.1 (A->B), U5.1 (A->B), U6.1 (A->B)
- net *WRITE_CORE: now also U15.1
- net +5V: now also R2.2, R2.2, R2.2, R2.2, R2.2, R2.2, R2.2, R2.2, R2.2, R2.2, R2.2, R2.2, R2.2, R2.2, R2.2, R2.2, R2.2, R2.2, U11.20 (VCC), U12.20 (VCC), U13.20 (VCC), U14.20 (VCC), U16.16 (VCC)
- net A0: now also U1.10 (A0), U2.10 (A0), U3.10 (A0)
- net A1: now also U1.9 (A1), U2.9 (A1), U3.9 (A1)
- net A10: now also U1.21 (A10), U2.21 (A10), U3.21 (A10)
- net A11: now also U1.23 (A11), U2.23 (A11), U3.23 (A11)
- net A12: now also U1.2 (A12), U2.2 (A12), U3.2 (A12)
- net A13: now also U1.26 (A13), U2.26 (A13), U3.26 (A13), U17.3; no longer U10.7 (Zb)
- net A14: now also U1.1 (A14), U2.1 (A14), U3.1 (A14), U17.6; no longer U10.12 (Zc)
- net A2: now also U1.8 (A2), U2.8 (A2), U3.8 (A2)
- net A3: now also U1.7 (A3), U2.7 (A3), U3.7 (A3)
- net A4: now also U1.6 (A4), U2.6 (A4), U3.6 (A4)
- net A5: now also U1.5 (A5), U2.5 (A5), U3.5 (A5)
- net A6: now also U1.4 (A6), U2.4 (A6), U3.4 (A6)
- net A7: now also U1.3 (A7), U2.3 (A7), U3.3 (A7)
- net A8: now also U1.25 (A8), U2.25 (A8), U3.25 (A8)
- net A9: now also U1.24 (A9), U2.24 (A9), U3.24 (A9)
- net ADDR_MODE0: now also U17.12, U18.1
- net ADDR_MODE1: now also U17.9, U18.2, U18.4, U18.5
- net CLK: now also U11.11 (CP), U12.11 (CP), U13.11 (CP), U14.11 (CP), U15.2
- net GND: now also U1.20 (~{CS}), U10.10 (I1d), U10.11 (I0d), U2.20 (~{CS}), U3.20 (~{CS}), U11.10 (GND), U12.10 (GND), U12.18 (D7), U13.10 (GND), U14.10 (GND), U14.18 (D7), U16.15 (OE), U16.8 (GND); no longer U6.4 (A2), U6.5 (A3), U6.6 (A4), U6.7 (A5), U6.8 (A6), U6.9 (A7)
- net M0: now also U1.11 (Q0), U11.3 (D0), U13.3 (D0)
- net M1: now also U1.12 (Q1), U11.4 (D1), U13.4 (D1)
- net M10: now also U2.13 (Q2), U12.7 (D2), U14.7 (D2)
- net M11: now also U2.15 (Q3), U12.8 (D3), U14.8 (D3)
- net M12: now also U2.16 (Q4), U12.13 (D4), U14.13 (D4)
- net M13: now also U2.17 (Q5), U16.3 (I1a)
- net M14: now also U2.18 (Q6), U16.6 (I1b)
- net M15: now also U2.19 (Q7)
- net M16: now also U3.11 (Q0)
- net M17: now also U3.12 (Q1)
- net M2: now also U1.13 (Q2), U11.7 (D2), U13.7 (D2)
- net M3: now also U1.15 (Q3), U11.8 (D3), U13.8 (D3)
- net M4: now also U1.16 (Q4), U11.13 (D4), U13.13 (D4)
- net M5: now also U1.17 (Q5), U11.14 (D5), U13.14 (D5)
- net M6: now also U1.18 (Q6), U11.17 (D6), U13.17 (D6)
- net M7: now also U1.19 (Q7), U11.18 (D7), U13.18 (D7)
- net M8: now also U2.11 (Q0), U12.3 (D0), U14.3 (D0)
- net M9: now also U2.12 (Q1), U12.4 (D1), U14.4 (D1)
- net MA11: now reaches U9.10 (I1d)
- net MA11: now also U14.9 (Q3)
- net PC11: now reaches U9.11 (I0d)
- net PC11: now also U12.9 (Q3)
- net MA10: now reaches U9.13 (I1c)
- net MA10: now also U14.6 (Q2)
- net PC10: now reaches U9.14 (I0c)
- net PC10: now also U12.6 (Q2)
- net PC8: now reaches U9.2 (I0a)
- net PC8: now also U12.2 (Q0)
- net MA8: now reaches U9.3 (I1a)
- net MA8: now also U14.2 (Q0)
- net PC9: now reaches U9.5 (I0b)
- net PC9: now also U12.5 (Q1)
- net MA9: now reaches U9.6 (I1b)
- net MA9: now also U14.5 (Q1)
- net MA14: now reaches U10.13 (I1c)
- net MA14: now also U14.16 (Q6)
- net PC14: now reaches U10.14 (I0c)
- net PC14: now also U12.16 (Q6), U16.5 (I0b)
- net PC12: now reaches U10.2 (I0a)
- net PC12: now also U12.12 (Q4)
- net MA12: now reaches U10.3 (I1a)
- net MA12: now also U14.12 (Q4)
- net PC13: now reaches U10.5 (I0b)
- net PC13: now also U12.15 (Q5), U16.2 (I0a)
- net MA13: now reaches U10.6 (I1b)
- net MA13: now also U14.15 (Q5)
- net at U1.27 (~{WE}): now also U2.27 (~{WE}), U3.27 (~{WE}), U15.3
- net T11: now reaches U6.11 (B7)
- net T11: now also R2.1
- net T10: now reaches U6.12 (B6)
- net T10: now also R2.1
- net T9: now reaches U6.13 (B5)
- net T9: now also R2.1
- net T8: now reaches U6.14 (B4)
- net T8: now also R2.1
- net T7: now reaches U6.15 (B3)
- net T7: now also R2.1
- net T6: now reaches U6.16 (B2)
- net T6: now also R2.1
- net MA7: now reaches U8.10 (I1d)
- net MA7: now also U13.19 (Q7)
- net PC7: now reaches U8.11 (I0d)
- net PC7: now also U11.19 (Q7)
- net MA6: now reaches U8.13 (I1c)
- net MA6: now also U13.16 (Q6)
- net PC6: now reaches U8.14 (I0c)
- net PC6: now also U11.16 (Q6)
- net PC4: now reaches U8.2 (I0a)
- net PC4: now also U11.12 (Q4)
- net MA4: now reaches U8.3 (I1a)
- net MA4: now also U13.12 (Q4)
- net PC5: now reaches U8.5 (I0b)
- net PC5: now also U11.15 (Q5)
- net MA5: now reaches U8.6 (I1b)
- net MA5: now also U13.15 (Q5)
- net MA3: now reaches U7.10 (I1d)
- net MA3: now also U13.9 (Q3)
- net PC3: now reaches U7.11 (I0d)
- net PC3: now also U11.9 (Q3)
- net MA2: now reaches U7.13 (I1c)
- net MA2: now also U13.6 (Q2)
- net PC2: now reaches U7.14 (I0c)
- net PC2: now also U11.6 (Q2)
- net PC0: now reaches U7.2 (I0a)
- net PC0: now also U11.2 (Q0)
- net MA0: now reaches U7.3 (I1a)
- net MA0: now also U13.2 (Q0)
- net PC1: now reaches U7.5 (I0b)
- net PC1: now also U11.5 (Q1)
- net MA1: now reaches U7.6 (I1b)
- net MA1: now also U13.5 (Q1)
- net T12: now reaches U3.13 (Q2)
- net T12: now also R2.1
- net T13: now reaches U3.15 (Q3)
- net T13: now also R2.1
- net T14: now reaches U3.16 (Q4)
- net T14: now also R2.1
- net T15: now reaches U3.17 (Q5)
- net T15: now also R2.1
- net T16: now reaches U3.18 (Q6)
- net T16: now also R2.1
- net T17: now reaches U3.19 (Q7)
- net T17: now also R2.1
- net EXTRA7 renamed NEXT_BANK0
- net NEXT_BANK0: now also U12.14 (D5), U14.14 (D5), U16.4 (Za)
- net EXTRA8 renamed NEXT_BANK1
- net NEXT_BANK1: now also U12.17 (D6), U14.17 (D6), U16.7 (Zb)
- net REST_PEND renamed *REST_PEND
- new net: U15.4, U17.11
- new net: U17.13, U18.6
- new net: U10.12 (Zc), U17.4
- new net: U10.7 (Zb), U17.1
- new net: U17.2, U17.5, U18.3
- new net: U17.10, U18.8
- new net: U15.5, U17.8
- new net EXTEND: U15.6, U16.1 (S)
- new net T0: R2.1, U6.4 (A2)
- new net T1: R2.1, U6.5 (A3)
- new net T2: R2.1, U6.6 (A4)
- new net T3: R2.1, U6.7 (A5)
- new net T4: R2.1, U6.8 (A6)
- new net T5: R2.1, U6.9 (A7)
- no-connect marks 93 -> 88

Commit message: Continue work on memory board
Parts:
- added C1 (x4), C2 (x4), C3 (x4), C4 (x4), C5 (x4): 0.1uF, symbol Device:C
- added C20: 100 uF, Capacitor_THT:CP_Radial_D6.3mm_P2.50mm, symbol Device:C_Polarized
- added U19: 74LS27, symbol 74xx:74LS27
- added U20: 74LS08, symbol 74xx:74LS08
Connections:
- net *LATCH_MA: now also U13.1 (~{E}), U14.1 (~{E})
- net *LATCH_PC: now also U11.1 (~{E}), U12.1 (~{E})
- net +5V: now also U15.14 (VCC), U17.14 (VCC), U18.14 (VCC), C1.1, C1.1, C1.1, C1.1, C2.1, C2.1, C2.1, C2.1, C20.1, C3.1, C3.1, C3.1, C3.1, C4.1, C4.1, C4.1, C4.1, C5.1, C5.1, C5.1, C5.1, U19.14 (VCC), U20.14 (VCC)
- net GND: now also U15.12, U15.13, U15.7 (GND), U16.10 (I1d), U16.11 (I0d), U16.13 (I1c), U16.14 (I0c), U17.7 (GND), U18.7 (GND), C1.2, C1.2, C1.2, C1.2, C2.2, C2.2, C2.2, C2.2, C20.2, C3.2, C3.2, C3.2, C3.2, C4.2, C4.2, C4.2, C4.2, C5.2, C5.2, C5.2, C5.2, U19.7 (GND), U20.10, U20.12, U20.13, U20.7 (GND), U20.9
- net MA10: now also U19.9
- net MA11: now also U19.10
- net MA12: now also U19.11
- net MA3: now also U18.12, U18.13
- net MA4: now also U15.10
- net MA5: now also U19.2
- net MA6: now also U19.13
- net MA7: now also U19.3
- net MA8: now also U19.4
- net MA9: now also U19.5
- net MA_AUTO_INX: now also U20.6
- net SELECT_PCMA: now also U10.1 (S), U7.1 (S), U8.1 (S), U9.1 (S)
- net at U15.8: now also U19.1
- net at U15.9: now also U18.11
- new net: U19.12, U20.1
- new net: U19.6, U20.2
- new net: U19.8, U20.5
- new net: U20.3, U20.4
- no-connect marks 88 -> 83
Other:
- moved on the sheet: U15C, U15D, U15E, U17E, U18D, U18E

Commit message: Finish pinout audit + fanout correction
Other:
- note added: "MA"
- note added: "PC"
- note added: "Register"

Commit message: Start work on backplane and fix connectors
Parts:
- removed J1: Control Connector, symbol Connector:DIN41612_02x32_AC
- removed J2: Data Connector, symbol Connector:DIN41612_02x32_AC
- added J1: Control Connector, Connector_DIN:DIN41612_B_2x32_Male_Horizontal_THT, symbol Connector:DIN41612_02x32_AB
- added J2: Data Connector, Connector_DIN:DIN41612_B_2x32_Male_Horizontal_THT, symbol Connector:DIN41612_02x32_AB
Connections:
- net *CAF: now also J2.a22 (Pin_a22)
- net *CHAN_REQ: now also J1.a7 (Pin_a7)
- net *DEV_REQ: now also J1.a8 (Pin_a8)
- net *DMA_REQ: now also J1.a6 (Pin_a6)
- net *INT_REQ: now also J1.a9 (Pin_a9)
- net *IOT_SKIP: now also J1.a10 (Pin_a10)
- net *IOT_SKIP_L: now also J1.a12 (Pin_a12)
- net *IOT_WAIT: now also J1.a11 (Pin_a11)
- net *LATCH_AC: now also J1.a16 (Pin_a16)
- net *LATCH_IR: now also J1.a13 (Pin_a13)
- net *LATCH_MA: now also J1.a14 (Pin_a14)
- net *LATCH_MB: now also J1.a19 (Pin_a19)
- net *LATCH_MQ: now also J1.a18 (Pin_a18)
- net *LATCH_OB: now also J1.a21 (Pin_a21)
- net *LATCH_PC: now also J1.a15 (Pin_a15)
- net *LATCH_STEP: now also J1.a17 (Pin_a17)
- net *LATCH_WRTBK: now also J1.a20 (Pin_a20)
- net *MEMM_ENABLE: now also J1.a4 (Pin_a4)
- net *PI_ENABLE: now also J1.a3 (Pin_a3)
- net *PROT_ENABLE: now also J1.a5 (Pin_a5)
- net *RESET: now also J2.a21 (Pin_a21)
- net *REST_PEND: now also J2.a28 (Pin_a28)
- net *SELECT_AC: now also J1.b12 (Pin_b12)
- net *SELECT_ALU: now also J1.b16 (Pin_b16)
- net *SELECT_CORE: now also J1.b17 (Pin_b17)
- net *SELECT_CROSS: now also J1.b15 (Pin_b15)
- net *SELECT_EXTRN: now also J1.b19 (Pin_b19)
- net *SELECT_MQ: now also J1.b14 (Pin_b14)
- net *SELECT_STEP: now also J1.b13 (Pin_b13)
- net *SELECT_SWR: now also J1.b18 (Pin_b18)
- net *WRITE_CORE: now also J1.a22 (Pin_a22)
- net +5V: now also J1.a32 (Pin_a32), J1.b1 (Pin_b1), J2.a32 (Pin_a32), J2.b1 (Pin_b1)
- net A0: now also J2.b3 (Pin_b3)
- net A1: now also J2.b4 (Pin_b4)
- net A10: now also J2.b13 (Pin_b13)
- net A11: now also J2.b14 (Pin_b14)
- net A12: now also J2.b15 (Pin_b15)
- net A13: now also J2.b16 (Pin_b16)
- net A14: now also J2.b17 (Pin_b17)
- net A2: now also J2.b5 (Pin_b5)
- net A3: now also J2.b6 (Pin_b6)
- net A4: now also J2.b7 (Pin_b7)
- net A5: now also J2.b8 (Pin_b8)
- net A6: now also J2.b9 (Pin_b9)
- net A7: now also J2.b10 (Pin_b10)
- net A8: now also J2.b11 (Pin_b11)
- net A9: now also J2.b12 (Pin_b12)
- net ADDR_MODE0: now also J1.b27 (Pin_b27)
- net ADDR_MODE1: now also J1.b28 (Pin_b28)
- net ALUO0: now also J1.a24 (Pin_a24)
- net ALUO1: now also J1.a25 (Pin_a25)
- net ALUO2: now also J1.a26 (Pin_a26)
- net ALU_ONES: now also J1.a30 (Pin_a30)
- net ALU_SHIFT: now also J1.a29 (Pin_a29)
- net BUS_SELECT0: now also J1.b9 (Pin_b9)
- net BUS_SELECT1: now also J1.b10 (Pin_b10)
- net BUS_SELECT2: now also J1.b11 (Pin_b11)
- net CLK: now also J2.a23 (Pin_a23)
- net CTL_CONST: now also J1.b29 (Pin_b29)
- net D0: now also J2.a3 (Pin_a3)
- net D1: now also J2.a4 (Pin_a4)
- net D10: now also J2.a13 (Pin_a13)
- net D11: now also J2.a14 (Pin_a14)
- net D12: now also J2.a15 (Pin_a15)
- net D13: now also J2.a16 (Pin_a16)
- net D14: now also J2.a17 (Pin_a17)
- net D15: now also J2.a18 (Pin_a18)
- net D16: now also J2.a19 (Pin_a19)
- net D17: now also J2.a20 (Pin_a20)
- net D2: now also J2.a5 (Pin_a5)
- net D3: now also J2.a6 (Pin_a6)
- net D4: now also J2.a7 (Pin_a7)
- net D5: now also J2.a8 (Pin_a8)
- net D6: now also J2.a9 (Pin_a9)
- net D7: now also J2.a10 (Pin_a10)
- net D8: now also J2.a11 (Pin_a11)
- net D9: now also J2.a12 (Pin_a12)
- net DRQ_GRANT: now also J1.b21 (Pin_b21)
- net EXTRA0: now also J1.b30 (Pin_b30)
- net EXTRA1: now also J2.a24 (Pin_a24)
- net EXTRA2: now also J2.b24 (Pin_b24)
- net EXTRA3: now also J2.a25 (Pin_a25)
- net EXTRA4: now also J2.b25 (Pin_b25)
- net EXTRA5: now also J2.a26 (Pin_a26)
- net EXTRA6: now also J2.b26 (Pin_b26)
- net FLAG_AC_SIGN: now also J1.b8 (Pin_b8)
- net FLAG_LINK: now also J1.b6 (Pin_b6)
- net FLAG_LINK_INIT: now also J1.b7 (Pin_b7)
- net FLAG_SIGN: now also J1.b5 (Pin_b5)
- net FLAG_ZERO: now also J1.b4 (Pin_b4)
- net FP0: now also J2.a29 (Pin_a29)
- net FP1: now also J2.b29 (Pin_b29)
- net FP2: now also J2.a30 (Pin_a30)
- net FP3: now also J2.b30 (Pin_b30)
- net GND: now also J1.a1 (Pin_a1), J1.b32 (Pin_b32), J2.a1 (Pin_a1), J2.b32 (Pin_b32)
- net HALT: now also J1.b26 (Pin_b26)
- net INT_DETECT: now also J1.b24 (Pin_b24)
- net IOT_PULSE: now also J1.b20 (Pin_b20)
- net JMP_I_DETECT: now also J1.b23 (Pin_b23)
- net LINKS0: now also J1.a27 (Pin_a27)
- net LINKS1: now also J1.a28 (Pin_a28)
- net MA_AUTO_INX: now also J2.b28 (Pin_b28)
- net NEXT_BANK0: now also J2.a27 (Pin_a27)
- net NEXT_BANK1: now also J2.b27 (Pin_b27)
- net READ_IN_PULSE: now also J1.b25 (Pin_b25)
- net REQ_ADDR: now also J1.b22 (Pin_b22)
- net SC0: now also J2.b18 (Pin_b18)
- net SC1: now also J2.b19 (Pin_b19)
- net SC2: now also J2.b20 (Pin_b20)
- net SC3: now also J2.b21 (Pin_b21)
- net SC4: now also J2.b22 (Pin_b22)
- net SC5: now also J2.b23 (Pin_b23)
- net SELECT_PCMA: now also J1.a23 (Pin_a23)
- net STEP_ZERO: now also J1.b3 (Pin_b3)
Changed lines of the file:
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@@
     )
   )
-  (symbol (lib_id "Connector:DIN41612_02x32_AC") (at 518.795 208.28 0) (unit 1)
-    (in_bom yes) (on_board yes) (dnp no)
-    (property "Reference" "J2" (at 520.065 167.64 0)
-      (effects (font (size 1.27 1.27)))
-    )
-    (property "Value" "Data Connector" (at 518.795 163.83 0)
-      (effects (font (size 1.27 1.27)))
-    )
-    (property "Footprint" "" (at 518.795 208.28 0)
-      (effects (font (size 1.27 1.27)) hide)
-    )
-    (property "Datasheet" "~" (at 518.795 208.28 0)
-      (effects (font (size 1.27 1.27)) hide)
-    )
-    (pin "a1")
-    (pin "a10")
-    (pin "a11")
-    (pin "a12")
-    (pin "a13")
-    (pin "a14")
-    (pin "a15")
-    (pin "a16")
-    (pin "a17")
-    (pin "a18")
-    (pin "a19")
-    (pin "a2")
-    (pin "a20")
-    (pin "a21")
-    (pin "a22")
-    (pin "a23")
-    (pin "a24")
-    (pin "a25")
-    (pin "a26")
-    (pin "a27")
-    (pin "a28")
-    (pin "a29")
-    (pin "a3")
-    (pin "a30")
-    (pin "a31")
-    (pin "a32")
-    (pin "a4")
-    (pin "a5")
-    (pin "a6")
-    (pin "a7")
-    (pin "a8")
-    (pin "a9")
-    (pin "c1")
-    (pin "c10")
-    (pin "c11")
-    (pin "c12")
-    (pin "c13")
-    (pin "c14")
-    (pin "c15")
-    (pin "c16")
-    (pin "c17")
-    (pin "c18")
-    (pin "c19")
-    (pin "c2")
-    (pin "c20")
-    (pin "c21")
-    (pin "c22")
-    (pin "c23")
-    (pin "c24")
-    (pin "c25")
-    (pin "c26")
-    (pin "c27")
-    (pin "c28")
-    (pin "c29")
-    (pin "c3")
-    (pin "c30")
-    (pin "c31")
-    (pin "c32")
-    (pin "c4")
-    (pin "c5")
-    (pin "c6")
-    (pin "c7")
-    (pin "c8")
-    (pin "c9")
-    (instances
-      (project "Registers"
-        (path "/8ed23248-dfae-4df3-a148-5197e001af70"
-          (reference "J2") (unit 1)
-        )
-      )
-      (project "ALU"
-        (path "/b26dce39-0c19-4808-8ddd-74847f21ad13"
-          (reference "J2") (unit 1)
-        )
-      )
-      (project "Memory"
-        (path "/b9764240-fb05-4333-bc5f-d2675d8c17cf"
-          (reference "J2") (unit 1)
-        )
-      )
-    )
-  )
   (symbol (lib_id "Device:R") (at 435.61 95.25 90) (unit 1)
     (in_bom yes) (on_board yes) (dnp no)
@@
     )
   )
+  (symbol (lib_id "Connector:DIN41612_02x32_AB") (at 518.795 93.98 0) (unit 1)
+    (in_bom yes) (on_board yes) (dnp no)
+    (property "Reference" "J1" (at 520.065 53.34 0)
+      (effects (font (size 1.27 1.27)))
+    )
+    (property "Value" "Control Connector" (at 520.065 48.895 0)
+      (effects (font (size 1.27 1.27)))
+    )
+    (property "Footprint" "Connector_DIN:DIN41612_B_2x32_Male_Horizontal_THT" (at 518.795 93.98 0)
+      (effects (font (size 1.27 1.27)) hide)
+    )
+    (property "Datasheet" "~" (at 518.795 93.98 0)
+      (effects (font (size 1.27 1.27)) hide)
+    )
+    (pin "a1")
+    (pin "a10")
+    (pin "a11")
+    (pin "a12")
+    (pin "a13")
+    (pin "a14")
+    (pin "a15")
+    (pin "a16")
+    (pin "a17")
+    (pin "a18")
+    (pin "a19")
+    (pin "a2")
+    (pin "a20")
+    (pin "a21")
+    (pin "a22")
+    (pin "a23")
+    (pin "a24")
+    (pin "a25")
+    (pin "a26")
+    (pin "a27")
+    (pin "a28")
+    (pin "a29")
+    (pin "a3")
+    (pin "a30")
+    (pin "a31")
+    (pin "a32")
+    (pin "a4")
+    (pin "a5")
+    (pin "a6")
+    (pin "a7")
+    (pin "a8")
+    (pin "a9")
+    (pin "b1")
+    (pin "b10")
+    (pin "b11")
+    (pin "b12")
+    (pin "b13")
+    (pin "b14")
+    (pin "b15")
+    (pin "b16")
+    (pin "b17")
+    (pin "b18")
+    (pin "b19")
+    (pin "b2")
+    (pin "b20")
+    (pin "b21")
+    (pin "b22")
+    (pin "b23")
+    (pin "b24")
+    (pin "b25")
+    (pin "b26")
+    (pin "b27")
+    (pin "b28")
+    (pin "b29")
+    (pin "b3")
+    (pin "b30")
+    (pin "b31")
+    (pin "b32")
+    (pin "b4")
+    (pin "b5")
+    (pin "b6")
+    (pin "b7")
+    (pin "b8")
+    (pin "b9")
+    (instances
+      (project "ALU"
+        (path "/b26dce39-0c19-4808-8ddd-74847f21ad13"
+          (reference "J1") (unit 1)
+        )
+      )
+      (project "Memory"
+        (path "/b9764240-fb05-4333-bc5f-d2675d8c17cf"
+          (reference "J2") (unit 1)
+        )
+      )
+    )
+  )
   (symbol (lib_id "power:+5V") (at 73.025 242.57 0) (unit 1)
     (in_bom yes) (on_board yes) (dnp no) (fields_autoplaced)
@@
     )
   )
-  (symbol (lib_id "Connector:DIN41612_02x32_AC") (at 518.795 93.98 0) (unit 1)
-    (in_bom yes) (on_board yes) (dnp no)
-    (property "Reference" "J1" (at 520.065 53.34 0)
-      (effects (font (size 1.27 1.27)))
-    )
-    (property "Value" "Control Connector" (at 499.11 54.61 0)
-      (effects (font (size 1.27 1.27)))
-    )
-    (property "Footprint" "" (at 518.795 93.98 0)
-      (effects (font (size 1.27 1.27)) hide)
-    )
-    (property "Datasheet" "~" (at 518.795 93.98 0)
-      (effects (font (size 1.27 1.27)) hide)
-    )
-    (pin "a1")
-    (pin "a10")
-    (pin "a11")
-    (pin "a12")
-    (pin "a13")
-    (pin "a14")
-    (pin "a15")
-    (pin "a16")
-    (pin "a17")
-    (pin "a18")
-    (pin "a19")
-    (pin "a2")
-    (pin "a20")
-    (pin "a21")
-    (pin "a22")
-    (pin "a23")
-    (pin "a24")
-    (pin "a25")
-    (pin "a26")
-    (pin "a27")
-    (pin "a28")
-    (pin "a29")
-    (pin "a3")
-    (pin "a30")
-    (pin "a31")
-    (pin "a32")
-    (pin "a4")
-    (pin "a5")
-    (pin "a6")
-    (pin "a7")
-    (pin "a8")
-    (pin "a9")
-    (pin "c1")
-    (pin "c10")
-    (pin "c11")
-    (pin "c12")
-    (pin "c13")
-    (pin "c14")
-    (pin "c15")
-    (pin "c16")
-    (pin "c17")
-    (pin "c18")
-    (pin "c19")
-    (pin "c2")
-    (pin "c20")
-    (pin "c21")
-    (pin "c22")
-    (pin "c23")
-    (pin "c24")
-    (pin "c25")
-    (pin "c26")
-    (pin "c27")
-    (pin "c28")
-    (pin "c29")
-    (pin "c3")
-    (pin "c30")
-    (pin "c31")
-    (pin "c32")
-    (pin "c4")
-    (pin "c5")
-    (pin "c6")
-    (pin "c7")
-    (pin "c8")
-    (pin "c9")
-    (instances
-      (project "Registers"
-        (path "/8ed23248-dfae-4df3-a148-5197e001af70"
-          (reference "J1") (unit 1)
-        )
-      )
-      (project "ALU"
-        (path "/b26dce39-0c19-4808-8ddd-74847f21ad13"
-          (reference "J1") (unit 1)
-        )
-      )
-      (project "Memory"
-        (path "/b9764240-fb05-4333-bc5f-d2675d8c17cf"
-          (reference "J1") (unit 1)
-        )
-      )
-    )
-  )
   (symbol (lib_id "power:+5V") (at 225.425 242.57 0) (unit 1)
     (in_bom yes) (on_board yes) (dnp no) (fields_autoplaced)
@@
         )
       )
+    )
+  )
+  (symbol (lib_id "Connector:DIN41612_02x32_AB") (at 518.795 208.28 0) (unit 1)
+    (in_bom yes) (on_board yes) (dnp no)
+    (property "Reference" "J2" (at 520.065 167.64 0)
+      (effects (font (size 1.27 1.27)))
+    )
+    (property "Value" "Data Connector" (at 519.43 163.83 0)
+      (effects (font (size 1.27 1.27)))
+    )
+    (property "Footprint" "Connector_DIN:DIN41612_B_2x32_Male_Horizontal_THT" (at 518.795 208.28 0)
+      (effects (font (size 1.27 1.27)) hide)
+    )
+    (property "Datasheet" "~" (at 518.795 208.28 0)
+      (effects (font (size 1.27 1.27)) hide)
+    )
+    (pin "a1")
+    (pin "a10")
+    (pin "a11")
+    (pin "a12")
+    (pin "a13")
+    (pin "a14")
+    (pin "a15")
+    (pin "a16")
+    (pin "a17")
+    (pin "a18")
+    (pin "a19")
+    (pin "a2")
+    (pin "a20")
+    (pin "a21")
+    (pin "a22")
+    (pin "a23")
+    (pin "a24")
+    (pin "a25")
+    (pin "a26")
+    (pin "a27")
+    (pin "a28")
+    (pin "a29")
+    (pin "a3")
+    (pin "a30")
+    (pin "a31")
+    (pin "a32")
+    (pin "a4")
+    (pin "a5")
+    (pin "a6")
+    (pin "a7")
+    (pin "a8")
+    (pin "a9")
+    (pin "b1")
+    (pin "b10")
+    (pin "b11")
+    (pin "b12")
+    (pin "b13")
+    (pin "b14")
+    (pin "b15")
+    (pin "b16")
+    (pin "b17")
+    (pin "b18")
+    (pin "b19")
+    (pin "b2")
+    (pin "b20")
+    (pin "b21")
+    (pin "b22")
+    (pin "b23")
+    (pin "b24")
+    (pin "b25")
+    (pin "b26")
+    (pin "b27")
+    (pin "b28")
+    (pin "b29")
+    (pin "b3")
+    (pin "b30")
+    (pin "b31")
+    (pin "b32")
+    (pin "b4")
+    (pin "b5")
+    (pin "b6")
+    (pin "b7")
+    (pin "b8")
+    (pin "b9")
+    (instances
+      (project "ALU"
+        (path "/b26dce39-0c19-4808-8ddd-74847f21ad13"
+          (reference "J2") (unit 1)
+        )
+      )
+      (project "Memory"
+        (path "/b9764240-fb05-4333-bc5f-d2675d8c17cf"
+          (reference "J1") (unit 1)
+        )
+      )
