File: kicad/Memory/Memory.kicad_sch (KiCad schematic)
At the start: 61 parts, among them J1 Control Connector, J2 Data Connector, U1 CY62256-70PC, U10 74LS257, U11 74LS377, U12 74LS377, U13 74LS377, U14 74LS377, U15 74LS32, U16 74LS257, U17 74LS08, U18 74LS00, U19 74LS27, U2 CY62256-70PC, U20 74LS08, U3 CY62256-70PC, U4 74LS245, U5 74LS245, U6 74LS245, U7 74LS257, U8 74LS257, U9 74LS257

Commit message: Update backplane pin logic levels
Connections:
- net DRQ_GRANT renamed *DRQ_GRANT
- net INT_DETECT renamed *INT_DETECT
- net IOT_PULSE renamed *IOT_PULSE
- net JMP_I_DETECT renamed *JMP_I_DETECT
- net READ_IN_PULSE renamed *READ_IN_PULSE
Changed lines of the file:
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@@
     (effects (font (size 1.27 1.27)) (justify right bottom))
   )
-  (label "READ_IN_PULSE" (at 526.415 116.84 0) (fields_autoplaced)
+  (label "*READ_IN_PULSE" (at 526.415 116.84 0) (fields_autoplaced)
     (effects (font (size 1.27 1.27)) (justify left bottom))
   )
@@
     (effects (font (size 1.27 1.27)) (justify right bottom))
   )
-  (label "IOT_PULSE" (at 526.415 104.14 0) (fields_autoplaced)
+  (label "*IOT_PULSE" (at 526.415 104.14 0) (fields_autoplaced)
     (effects (font (size 1.27 1.27)) (justify left bottom))
   )
@@
     (effects (font (size 1.27 1.27)) (justify right bottom))
   )
-  (label "INT_DETECT" (at 526.415 114.3 0) (fields_autoplaced)
+  (label "*INT_DETECT" (at 526.415 114.3 0) (fields_autoplaced)
     (effects (font (size 1.27 1.27)) (justify left bottom))
   )
@@
     (effects (font (size 1.27 1.27)) (justify right bottom))
   )
-  (label "JMP_I_DETECT" (at 526.415 111.76 0) (fields_autoplaced)
+  (label "*JMP_I_DETECT" (at 526.415 111.76 0) (fields_autoplaced)
     (effects (font (size 1.27 1.27)) (justify left bottom))
   )
@@
     (effects (font (size 1.27 1.27)) (justify right bottom))
   )
-  (label "DRQ_GRANT" (at 526.415 106.68 0) (fields_autoplaced)
-    (effects (font (size 1.27 1.27)) (justify left bottom))
-  )
+  (label "*DRQ_GRANT" (at 526.415 106.68 0) (fields_autoplaced)
+    (effects (font (size 1.27 1.27)) (justify left bottom))
+  )

Commit message: The great PCB layout-athon
Parts:
- C1, C2, C3, C4, C5: footprint (none) -> Capacitor_THT:C_Disc_D5.0mm_W2.5mm_P5.00mm
- R2: footprint (none) -> Resistor_THT:R_Axial_DIN0207_L6.3mm_D2.5mm_P7.62mm_Horizontal
- U10, U16, U7, U8, U9: footprint (none) -> Package_DIP:DIP-16_W7.62mm
- U11, U12, U13, U14, U4, U5, U6: footprint (none) -> Package_DIP:DIP-20_W7.62mm
- U15, U17, U18, U19, U20: footprint (none) -> Package_DIP:DIP-14_W7.62mm
