File: kicad/Memory/Memory.kicad_pcb (KiCad board)
At the start: 2 copper layers, 206.4 x 137.5 mm, 61 parts, among them J1 Control Connector, J2 Data Connector, U1 CY62256-70PC, U10 74LS257, U11 74LS377, U12 74LS377, U13 74LS377, U14 74LS377, U15 74LS32, U16 74LS257, U17 74LS08, U18 74LS00, U19 74LS27, U2 CY62256-70PC, U20 74LS08, U3 CY62256-70PC, U4 74LS245, U5 74LS245, U6 74LS245, U7 74LS257, U8 74LS257, U9 74LS257

Commit message: Gerber creation marathon
Routing:
- net GND: track 0.00 -> 1164.2 mm
- net +5V: track 0.00 -> 846.1 mm
- net /*SELECT_CORE: track 0.00 -> 411.6 mm
- net /A13: track 0.00 -> 326.8 mm
- net /A12: track 0.00 -> 304.2 mm
- net /M6: track 0.00 -> 296.9 mm, vias 0 -> 2
- net /M4: track 0.00 -> 296.2 mm, vias 0 -> 2
- net /M3: track 0.00 -> 294.3 mm, vias 0 -> 2
- net /M7: track 0.00 -> 290.7 mm
- net /M2: track 0.00 -> 289.3 mm, vias 0 -> 2
- net /A14: track 0.00 -> 286.7 mm
- net /M11: track 0.00 -> 283.5 mm, vias 0 -> 1
- net /M10: track 0.00 -> 277.3 mm, vias 0 -> 3
- net /A2: track 0.00 -> 276.2 mm
- net /M5: track 0.00 -> 272.8 mm
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- added copper zone on B.Cu, net GND
- added copper zone on F.Cu, net GND
Other:
- board text removed: "JLCJLCJLCJLC"
